Commit message: update

File: sobit_mini_description/model/urdf/sobit_mini_description.urdf (robot description, URDF)
Before this commit: robot sobit_mini_description, 54 links, 53 joints
Joints:
- joint depth_link_xtion_joint: origin xyz=0 0.0475 0 rpy=-1.57 0 -1.57 -> xyz=0.02 0.0475 0.0375 rpy=-1.57 0 -1.57
- joint joint11: origin xyz=0 0 0.03 rpy=0 0 0 -> xyz=0 0 0.141 rpy=0 0 -1.57
- joint rgb_link_xtion_joint: origin xyz=0 0.0205 0 rpy=-1.57 0 -1.57 -> xyz=0.02 0.0205 0.0375 rpy=-1.57 0 -1.57
