Commit message: URDFの書き換え

File: sobit_mini_description/model/urdf/kobuki_hexagons_asus_xtion_pro_offset_turtlebot_op.urdf.xacro (robot description, xacro)
@@ -6,7 +6,7 @@
 -->
 <robot name="turtlebot" xmlns:xacro="http://ros.org/wiki/xacro">
-  <xacro:include filename="$(find sobit_mini_description)/model/urdf/turtlebot_op_common_library.urdf.xacro" />
+  <xacro:include filename="$(find sobit_mini_description)/model/urdf/sobit_mini_description_common_library.urdf.xacro" />
   <xacro:include filename="$(find sobit_mini_description)/model/urdf/kobuki.urdf.xacro" />
-  <xacro:include filename="$(find sobit_mini_description)/model/urdf/stacks/turtlebot_op_hexagons.urdf.xacro"/>
+  <xacro:include filename="$(find sobit_mini_description)/model/urdf/stacks/sobit_mini_description_hexagons.urdf.xacro"/>
   <xacro:include filename="$(find sobit_mini_description)/model/urdf/sensors/asus_xtion_pro_offset_fix.urdf.xacro"/>
   <kobuki/>

File: sobit_mini_description/model/urdf/sobit_mini_description.urdf (robot description, URDF)
Before this commit: robot sobit_mini_description, 54 links, 53 joints
Joints:
- joint joint11: origin xyz=0 0 0.141 rpy=0 0 -1.57 -> xyz=0 0 0.22 rpy=0 0 -1.57
