Commit message: urdfの作成

File: sobit_mini_description/robots/backup.xacro (robot description, xacro)
@@ -3,5 +3,5 @@
   <!-- common xacro -->
   <xacro:include filename="$(find sobit_mini_description)/urdf/common.xacro" />
-  <xacro:include filename="$(find hsr_description)/urdf/materials.urdf.xacro" />
+  <xacro:include filename="$(find sobit_mini_description)/urdf/materials.urdf.xacro" />
   <!-- links and joints -->
   <xacro:include filename="$(find sobit_mini_description)/urdf/base/base.urdf.xacro" />
@@ -17,11 +17,11 @@
   <xacro:include filename="$(find sobit_mini_description)/urdf/stacks/stacks.urdf.xacro" />
   <xacro:base/>
-  <xacro:body prefix="body" parent="plate_middle"/>
   <xacro:head prefix="head" parent="body_lift_link"/>
+  <xacro:body prefix="body" parent="plate_middle_link"/>
   <xacro:left_arm prefix="left" parent="body_lift_link"/>
-  <xacro:left_hand prefix="left_hand" parent="body_lift_link"/>
+  <xacro:left_hand prefix="left_hand" parent="left_wrist_flex_joint"/>
   <xacro:ribs prefix="ribs" parent="body_lift_link"/>
   <xacro:right_arm prefix="right" parent="body_lift_link"/>
-  <xacro:right_hand prefix="right_hand" parent="body_lift_link"/>
+  <xacro:right_hand prefix="right_hand" parent="right_wrist_flex_joint"/>
   <xacro:urg parent="base_link"/>
   <xacro:sensor_asus_xtion_pro parent="head_tilt_link"/>

File: sobit_mini_description/robots/sobit_mini.urdf.xacro (robot description, xacro)
@@ -3,5 +3,5 @@
   <!-- common xacro -->
   <xacro:include filename="$(find sobit_mini_description)/urdf/common.xacro" />
-  <xacro:include filename="$(find hsr_description)/urdf/materials.urdf.xacro" />
+  <xacro:include filename="$(find sobit_mini_description)/urdf/materials.urdf.xacro" />
   <!-- links and joints -->
   <xacro:include filename="$(find sobit_mini_description)/urdf/base/base.urdf.xacro" />
@@ -17,13 +17,12 @@
   <xacro:include filename="$(find sobit_mini_description)/urdf/stacks/stacks.urdf.xacro" />
   <xacro:base/>
-  <xacro:head prefix="head" parent="body_lift_link"/>
+  <stack_hexagons parent="base_link" />
+  <xacro:urg parent="base_link"/>
   <xacro:body prefix="body" parent="plate_middle_link"/>
   <xacro:left_arm prefix="left" parent="body_lift_link"/>
-  <xacro:left_hand prefix="left_hand" parent="left_wrist_flex_joint"/>
-  <xacro:ribs prefix="ribs" parent="body_lift_link"/>
   <xacro:right_arm prefix="right" parent="body_lift_link"/>
-  <xacro:right_hand prefix="right_hand" parent="right_wrist_flex_joint"/>
-  <xacro:urg parent="base_link"/>
+  <xacro:left_hand prefix="left_hand" parent="left_wrist_flex_link"/>
+  <xacro:right_hand prefix="right_hand" parent="right_wrist_flex_link"/>
+  <xacro:head prefix="head" parent="body_lift_link"/>
   <xacro:sensor_asus_xtion_pro parent="head_tilt_link"/>
-  <stack_hexagons parent="base_link" />
 </robot>

File: sobit_mini_description/urdf/base/base.urdf.xacro (robot description, xacro)
@@ -190,6 +190,4 @@
       </inertial>
     </link>
-    <!-- Kobuki Gazebo simulation details -->
-    <kobuki_sim />
   </xacro:macro>
 </robot>

File: sobit_mini_description/urdf/body/body.urdf.xacro (robot description, xacro)
@@ -1,6 +1,46 @@
 <?xml version="1.0" encoding="UTF-8" ?>
-<robot name="body" xmlns:xacro="http://ros.org/wiki/xacro">
+<robot name="body"
+  xmlns:xacro="http://ros.org/wiki/xacro">
   <xacro:include filename="$(find sobit_mini_description)/urdf/body/body.transmission.xacro" />
   <xacro:macro name="body" params="prefix parent">
+    <joint name="${prefix}_square_bottom_joint" type="fixed">
+      <parent link="${parent}" />
+      <child link="${prefix}_square_bottom_link" />
+      <origin rpy="0 0 0" xyz="0.017 0 0.0" />
+      <axis xyz="0 0 1" />
+    </joint>
+    <link name="${prefix}_square_bottom_link">
+      <visual>
+        <origin rpy="0 0 0" xyz="0 0 0.003" />
+        <geometry>
+          <box size="0.16 0.16 0.003" />
+        </geometry>
+        <material name="silver" />
+      </visual>
+      <inertial>
+        <origin rpy="0 0 0" xyz="0 0 0.0" />
+        <mass value="1" />
+        <inertia ixx="1.0" ixy="0.0" ixz="0.0" iyy="1.0" iyz="0.0" izz="1.0" />
+      </inertial>
+    </link>
+    <joint name="${prefix}_small_gear_joint" type="fixed">
+      <parent link="${parent}" />
+      <child link="${prefix}_small_gear_link" />
+      <origin rpy="0 0 0" xyz="0.0 0.14 0.0" />
+      <axis xyz="0 0 1" />
+    </joint>
+    <link name="${prefix}_small_gear_link">
+      <visual>
+        <origin rpy="${M_PI/2.0} 0 ${M_PI/2.0}" xyz="0 0 0.034" />
+        <geometry>
+          <mesh filename="package://sobit_mini_description/meshes/sobit_mini_small_gear.dae" />
+        </geometry>
+      </visual>
+      <inertial>
+        <origin rpy="0 0 0" xyz="0 0 0.0" />
+        <mass value="1" />
+        <inertia ixx="1.0" ixy="0.0" ixz="0.0" iyy="1.0" iyz="0.0" izz="1.0" />
+      </inertial>
+    </link>
     <joint name="${prefix}_roll_joint" type="revolute">
       <parent link="${parent}" />
@@ -10,103 +50,88 @@
       <limit effort="30" lower="${-M_PI/2.0}" upper="${M_PI/2}" velocity="${M_PI/2.0}" />
     </joint>
-    <link name="${prefix}_roll_link">
-      <collision>
-        <origin rpy="0 0 0" xyz="0 0 0.03" />
+    <link name="${prefix}_roll_link"/>
+    <joint name="${prefix}_square_top_joint" type="fixed">
+      <parent link="${prefix}_roll_link" />
+      <child link="${prefix}_square_top_link" />
+      <origin rpy="0 0 ${M_PI/4.0}" xyz="0.0 0 0.0135" />
+      <axis xyz="0 0 1" />
+    </joint>
+    <link name="${prefix}_square_top_link">
+      <visual>
+        <origin rpy="0 0 0" xyz="0 0 0.0015" />
         <geometry>
-          <box size="0.16 0.16 0.06" />
+          <box size="0.16 0.16 0.003" />
         </geometry>
-      </collision>
-      <visual>
-        <origin rpy="0 0 0" xyz="0 0 0.03" />
-        <geometry>
-          <box size="0.16 0.16 0.06" />
-        </geometry>
-        <material name="black" />
+        <material name="silver" />
       </visual>
       <inertial>
-        <origin rpy="0 0 0" xyz="0 0 0.03" />
+        <origin rpy="0 0 0" xyz="0 0 0.0" />
         <mass value="1" />
         <inertia ixx="1.0" ixy="0.0" ixz="0.0" iyy="1.0" iyz="0.0" izz="1.0" />
       </inertial>
     </link>
-    <joint name="${prefix}_roll_dummy_joint" type="fixed">
+    <joint name="${prefix}_big_gear_joint" type="fixed">
       <parent link="${prefix}_roll_link" />
-      <child link="${prefix}_roll_dummy_link" />
-      <origin rpy="0 0 0" xyz="-0.03 0 0.06" />
-      <axis xyz="1 0 0" />
-      <limit effort="30" lower="-2.35" upper="0" velocity="1.571" />
+      <child link="${prefix}_big_gear_link" />
+      <origin rpy="0 0 0" xyz="0 0 0.015" />
+      <axis xyz="0 0 1" />
     </joint>
-    <link name="${prefix}_roll_dummy_link">
-      <collision>
-        <origin rpy="0 0 0" xyz="0.0 0.0 0.255" />
+    <link name="${prefix}_big_gear_link">
+      <visual>
+        <origin rpy="${M_PI/2.0} 0 ${M_PI/2.0}" xyz="0 0 0.02" />
         <geometry>
-          <box size="0.02 0.03 0.51" />
+          <mesh filename="package://sobit_mini_description/meshes/sobit_mini_big_gear.dae" />
         </geometry>
-      </collision>
-      <visual>
-        <origin rpy="0 0 0" xyz="0.0 0.0 0.255" />
-        <geometry>
-          <box size="0.02 0.03 0.51" />
-        </geometry>
-        <material name="black" />
       </visual>
       <inertial>
-        <origin rpy="0 0 0" xyz="0.0 0.0 0.255" />
-        <mass value="0.08" />
+        <origin rpy="0 0 0" xyz="0 0 0.0" />
+        <mass value="1" />
+        <inertia ixx="1.0" ixy="0.0" ixz="0.0" iyy="1.0" iyz="0.0" izz="1.0" />
+      </inertial>
+    </link>
+    <joint name="${prefix}_back_pole_joint" type="fixed">
+      <parent link="${prefix}_big_gear_link" />
+      <child link="${prefix}_back_pole_link" />
+      <origin rpy="0 0 0" xyz="-0.03 0 0.019" />
+      <axis xyz="0 0 1" />
+    </joint>
+    <link name="${prefix}_back_pole_link">
+      <visual>
+        <origin rpy="${M_PI/2.0} 0 ${M_PI/2.0}" xyz="-0.01 -0.01 0.0" />
+        <geometry>
+          <mesh filename="package://sobit_mini_description/meshes/sobit_mini_center_back.dae" />
+        </geometry>
+      </visual>
+      <inertial>
+        <origin rpy="0 0 0" xyz="0 0 0.0" />
+        <mass value="1" />
         <inertia ixx="1.0" ixy="0.0" ixz="0.0" iyy="1.0" iyz="0.0" izz="1.0" />
       </inertial>
     </link>
     <joint name="${prefix}_lift_joint" type="prismatic">
-      <parent link="${prefix}_roll_dummy_link" />
+      <parent link="${prefix}_back_pole_link" />
       <child link="${prefix}_lift_link" />
-      <origin rpy="0 0 ${M_PI/2.0}" xyz="0.03 0.0 0.0" />
+      <origin rpy="0 0.01 0" xyz="0.03 0.0 0.03" />
       <axis xyz="0 0 1" />
       <limit effort="30" lower="0" upper="0.17" velocity="0.2" />
       <dynamics damping="1.0" />
     </joint>
-    <link name="${prefix}_lift_link">
-      <collision>
-        <origin rpy="0 0 0" xyz="0.0 0 0.2575" />
+    <link name="${prefix}_lift_link"/>
+    <joint name="${prefix}_front_pole_joint" type="fixed">
+      <parent link="${prefix}_lift_link" />
+      <child link="${prefix}_front_pole_link" />
+      <origin rpy="0 0 0" xyz="0.00 0 0.00" />
+      <axis xyz="0 0 1" />
+    </joint>
+    <link name="${prefix}_front_pole_link">
+      <visual>
+        <origin rpy="${M_PI/2.0} 0 ${M_PI/2.0}" xyz="0.0 0.015 0.513" />
         <geometry>
-          <box size="0.02 0.02 0.515" />
-        </geometry>
-      </collision>
-      <visual>
-        <origin rpy="0 0 0" xyz="0.0 0 0.2575" />
-        <geometry>
-          <box size="0.02 0.02 0.515" />
-        </geometry>
-        <material name="black" />
-      </visual>
-      <inertial>
-        <origin rpy="0 0 0" xyz="0 0 0.2575" />
-        <mass value="0.08" />
-        <inertia ixx="1.0" ixy="0.0" ixz="0.0" iyy="1.0" iyz="0.0" izz="1.0" />
-      </inertial>
-    </link>
-    <joint name="${prefix}_joint" type="fixed">
-      <parent link="${prefix}_lift_link" />
-      <child link="${prefix}_link" />
-      <origin rpy="0 0 0" xyz="0 0 0.3" />
-      <axis xyz="0 0 1" />
-      <limit effort="30" lower="-0.1" upper="0.1" velocity="${M_PI}" />
-    </joint>
-    <!-- sobit Body -->
-    <link name="body_link">
-      <collision>
-        <origin rpy="0 0 0" xyz="0 0 0" />
-        <geometry>
-          <mesh filename="package://sobit_mini_description/meshes/mini_sobit_body_size_fix.dae" />
-        </geometry>
-      </collision>
-      <visual>
-        <origin rpy="0 0 0" xyz="0 0 0" />
-        <geometry>
-          <mesh filename="package://sobit_mini_description/meshes/mini_sobit_body_size_fix.dae" />
+          <mesh filename="package://sobit_mini_description/meshes/sobit_mini_center_front.dae" />
         </geometry>
       </visual>
       <inertial>
-        <origin rpy="0 0 0" xyz="0 0 0" />
-        <mass value="0.08" />
+        <origin rpy="0 0 0" xyz="0 0 0.0" />
+        <mass value="1" />
         <inertia ixx="1.0" ixy="0.0" ixz="0.0" iyy="1.0" iyz="0.0" izz="1.0" />
       </inertial>

File: sobit_mini_description/urdf/head/head.urdf.xacro (robot description, xacro)
@@ -6,5 +6,5 @@
       <parent link="${parent}" />
       <child link="${prefix}_pan_link" />
-      <origin rpy="0 0 0" xyz="0 0 0.515" />
+      <origin rpy="0 0 0" xyz="0 0 0.51217" />
       <axis xyz="0 0 1" />
       <limit effort="30" lower="-2.617" upper="2.617" velocity="${M_PI/2.0}" />
@@ -14,15 +14,12 @@
         <origin rpy="${M_PI/2.0} 0 0" xyz="0 0 0.0135" />
         <geometry>
-          <mesh filename="package://sobit_mini_description/meshes/sobit hed_neck.dae" />
+          <mesh filename="package://sobit_mini_description/meshes/sobit_mini_head_neck.dae" />
         </geometry>
       </collision>
       <visual>
-        <origin rpy="${M_PI/2.0} 0 0" xyz="0 0 0.0135" />
+        <origin rpy="${M_PI/2.0} 0 ${-M_PI/2.0}" xyz="0 -0.01437 0" />
         <geometry>
-          <mesh filename="package://sobit_mini_description/meshes/sobit hed_neck.dae" />
+          <mesh filename="package://sobit_mini_description/meshes/sobit_mini_head_neck.dae" />
         </geometry>
-        <material name="black">
-          <color rgba="0.0 0.0 0.0 1.0" />
-        </material>
       </visual>
       <inertial>
@@ -35,6 +32,6 @@
       <parent link="${prefix}_pan_link" />
       <child link="${prefix}_tilt_link" />
-      <origin rpy="0 0 0" xyz="0 0 0.025" />
-      <axis xyz="1 0 0" />
+      <origin rpy="0 0 0" xyz="0 0 0.01273" />
+      <axis xyz="0 1 0" />
       <limit effort="30" lower="-1" upper="1" velocity="${M_PI/2.0}" />
     </joint>
@@ -43,15 +40,12 @@
         <origin rpy="${M_PI/2.0} 0 0" xyz="0 0 -0.012" />
         <geometry>
-          <mesh filename="package://sobit_mini_description/meshes/sobit hed_top.dae" />
+          <mesh filename="package://sobit_mini_description/meshes/sobit_mini_head_top.dae" />
         </geometry>
       </collision>
       <visual>
-        <origin rpy="${M_PI/2.0} 0 0" xyz="0 0 -0.012" />
+        <origin rpy="${M_PI/2.0} 0 ${-M_PI/2.0}" xyz="0 -0.01435 -0.0157" />
         <geometry>
-          <mesh filename="package://sobit_mini_description/meshes/sobit hed_top.dae" />
+          <mesh filename="package://sobit_mini_description/meshes/sobit_mini_head_top.dae" />
         </geometry>
-        <material name="blue">
-          <color rgba="0.0 0.0 1.0 1.0" />
-        </material>
       </visual>
       <inertial>

File: sobit_mini_description/urdf/left_arm/left_arm.urdf.xacro (robot description, xacro)
@@ -6,24 +6,17 @@
       <parent link="${parent}" />
       <child link="${prefix}_shoulder_fixed_link" />
-      <origin rpy="0 0 0" xyz="0.01 0 0.4" />
+      <origin rpy="0 0 0" xyz="0.0 0 0.343" />
       <axis xyz="0 0 1" />
       <limit effort="30" lower="-0.1" upper="0.1" velocity="1.571" />
     </joint>
     <link name="${prefix}_shoulder_fixed_link">
-      <collision>
-        <origin rpy="0 0 0" xyz="0.0525 0 0.0" />
+      <visual>
+        <origin rpy="${M_PI/2.0} 0 ${M_PI}" xyz="0.0 0.081 0.007" />
         <geometry>
-          <box size="0.105 0.03 0.055" />
+          <mesh filename="package://sobit_mini_description/meshes/sobit_mini_shoulder1.dae" />
         </geometry>
-      </collision>
-      <visual>
-        <origin rpy="0 0 0" xyz="0.0525 0 0.0" />
-        <geometry>
-          <box size="0.105 0.03 0.055" />
-        </geometry>
-        <material name="black" />
       </visual>
       <inertial>
-        <origin rpy="0 0 0" xyz="0.0525 0 0.0" />
+        <origin rpy="0 0 0" xyz="0.0 0 0.0" />
         <mass value="0.08" />
         <inertia ixx="1.0" ixy="0.0" ixz="0.0" iyy="1.0" iyz="0.0" izz="1.0" />
@@ -33,11 +26,11 @@
       <parent link="${prefix}_shoulder_fixed_link" />
       <child link="${prefix}_shoulder_roll_link" />
-      <origin rpy="0 0 0" xyz="0.105 0 0.02" />
-      <axis xyz="1 0 0" />
-      <limit effort="30" lower="${-M_PI/2.0}" upper="0" velocity="${M_PI}" />
+      <origin rpy="0 0 0" xyz="0.0 0.11986 0.03941" />
+      <axis xyz="0 -1 0" />
+      <limit effort="30" lower="${-M_PI/2.0}" upper="${M_PI/2.0}" velocity="${M_PI}" />
     </joint>
     <link name="${prefix}_shoulder_roll_link">
       <collision>
-        <origin rpy="0 0 0" xyz="0.034 0 0.0" />
+        <origin rpy="0 0 0" xyz="0.0 0 0.0" />
         <geometry>
           <box size="0.068 0.05 0.04" />
@@ -45,9 +38,8 @@
       </collision>
       <visual>
-        <origin rpy="0 0 0" xyz="0.034 0 0.0" />
+        <origin rpy="0 ${M_PI/2.0} 0" xyz="0.0 0.0525 0.0" />
         <geometry>
-          <box size="0.068 0.05 0.04" />
+          <mesh filename="package://sobit_mini_description/meshes/sobit_mini_shoulder2.dae" />
         </geometry>
-        <material name="black" />
       </visual>
       <inertial>
@@ -60,7 +52,7 @@
       <parent link="${prefix}_shoulder_roll_link" />
       <child link="${prefix}_shoulder_flex_link" />
-      <origin rpy="0 0 0" xyz="0.053 0.0 0.0" />
-      <axis xyz="0 1 0" />
-      <limit effort="30" lower="${-M_PI}" upper="0" velocity="${M_PI/2.0}" />
+      <origin rpy="${M_PI/2.0} 0 0" xyz="0.0 0.0525 0.0" />
+      <axis xyz="1 0 0" />
+      <limit effort="30" lower="${-M_PI/2.0}" upper="${M_PI/2.0}" velocity="${M_PI/2.0}" />
     </joint>
     <link name="${prefix}_shoulder_flex_link">
@@ -72,9 +64,8 @@
       </collision>
       <visual>
-        <origin rpy="0 0 0" xyz="0.0 0 -0.095" />
+        <origin rpy="0 ${M_PI} ${M_PI/2.0}" xyz="0.018 0.017 -0.14803" />
         <geometry>
-          <box size="0.035 0.05 0.19" />
+          <mesh filename="package://sobit_mini_description/meshes/sobit_mini_arm.dae" />
         </geometry>
-        <material name="black" />
       </visual>
       <inertial>
@@ -86,10 +77,10 @@
     <joint name="${prefix}_wrist_flex_joint" type="revolute">
       <parent link="${prefix}_shoulder_flex_link" />
-      <child link="${prefix}_wrist_flex_joint" />
-      <origin rpy="0 0 0" xyz="0 0 -0.19" />
-      <axis xyz="0 1 0" />
+      <child link="${prefix}_wrist_flex_link" />
+      <origin rpy="0 0 0" xyz="0 0 -0.1892" />
+      <axis xyz="1 0 0" />
       <limit effort="30" lower="${-M_PI/2.0}" upper="${M_PI/2.0}" velocity="${M_PI/2.0}" />
     </joint>
-    <link name="${prefix}_wrist_flex_joint">
+    <link name="${prefix}_wrist_flex_link">
       <collision>
         <origin rpy="0 0 0" xyz="0.0 0 -0.035" />
@@ -99,9 +90,8 @@
       </collision>
       <visual>
-        <origin rpy="0 0 0" xyz="0.0 0 -0.035" />
+        <origin rpy="${M_PI/2.0} 0 ${M_PI/2.0}" xyz="0.021 0.01 -0.029" />
         <geometry>
-          <box size="0.06 0.04 0.07" />
+          <mesh filename="package://sobit_mini_description/meshes/sobit_mini_wrist.dae" />
         </geometry>
-        <material name="black" />
       </visual>
       <inertial>

File: sobit_mini_description/urdf/left_hand/left_hand.urdf.xacro (robot description, xacro)
@@ -3,44 +3,18 @@
   <xacro:include filename="$(find sobit_mini_description)/urdf/left_hand/left_hand.transmission.xacro" />
   <xacro:macro name="left_hand" params="prefix parent">
-    <joint name="${prefix}_base_fixed_joint" type="fixed">
+    <joint name="${prefix}_motor_joint" type="revolute">
       <parent link="${parent}" />
-      <child link="${prefix}_base_fixed_link" />
-      <origin rpy="0 0 0" xyz="0 0 -0.05" />
+      <child link="${prefix}_motor_link" />
       <axis xyz="0 1 0" />
-      <limit effort="30" lower="${-M_PI/2.0}" upper="${M_PI/2.0}" velocity="${M_PI/2.0}" />
+      <limit lower="0.0" upper="${M_PI/2.0}" effort="1" velocity="1" />
     </joint>
-    <link name="${prefix}_base_fixed_link">
-      <collision>
-        <origin rpy="0 ${M_PI} 0" xyz="0.0 0 0" />
-        <geometry>
-          <mesh filename="package://sobit_mini_description/meshes/Manipulator_X4_Gripper_fix.dae" />
-        </geometry>
-      </collision>
-      <visual>
-        <origin rpy="0 ${M_PI} 0" xyz="0.0 0 0" />
-        <geometry>
-          <mesh filename="package://sobit_mini_description/meshes/Manipulator_X4_Gripper_fix.dae" />
-        </geometry>
-      </visual>
-      <inertial>
-        <origin rpy="0 ${M_PI} 0" xyz="0 0 0" />
-        <mass value="0.08" />
-        <inertia ixx="1.0" ixy="0.0" ixz="0.0" iyy="1.0" iyz="0.0" izz="1.0" />
-      </inertial>
-    </link>
-    <joint name="${prefix}_motor_joint" type="revolute">
-      <parent link="${prefix}_base_fixed_link" />
-      <child link="${prefix}_motor_dummy_link" />
-      <axis xyz="1 0 0" />
-      <limit lower="0.0" upper="1.57" effort="1" velocity="1" />
-    </joint>
-    <link name="${prefix}_motor_dummy_link" />
+    <link name="${prefix}_motor_link" />
     <joint name="${prefix}_left_finger_joint" type="revolute">
-      <parent link="${prefix}_base_fixed_link" />
+      <parent link="${parent}" />
       <child link="${prefix}_left_finger_link" />
-      <origin rpy="0 0 0" xyz="0 0.018 -0.043" />
-      <axis xyz="1 0 0" />
+      <origin rpy="0 0 0" xyz="-0.015855 0.0 -0.04202" />
+      <axis xyz="0 1 0" />
       <limit lower="-1.0" upper="0.0" effort="1" velocity="1" />
-      <mimic joint="${prefix}_motor_joint" multiplier="1.0" offset="-1.0" />
+      <mimic joint="${prefix}_motor_joint" multiplier="1.0" offset="-0.1" />
     </joint>
     <link name="${prefix}_left_finger_link">
@@ -48,11 +22,11 @@
         <origin rpy="0 ${M_PI} ${M_PI}" xyz="0 0 0" />
         <geometry>
-          <mesh filename="package://sobit_mini_description/meshes/ManipulatorX4_Finger_left.dae" />
+          <mesh filename="package://sobit_mini_description/meshes/sobit_mini_hand.dae" />
         </geometry>
       </collision>
       <visual>
-        <origin rpy="0 ${M_PI} ${M_PI}" xyz="0 0 0" />
+        <origin rpy="0 ${M_PI/2.0} ${M_PI/2.0}" xyz="0.0164 0.0027 -0.0393" />
         <geometry>
-          <mesh filename="package://sobit_mini_description/meshes/ManipulatorX4_Finger_left.dae" />
+          <mesh filename="package://sobit_mini_description/meshes/sobit_mini_hand.dae" />
         </geometry>
       </visual>
@@ -64,10 +38,10 @@
     </link>
     <joint name="${prefix}_right_finger_joint" type="revolute">
-      <parent link="${prefix}_base_fixed_link" />
+      <parent link="${parent}" />
       <child link="${prefix}_right_finger_link" />
-      <origin rpy="0 0 0" xyz="0 -0.018 -0.043" />
-      <axis xyz="1 0 0" />
+      <origin rpy="0 0 0" xyz="0.015855 0.0 -0.04202" />
+      <axis xyz="0 1 0" />
       <limit lower="0.0" upper="1.0" effort="1" velocity="1" />
-      <mimic joint="${prefix}_motor_joint" multiplier="-1.0" offset="1.0" />
+      <mimic joint="${prefix}_motor_joint" multiplier="-1.0" offset="0.1" />
     </joint>
     <link name="${prefix}_right_finger_link">
@@ -75,11 +49,11 @@
         <origin rpy="0 ${M_PI} 0" xyz="0 0 0" />
         <geometry>
-          <mesh filename="package://sobit_mini_description/meshes/ManipulatorX4_Finger_left.dae" />
+          <mesh filename="package://sobit_mini_description/meshes/sobit_mini_hand.dae" />
         </geometry>
       </collision>
       <visual>
-        <origin rpy="0 ${M_PI} 0" xyz="0 0 0" />
+        <origin rpy="0 ${M_PI/2.0} ${-M_PI/2.0}" xyz="-0.0164 -0.0027 -0.0393" />
         <geometry>
-          <mesh filename="package://sobit_mini_description/meshes/ManipulatorX4_Finger_left.dae" />
+          <mesh filename="package://sobit_mini_description/meshes/sobit_mini_hand.dae" />
         </geometry>
       </visual>

File: sobit_mini_description/urdf/materials.urdf.xacro (robot description, xacro)
@@ -6,4 +6,10 @@
   <material name="black">
     <color rgba="0.1 0.1 0.1 1.0" />
+  </material>
+  <material name="white">
+    <color rgba="1.0 1.0 1.0 1.0" />
+  </material>
+  <material name="silver">
+    <color rgba="0.741 0.752 0.760 1.0" />
   </material>
   <material name="red">
