Commit message: urdfの作成

File: sobit_mini_description/urdf/right_arm/right_arm.urdf.xacro (robot description, xacro)
@@ -6,5 +6,5 @@
       <parent link="${parent}" />
       <child link="${prefix}_shoulder_fixed_link" />
-      <origin rpy="0 0 0" xyz="-0.01 0 0.4" />
+      <origin rpy="0 0 0" xyz="0.0 0 0.343" />
       <axis xyz="0 0 1" />
       <limit effort="30" lower="-0.1" upper="0.1" velocity="1.571" />
@@ -12,5 +12,5 @@
     <link name="${prefix}_shoulder_fixed_link">
       <collision>
-        <origin rpy="0 0 0" xyz="-0.0525 0 0.0" />
+        <origin rpy="0 0 0" xyz="0 0 0.0" />
         <geometry>
           <box size="0.105 0.03 0.055" />
@@ -18,9 +18,8 @@
       </collision>
       <visual>
-        <origin rpy="0 0 0" xyz="-0.0525 0 0.0" />
+        <origin rpy="${M_PI/2.0} 0 0" xyz="0.0 -0.081 0.007" />
         <geometry>
-          <box size="0.105 0.03 0.055" />
+          <mesh filename="package://sobit_mini_description/meshes/sobit_mini_shoulder1.dae" />
         </geometry>
-        <material name="black" />
       </visual>
       <inertial>
@@ -30,10 +29,18 @@
       </inertial>
     </link>
+    <joint name="test_joint" type="fixed">
+      <parent link="${prefix}_shoulder_fixed_link" />
+      <child link="test" />
+      <origin rpy="0 0 0" xyz="0.0 0.11751 0.03822" />
+      <axis xyz="0 0 1" />
+      <limit effort="30" lower="-0.1" upper="0.1" velocity="1.571" />
+    </joint>
+    <link name="test"/>
     <joint name="${prefix}_shoulder_roll_joint" type="revolute">
       <parent link="${prefix}_shoulder_fixed_link" />
       <child link="${prefix}_shoulder_roll_link" />
-      <origin rpy="0 0 0" xyz="-0.105 0 0.02" />
-      <axis xyz="1 0 0" />
-      <limit effort="30" lower="${-M_PI/2.0}" upper="0" velocity="${M_PI/2.0}" />
+      <origin rpy="0 0 0" xyz="0.0 -0.11986 0.03941" />
+      <axis xyz="0 -1 0" />
+      <limit effort="30" lower="${-M_PI/2.0}" upper="${M_PI/2.0}" velocity="${M_PI/2.0}" />
     </joint>
     <link name="${prefix}_shoulder_roll_link">
@@ -45,9 +52,8 @@
       </collision>
       <visual>
-        <origin rpy="0 0 0" xyz="-0.034 0 0.0" />
+        <origin rpy="0 ${-M_PI/2.0} ${M_PI}" xyz="0.0 -0.0525 0.0" />
         <geometry>
-          <box size="0.068 0.05 0.04" />
+          <mesh filename="package://sobit_mini_description/meshes/sobit_mini_shoulder2.dae" />
         </geometry>
-        <material name="black" />
       </visual>
       <inertial>
@@ -60,7 +66,7 @@
       <parent link="${prefix}_shoulder_roll_link" />
       <child link="${prefix}_shoulder_flex_link" />
-      <origin rpy="0 0 0" xyz="-0.053 0.0 0.0" />
-      <axis xyz="0 1 0" />
-      <limit effort="30" lower="0" upper="${M_PI}" velocity="${M_PI/2.0}" />
+      <origin rpy="${-M_PI/2.0} 0 0" xyz="0 -0.0525 0.0" />
+      <axis xyz="-1 0 0" />
+      <limit effort="30" lower="${-M_PI/2.0}" upper="${M_PI/2.0}" velocity="${M_PI/2.0}" />
     </joint>
     <link name="${prefix}_shoulder_flex_link">
@@ -72,9 +78,8 @@
       </collision>
       <visual>
-        <origin rpy="0 0 0" xyz="0.0 0 -0.095" />
+        <origin rpy="0 ${M_PI} ${M_PI/2.0}" xyz="0.018 0.017 -0.14803" />
         <geometry>
-          <box size="0.035 0.05 0.19" />
+          <mesh filename="package://sobit_mini_description/meshes/sobit_mini_arm.dae" />
         </geometry>
-        <material name="black" />
       </visual>
       <inertial>
@@ -86,10 +91,10 @@
     <joint name="${prefix}_wrist_flex_joint" type="revolute">
       <parent link="${prefix}_shoulder_flex_link" />
-      <child link="${prefix}_wrist_flex_joint" />
-      <origin rpy="0 0 0" xyz="0 0 -0.19" />
-      <axis xyz="0 1 0" />
+      <child link="${prefix}_wrist_flex_link" />
+      <origin rpy="0 0 0" xyz="0 0 -0.1892" />
+      <axis xyz="-1 0 0" />
       <limit effort="30" lower="${-M_PI/2.0}" upper="${M_PI/2.0}" velocity="${M_PI/2.0}" />
     </joint>
-    <link name="${prefix}_wrist_flex_joint">
+    <link name="${prefix}_wrist_flex_link">
       <collision>
         <origin rpy="0 0 0" xyz="0.0 0 -0.035" />
@@ -99,9 +104,8 @@
       </collision>
       <visual>
-        <origin rpy="0 0 0" xyz="0.0 0 -0.035" />
+        <origin rpy="${M_PI/2.0} 0 ${-M_PI/2.0}" xyz="-0.021 -0.01 -0.029" />
         <geometry>
-          <box size="0.06 0.04 0.07" />
+          <mesh filename="package://sobit_mini_description/meshes/sobit_mini_wrist.dae" />
         </geometry>
-        <material name="black" />
       </visual>
       <inertial>

File: sobit_mini_description/urdf/right_hand/right_hand.urdf.xacro (robot description, xacro)
@@ -3,22 +3,30 @@
   <xacro:include filename="$(find sobit_mini_description)/urdf/right_hand/right_hand.transmission.xacro" />
   <xacro:macro name="right_hand" params="prefix parent">
-    <joint name="${prefix}_base_fixed_joint" type="fixed">
+    <joint name="${prefix}_motor_joint" type="revolute">
       <parent link="${parent}" />
-      <child link="${prefix}_base_fixed_link" />
-      <origin rpy="0 0 0" xyz="0 0 -0.05" />
+      <child link="${prefix}_motor_link" />
       <axis xyz="0 1 0" />
-      <limit effort="30" lower="${-M_PI/2.0}" upper="${M_PI/2.0}" velocity="${M_PI/2.0}" />
+      <limit lower="0.0" upper="${M_PI/2.0}" effort="1" velocity="1" />
     </joint>
-    <link name="${prefix}_base_fixed_link">
+    <link name="${prefix}_motor_link" />
+    <joint name="${prefix}_left_finger_joint" type="revolute">
+      <parent link="${parent}" />
+      <child link="${prefix}_left_finger_link" />
+      <origin rpy="0 0 0" xyz="0.015855 0.0 -0.04202" />
+      <axis xyz="0 1 0" />
+      <limit lower="-1" upper="0" effort="1" velocity="1" />
+      <mimic joint="${prefix}_motor_joint" multiplier="-1.0" offset="0.1" />
+    </joint>
+    <link name="${prefix}_left_finger_link">
       <collision>
         <origin rpy="0 ${M_PI} 0" xyz="0 0 0" />
         <geometry>
-          <mesh filename="package://sobit_mini_description/meshes/Manipulator_X4_Gripper_fix.dae" />
+          <mesh filename="package://sobit_mini_description/meshes/sobit_mini_hand.dae" />
         </geometry>
       </collision>
       <visual>
-        <origin rpy="0 ${M_PI} 0" xyz="0 0 0" />
+        <origin rpy="0 ${M_PI/2.0} ${-M_PI/2.0}" xyz="-0.0164 -0.0027 -0.0393" />
         <geometry>
-          <mesh filename="package://sobit_mini_description/meshes/Manipulator_X4_Gripper_fix.dae" />
+          <mesh filename="package://sobit_mini_description/meshes/sobit_mini_hand.dae" />
         </geometry>
       </visual>
@@ -29,30 +37,23 @@
       </inertial>
     </link>
-    <joint name="${prefix}_motor_joint" type="revolute">
-      <parent link="${prefix}_base_fixed_link" />
-      <child link="${prefix}_motor_dummy_link" />
-      <axis xyz="1 0 0" />
-      <limit lower="0.0" upper="${M_PI/2.0}" effort="1" velocity="1" />
+    <joint name="${prefix}_right_finger_joint" type="revolute">
+      <parent link="${parent}" />
+      <child link="${prefix}_right_finger_link" />
+      <origin rpy="0 0 0" xyz="-0.015855 0.0 -0.04202" />
+      <axis xyz="0 1 0" />
+      <limit lower="-1.0" upper="0.0" effort="1" velocity="1" />
+      <mimic joint="${prefix}_motor_joint" multiplier="1.0" offset="-0.1" />
     </joint>
-    <link name="${prefix}_motor_dummy_link" />
-    <joint name="${prefix}_left_finger_joint" type="revolute">
-      <parent link="${prefix}_base_fixed_link" />
-      <child link="${prefix}_left_finger_link" />
-      <origin rpy="0 0 0" xyz="0 0.018 -0.043" />
-      <axis xyz="1 0 0" />
-      <limit lower="-1" upper="0" effort="1" velocity="1" />
-      <mimic joint="${prefix}_motor_joint" multiplier="1.0" offset="-1.0" />
-    </joint>
-    <link name="${prefix}_left_finger_link">
+    <link name="${prefix}_right_finger_link">
       <collision>
         <origin rpy="0 ${M_PI} ${M_PI}" xyz="0 0 0" />
         <geometry>
-          <mesh filename="package://sobit_mini_description/meshes/ManipulatorX4_Finger_left.dae" />
+          <mesh filename="package://sobit_mini_description/meshes/sobit_mini_hand.dae" />
         </geometry>
       </collision>
       <visual>
-        <origin rpy="0 ${M_PI} ${M_PI}" xyz="0 0 0" />
+        <origin rpy="0 ${M_PI/2.0} ${M_PI/2.0}" xyz="0.0164 0.0027 -0.0393" />
         <geometry>
-          <mesh filename="package://sobit_mini_description/meshes/ManipulatorX4_Finger_left.dae" />
+          <mesh filename="package://sobit_mini_description/meshes/sobit_mini_hand.dae" />
         </geometry>
       </visual>
@@ -63,31 +64,4 @@
       </inertial>
     </link>
-    <joint name="${prefix}_right_finger_joint" type="revolute">
-      <parent link="${prefix}_base_fixed_link" />
-      <child link="${prefix}_right_finger_link" />
-      <origin rpy="0 0 0" xyz="0 -0.018 -0.043" />
-      <axis xyz="1 0 0" />
-      <limit lower="0.0" upper="1" effort="1" velocity="1" />
-      <mimic joint="${prefix}_motor_joint" multiplier="-1.0" offset="1.0" />
-    </joint>
-    <link name="${prefix}_right_finger_link">
-      <collision>
-        <origin rpy="0 ${M_PI} 0" xyz="0 0 0" />
-        <geometry>
-          <mesh filename="package://sobit_mini_description/meshes/ManipulatorX4_Finger_left.dae" />
-        </geometry>
-      </collision>
-      <visual>
-        <origin rpy="0 ${M_PI} 0" xyz="0 0 0" />
-        <geometry>
-          <mesh filename="package://sobit_mini_description/meshes/ManipulatorX4_Finger_left.dae" />
-        </geometry>
-      </visual>
-      <inertial>
-        <origin rpy="0 ${M_PI} 0" xyz="0 0 0" />
-        <mass value="0.08" />
-        <inertia ixx="1.0" ixy="0.0" ixz="0.0" iyy="1.0" iyz="0.0" izz="1.0" />
-      </inertial>
-    </link>
     <xacro:right_hand_transmission prefix="${prefix}"/>
   </xacro:macro>

File: sobit_mini_description/urdf/sensor/xtion.urdf.xacro (robot description, xacro)
@@ -8,16 +8,21 @@
   <xacro:property name="asus_xtion_pro_depth_rel_rgb_py" value="0.0270" />
   <xacro:property name="asus_xtion_pro_cam_rel_rgb_py" value="-0.0220" />
-  <xacro:include filename="$(find sobit_mini_description)/urdf/sensor/xtion_properties.urdf.xacro" />
   <!-- Parameterised in part by the values in turtlebot_properties.urdf.xacro -->
   <xacro:macro name="sensor_asus_xtion_pro" params="parent">
+    <joint name="camera_fixed_joint" type="fixed">
+      <origin xyz="0.0 0.0 0.165" rpy="0 0 0" />
+      <parent link="${parent}" />
+      <child link="camera_fixed_link" />
+    </joint>
+    <link name="camera_fixed_link" />
     <joint name="camera_rgb_joint" type="fixed">
-      <origin xyz="${cam_px} ${cam_py} ${cam_pz}" rpy="${cam_or} ${cam_op} ${cam_oy}" />
-      <parent link="${parent}" />
-      <child link="camera_rgb_frame" />
+      <origin xyz="0.013 0.0220 0.022" rpy="0 -0.1221 0" />
+      <parent link="camera_fixed_link" />
+      <child link="rgb_link" />
     </joint>
-    <link name="camera_rgb_frame" />
+    <link name="rgb_link" />
     <joint name="camera_rgb_optical_joint" type="fixed">
       <origin xyz="0 0 0" rpy="${-M_PI/2} 0 ${-M_PI/2}" />
-      <parent link="camera_rgb_frame" />
+      <parent link="rgb_link" />
       <child link="camera_rgb_optical_frame" />
     </joint>
@@ -25,5 +30,5 @@
     <joint name="camera_joint" type="fixed">
       <origin xyz="0 ${asus_xtion_pro_cam_rel_rgb_py} 0" rpy="0 0 0" />
-      <parent link="camera_rgb_frame" />
+      <parent link="rgb_link" />
       <child link="camera_link" />
     </joint>
@@ -49,16 +54,14 @@
     <joint name="camera_depth_joint" type="fixed">
       <origin xyz="0 ${asus_xtion_pro_depth_rel_rgb_py} 0" rpy="0 0 0" />
-      <parent link="camera_rgb_frame" />
-      <child link="camera_depth_frame" />
+      <parent link="rgb_link" />
+      <child link="depth_link" />
     </joint>
-    <link name="camera_depth_frame" />
+    <link name="depth_link" />
     <joint name="camera_depth_optical_joint" type="fixed">
       <origin xyz="0 0 0" rpy="${-M_PI/2} 0 ${-M_PI/2}" />
-      <parent link="camera_depth_frame" />
+      <parent link="depth_link" />
       <child link="camera_depth_optical_frame" />
     </joint>
     <link name="camera_depth_optical_frame" />
-    <!-- RGBD sensor for simulation, same as Kinect -->
-    <turtlebot_sim_3dsensor />
   </xacro:macro>
 </robot>

File: sobit_mini_description/urdf/stacks/stacks.urdf.xacro (robot description, xacro)
@@ -45,5 +45,5 @@
         <origin xyz="0 0 0" rpy="0 ${M_PI} 0" />
         <geometry>
-          <mesh filename="package://turtlebot_description/meshes/stacks/hexagons/pole_middle.dae" />
+          <mesh filename="package://turtlebot_description/meshes/sensors/sensor_pole.dae" />
         </geometry>
       </visual>
@@ -149,10 +149,10 @@
       </inertial>
     </link>
-    <stack_middle_pole parent="${parent}" number="0" x_loc="0.0381" y_loc="0.1505" z_loc="0.1640" />
-    <stack_middle_pole parent="${parent}" number="1" x_loc="0.0381" y_loc="-0.1505" z_loc="0.1640" />
-    <stack_middle_pole parent="${parent}" number="2" x_loc="-0.0381" y_loc="0.1505" z_loc="0.1640" />
-    <stack_middle_pole parent="${parent}" number="3" x_loc="-0.0381" y_loc="-0.1505" z_loc="0.1640" />
+    <stack_middle_pole parent="${parent}" number="0" x_loc="0.0381" y_loc="0.1505" z_loc="0.1735" />
+    <stack_middle_pole parent="${parent}" number="1" x_loc="0.0381" y_loc="-0.1505" z_loc="0.1735" />
+    <stack_middle_pole parent="${parent}" number="2" x_loc="-0.0381" y_loc="0.1505" z_loc="0.1735" />
+    <stack_middle_pole parent="${parent}" number="3" x_loc="-0.0381" y_loc="-0.1505" z_loc="0.1735" />
     <joint name="plate_middle_joint" type="fixed">
-      <origin xyz="-0.01364 0.0 0.1874" rpy="0 0 0" />
+      <origin xyz="-0.01364 0.0 0.222" rpy="0 0 0" />
       <parent link="${parent}" />
       <child link="plate_middle_link" />
@@ -162,5 +162,5 @@
         <origin xyz="0 0 0" rpy="0 0 0" />
         <geometry>
-          <mesh filename="package://turtlebot_description/meshes/stacks/hexagons/plate_middle.dae" />
+          <mesh filename="package://turtlebot_description/meshes/stacks/hexagons/plate_top.dae" />
         </geometry>
       </visual>
