Commit message: モーターの位置修正

File: sobit_mini_description/robots/test.urdf (robot description, URDF)
Before this commit: robot sobit_mini, 52 links, 51 joints
Links:
- removed link body_link
- removed link body_roll_dummy_link
- removed link camera_depth_frame
- removed link camera_rgb_frame
- removed link left_hand_base_fixed_link
- removed link left_wrist_flex_joint
- removed link pole_middle_0_link
- removed link pole_middle_1_link
- removed link pole_middle_2_link
- removed link pole_middle_3_link
- removed link ribs_left_link
- removed link ribs_right_link
- removed link right_hand_base_fixed_link
- removed link right_hand_motor_dummy_link
- removed link right_wrist_flex_joint
- added link body_back_pole_link, mass 1; visual mesh filename=package://sobit_mini_description/meshes/sobit_mini_center_b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
- added link body_big_gear_link, mass 1; visual mesh filename=package://sobit_mini_description/meshes/sobit_mini_big_gear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
- added link body_front_pole_link, mass 1; visual mesh filename=package://sobit_mini_description/meshes/sobit_mini_center_f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
- added link body_small_gear_link, mass 1; visual mesh filename=package://sobit_mini_description/meshes/sobit_mini_small_ge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
- added link body_square_bottom_link, mass 1; visual box size=0.16 0.16 0.003
- added link body_square_top_link, mass 1; visual box size=0.16 0.16 0.003
- added link camera_fixed_link
- added link depth_link
- added link left_elbow_roll_link, mass 0.08; collision box size=0.06 0.04 0.07; visual mesh filename=package://sobit_mini_description/meshes/arm2_left.dae
- added link left_hand_motor_link
- added link pole_kinect_0_link, mass 0.020; collision cylinder length=0.0936 radius=0.006; visual mesh filename=package://turtlebot_description/meshes/sensors/sensor_pole.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
- added link pole_kinect_1_link, mass 0.020; collision cylinder length=0.0936 radius=0.006; visual mesh filename=package://turtlebot_description/meshes/sensors/sensor_pole.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
- added link pole_kinect_2_link, mass 0.020; collision cylinder length=0.0936 radius=0.006; visual mesh filename=package://turtlebot_description/meshes/sensors/sensor_pole.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
- added link pole_kinect_3_link, mass 0.020; collision cylinder length=0.0936 radius=0.006; visual mesh filename=package://turtlebot_description/meshes/sensors/sensor_pole.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
- added link rgb_link
- added link right_elbow_roll_link, mass 0.08; collision box size=0.06 0.04 0.07; visual mesh filename=package://sobit_mini_description/meshes/arm2_right.dae
- added link right_hand_motor_dummylink
- added link right_hand_motor_link
- link body_lift_link: mass 0.08 -> None; geometry 
- link body_roll_link: mass 1 -> None; geometry 
- link head_pan_link: geometry collision mesh filename=package://sobit_mini_description/meshes/sobit_mini_head_nec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; visual mesh filename=package://sobit_mini_description/meshes/sobit_mini_head_nec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
- link head_tilt_link: geometry collision mesh filename=package://sobit_mini_description/meshes/sobit_mini_head_top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; visual mesh filename=package://sobit_mini_description/meshes/sobit_mini_head_top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
- link left_hand_left_finger_link: geometry collision mesh filename=package://sobit_mini_description/meshes/sobit_mini_hand.dae; visual mesh filename=package://sobit_mini_description/meshes/sobit_mini_hand.dae
- link left_hand_right_finger_link: geometry collision mesh filename=package://sobit_mini_description/meshes/sobit_mini_hand.dae; visual mesh filename=package://sobit_mini_description/meshes/sobit_mini_hand.dae
- link left_shoulder_fixed_link: geometry visual mesh filename=package://sobit_mini_description/meshes/shoulder1.dae
- link left_shoulder_flex_link: geometry collision box size=0.035 0.05 0.19; visual mesh filename=package://sobit_mini_description/meshes/arm1_left.dae
- link left_shoulder_roll_link: geometry collision box size=0.068 0.05 0.04; visual mesh filename=package://sobit_mini_description/meshes/sobit_mini_shoulder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
- link right_hand_left_finger_link: geometry collision mesh filename=package://sobit_mini_description/meshes/sobit_mini_hand.dae; visual mesh filename=package://sobit_mini_description/meshes/sobit_mini_hand.dae
- link right_hand_right_finger_link: geometry collision mesh filename=package://sobit_mini_description/meshes/sobit_mini_hand.dae; visual mesh filename=package://sobit_mini_description/meshes/sobit_mini_hand.dae
- link right_shoulder_fixed_link: geometry collision box size=0.105 0.03 0.055; visual mesh filename=package://sobit_mini_description/meshes/shoulder1.dae
- link right_shoulder_flex_link: geometry collision box size=0.035 0.05 0.19; visual mesh filename=package://sobit_mini_description/meshes/arm1_right.dae
- link right_shoulder_roll_link: geometry collision box size=0.068 0.05 0.04; visual mesh filename=package://sobit_mini_description/meshes/sobit_mini_shoulder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
Joints:
- removed joint body_joint
- removed joint body_roll_dummy_joint
- removed joint left_hand_base_fixed_joint
- removed joint left_wrist_flex_joint
- removed joint pole_middle_0_joint
- removed joint pole_middle_1_joint
- removed joint pole_middle_2_joint
- removed joint pole_middle_3_joint
- removed joint ribs_left_fixed_joint
- removed joint ribs_right_fixed_joint
- removed joint right_hand_base_fixed_joint
- removed joint right_wrist_flex_joint
- added joint body_back_pole_joint: type fixed, parent body_big_gear_link, child body_back_pole_link, origin xyz=-0.03 0 0.019 rpy=0 0 0, axis 0 0 1
- added joint body_big_gear_joint: type fixed, parent body_roll_link, child body_big_gear_link, origin xyz=0 0 0.015 rpy=0 0 0, axis 0 0 1
- added joint body_front_pole_joint: type fixed, parent body_lift_link, child body_front_pole_link, origin xyz=0.00 0 0.00 rpy=0 0 0, axis 0 0 1
- added joint body_small_gear_joint: type fixed, parent plate_middle_link, child body_small_gear_link, origin xyz=0.0 0.14 0.0 rpy=0 0 0, axis 0 0 1
- added joint body_square_bottom_joint: type fixed, parent plate_middle_link, child body_square_bottom_link, origin xyz=0.017 0 0.0 rpy=0 0 0, axis 0 0 1
- added joint body_square_top_joint: type fixed, parent body_roll_link, child body_square_top_link, origin xyz=0.0 0 0.0135 rpy=0 0 0.785398163397, axis 0 0 1
- added joint camera_fixed_joint: type fixed, parent head_tilt_link, child camera_fixed_link, origin xyz=0.0 0.0 0.165 rpy=0 0 0
- added joint left_elbow_roll_joint: type revolute, parent left_shoulder_flex_link, child left_elbow_roll_link, origin xyz=-0.0005 0.1105 0 rpy=0 0 0, axis 0 0 -1, limit lower=-1.57079632679 upper=1.57079632679 effort=30 velocity=1.57079632679
- added joint left_hand_motor_dummy_joint: type fixed, parent left_elbow_roll_link, child left_hand_motor_dummy_link, origin xyz=0 0.15 0 rpy=1.57079632679 -1.57079632679 0, axis 0 1 0, limit lower=0.0 upper=1.57079632679 effort=1 velocity=1
- added joint pole_kinect_0_joint: type fixed, parent base_link, child pole_kinect_0_link, origin xyz=0.0381 0.1505 0.1735 rpy=0 0 0
- added joint pole_kinect_1_joint: type fixed, parent base_link, child pole_kinect_1_link, origin xyz=0.0381 -0.1505 0.1735 rpy=0 0 0
- added joint pole_kinect_2_joint: type fixed, parent base_link, child pole_kinect_2_link, origin xyz=-0.0381 0.1505 0.1735 rpy=0 0 0
- added joint pole_kinect_3_joint: type fixed, parent base_link, child pole_kinect_3_link, origin xyz=-0.0381 -0.1505 0.1735 rpy=0 0 0
- added joint right_elbow_roll_joint: type revolute, parent right_shoulder_flex_link, child right_elbow_roll_link, origin xyz=-0.0005 -0.1105 0 rpy=0 0 0, axis 0 0 1, limit lower=-1.57079632679 upper=1.57079632679 effort=30 velocity=1.57079632679
- added joint right_hand_motor_dummy_joint: type fixed, parent right_elbow_roll_link, child right_hand_motor_dummylink, origin xyz=0 -0.15 0 rpy=-1.57079632679 1.57079632679 0, axis 0 1 0, limit lower=0.0 upper=1.57079632679 effort=1 velocity=1
- joint body_lift_joint: origin xyz=0.03 0.0 0.0 rpy=0 0 1.57079632679 -> xyz=0.03 0.0 0.03 rpy=0 0.01 0; parent body_roll_dummy_link -> body_back_pole_link; type prismatic -> fixed
- joint camera_depth_joint: child camera_depth_frame -> depth_link; parent camera_rgb_frame -> rgb_link
- joint camera_depth_optical_joint: parent camera_depth_frame -> depth_link
- joint camera_joint: parent camera_rgb_frame -> rgb_link
- joint camera_rgb_joint: child camera_rgb_frame -> rgb_link; origin xyz=0 0 0.2 rpy=0 0 -1.57 -> xyz=0.011 0.0220 0.022 rpy=0 -0.1221 0; parent head_tilt_link -> camera_fixed_link
- joint camera_rgb_optical_joint: parent camera_rgb_frame -> rgb_link
- joint head_pan_joint: origin xyz=0 0 0.515 rpy=0 0 0 -> xyz=0 0 0.51217 rpy=0 0 0
- joint head_tilt_joint: axis 1 0 0 -> 0 1 0; origin xyz=0 0 0.025 rpy=0 0 0 -> xyz=0 0 0.01273 rpy=0 0 0
- joint left_hand_left_finger_joint: axis 1 0 0 -> 0 1 0; mimic joint=left_hand_motor_joint multiplier=1.0 offset=-1.0 -> joint=left_hand_motor_joint multiplier=1.0 offset=-0.1; origin xyz=0 0.018 -0.043 rpy=0 0 0 -> xyz=-0.015855 0.0 0.0 rpy=0 0 0; parent left_hand_base_fixed_link -> left_hand_motor_dummy_link
- joint left_hand_motor_joint: axis 1 0 0 -> 0 1 0; child left_hand_motor_dummy_link -> left_hand_motor_link; limit lower=0.0 upper=1.57 effort=1 velocity=1 -> lower=0.0 upper=1.57079632679 effort=1 velocity=1; origin (none) -> xyz=0 0 0 rpy=0 0 0; parent left_hand_base_fixed_link -> left_hand_motor_dummy_link
- joint left_hand_right_finger_joint: axis 1 0 0 -> 0 1 0; mimic joint=left_hand_motor_joint multiplier=-1.0 offset=1.0 -> joint=left_hand_motor_joint multiplier=-1.0 offset=0.1; origin xyz=0 -0.018 -0.043 rpy=0 0 0 -> xyz=0.015855 0.0 0.0 rpy=0 0 0; parent left_hand_base_fixed_link -> left_hand_motor_dummy_link
- joint left_shoulder_fixed_joint: origin xyz=0.01 0 0.4 rpy=0 0 0 -> xyz=0.0 0 0.343 rpy=0 0 0
- joint left_shoulder_flex_joint: axis 0 1 0 -> 1 0 0; limit lower=-3.14159265359 upper=0 effort=30 velocity=1.57079632679 -> lower=-1.57079632679 upper=1.57079632679 effort=30 velocity=1.57079632679; origin xyz=0.053 0.0 0.0 rpy=0 0 0 -> xyz=0 0.0511 0.0 rpy=0 0 0
- joint left_shoulder_roll_joint: axis 1 0 0 -> 0 -1 0; limit lower=-1.57079632679 upper=0 effort=30 velocity=3.14159265359 -> lower=-1.57079632679 upper=1.57079632679 effort=30 velocity=3.14159265359; origin xyz=0.105 0 0.02 rpy=0 0 0 -> xyz=0.0 0.14146 0.03941 rpy=0 0 0
- joint plate_middle_joint: origin xyz=-0.01364 0.0 0.1874 rpy=0 0 0 -> xyz=-0.01364 0.0 0.222 rpy=0 0 0
- joint right_hand_left_finger_joint: axis 1 0 0 -> 0 1 0; mimic joint=right_hand_motor_joint multiplier=1.0 offset=-1.0 -> joint=right_hand_motor_joint multiplier=-1.0 offset=0.1; origin xyz=0 0.018 -0.043 rpy=0 0 0 -> xyz=0.015855 0.0 0 rpy=0 0 0; parent right_hand_base_fixed_link -> right_hand_motor_dummylink
- joint right_hand_motor_joint: axis 1 0 0 -> 0 1 0; child right_hand_motor_dummy_link -> right_hand_motor_link; origin (none) -> xyz=0 0 0 rpy=0 0 0; parent right_hand_base_fixed_link -> right_hand_motor_dummylink
- joint right_hand_right_finger_joint: axis 1 0 0 -> 0 1 0; limit lower=0.0 upper=1 effort=1 velocity=1 -> lower=-1.0 upper=0.0 effort=1 velocity=1; mimic joint=right_hand_motor_joint multiplier=-1.0 offset=1.0 -> joint=right_hand_motor_joint multiplier=1.0 offset=-0.1; origin xyz=0 -0.018 -0.043 rpy=0 0 0 -> xyz=-0.015855 0.0 0 rpy=0 0 0; parent right_hand_base_fixed_link -> right_hand_motor_dummylink
- joint right_shoulder_fixed_joint: origin xyz=-0.01 0 0.4 rpy=0 0 0 -> xyz=0.0 0 0.343 rpy=0 0 0
- joint right_shoulder_flex_joint: axis 0 1 0 -> -1 0 0; limit lower=0 upper=3.14159265359 effort=30 velocity=1.57079632679 -> lower=-1.57079632679 upper=1.57079632679 effort=30 velocity=1.57079632679; origin xyz=-0.053 0.0 0.0 rpy=0 0 0 -> xyz=0 -0.0511 0.0 rpy=0 0 0
- joint right_shoulder_roll_joint: axis 1 0 0 -> 0 -1 0; limit lower=-1.57079632679 upper=0 effort=30 velocity=1.57079632679 -> lower=-1.57079632679 upper=1.57079632679 effort=30 velocity=1.57079632679; origin xyz=-0.105 0 0.02 rpy=0 0 0 -> xyz=0.0 -0.14146 0.03941 rpy=0 0 0

File: sobit_mini_description/urdf/body/body.transmission.xacro (robot description, xacro)
@@ -2,5 +2,5 @@
 <robot xmlns:xacro="http://ros.org/wiki/xacro">
   <xacro:macro name="body_transmission" params="prefix">
-    <position_joint_transmission joint="${prefix}_lift_joint" reduction="1" />
+    <!--position_joint_transmission joint="${prefix}_lift_joint" reduction="1" /-->
     <position_joint_transmission joint="${prefix}_roll_joint" reduction="1" />
   </xacro:macro>

File: sobit_mini_description/urdf/body/body.urdf.xacro (robot description, xacro)
@@ -109,8 +109,8 @@
       </inertial>
     </link>
-    <joint name="${prefix}_lift_joint" type="prismatic">
+    <joint name="${prefix}_lift_joint" type="fixed">
       <parent link="${prefix}_back_pole_link" />
       <child link="${prefix}_lift_link" />
-      <origin rpy="0 0.01 0" xyz="0.03 0.0 0.03" />
+      <origin rpy="0 0.0 0" xyz="0.03 0.0 0.03" />
       <axis xyz="0 0 1" />
       <limit effort="30" lower="0" upper="0.17" velocity="0.2" />

File: sobit_mini_description/urdf/sensor/xtion.urdf.xacro (robot description, xacro)
@@ -17,5 +17,5 @@
     <link name="camera_fixed_link" />
     <joint name="camera_rgb_joint" type="fixed">
-      <origin xyz="0.011 0.0220 0.022" rpy="0 -0.1221 0" />
+      <origin xyz="0.011 0.0220 0.022" rpy="0 -0.0 0" />
       <parent link="camera_fixed_link" />
       <child link="rgb_link" />
