Commit message: urdf の修正

File: sobit_mini_description/robots/sobit_mini.urdf.xacro (robot description, xacro)
@@ -20,5 +20,5 @@
   <stack_hexagons parent="base_link" />
   <xacro:urg parent="base_link"/>
-  <xacro:real_sense parent="base_link"/>
+  <xacro:real_sense child="base_footprint"/>
   <xacro:body prefix="body" parent="plate_middle_link"/>
   <xacro:left_arm prefix="left" parent="body_lift_link"/>

File: sobit_mini_description/urdf/sensor/real_sense.urdf.xacro (robot description, xacro)
@@ -1,11 +1,11 @@
 <?xml version="1.0" encoding="UTF-8" ?>
 <robot name="real_sense" xmlns:xacro="http://ros.org/wiki/xacro">
-  <xacro:macro name="real_sense" params="parent">
+  <xacro:macro name="real_sense" params="child">
+    <link name="t265_odom_frame"/>
     <joint name="real_sense_joint" type="fixed">
       <origin xyz="0.205 0.0 0.01" rpy="0 0 0" />
-      <parent link="${parent}" />
-      <child link="t265_odom_frame" />
+      <parent link="t265_odom_frame" />
+      <child link="${child}" />
     </joint>
-    <link name="t265_odom_frame"/>
   </xacro:macro>
 </robot>

Commit message: urdfの修正

File: sobit_mini_description/robots/sobit_mini.urdf.xacro (robot description, xacro)
@@ -15,10 +15,8 @@
   <xacro:include filename="$(find sobit_mini_description)/urdf/sensor/urg.urdf.xacro" />
   <xacro:include filename="$(find sobit_mini_description)/urdf/sensor/xtion.urdf.xacro" />
-  <xacro:include filename="$(find sobit_mini_description)/urdf/sensor/real_sense.urdf.xacro" />
   <xacro:include filename="$(find sobit_mini_description)/urdf/stacks/stacks.urdf.xacro" />
   <xacro:base/>
   <stack_hexagons parent="base_link" />
   <xacro:urg parent="base_link"/>
-  <xacro:real_sense child="base_footprint"/>
   <xacro:body prefix="body" parent="plate_middle_link"/>
   <xacro:left_arm prefix="left" parent="body_lift_link"/>

File: sobit_mini_description/urdf/right_arm/right_arm.urdf.xacro (robot description, xacro)
@@ -18,7 +18,7 @@
       </collision>
       <visual>
-        <origin rpy="${M_PI/2.0} 0 0" xyz="0.0 -0.081 0.007" />
+        <origin rpy="${M_PI/2.0} 0 0" xyz="-0.0199 -0.09019 -0.0089" />
         <geometry>
-          <mesh filename="package://sobit_mini_description/meshes/sobit_mini_shoulder1.dae" />
+          <mesh filename="package://sobit_mini_description/meshes/shoulder1.dae" />
         </geometry>
       </visual>
@@ -29,16 +29,8 @@
       </inertial>
     </link>
-    <joint name="test_joint" type="fixed">
-      <parent link="${prefix}_shoulder_fixed_link" />
-      <child link="test" />
-      <origin rpy="0 0 0" xyz="0.0 0.11751 0.03822" />
-      <axis xyz="0 0 1" />
-      <limit effort="30" lower="-0.1" upper="0.1" velocity="1.571" />
-    </joint>
-    <link name="test"/>
     <joint name="${prefix}_shoulder_roll_joint" type="revolute">
       <parent link="${prefix}_shoulder_fixed_link" />
       <child link="${prefix}_shoulder_roll_link" />
-      <origin rpy="0 0 0" xyz="0.0 -0.11986 0.03941" />
+      <origin rpy="0 0 0" xyz="0.0 -0.13946 0.03941" />
       <axis xyz="0 -1 0" />
       <limit effort="30" lower="${-M_PI/2.0}" upper="${M_PI/2.0}" velocity="${M_PI/2.0}" />
@@ -80,5 +72,5 @@
         <origin rpy="0 ${M_PI} ${M_PI/2.0}" xyz="0.018 0.017 -0.14803" />
         <geometry>
-          <mesh filename="package://sobit_mini_description/meshes/sobit_mini_arm.dae" />
+          <mesh filename="package://sobit_mini_description/meshes/arm1_right.dae" />
         </geometry>
       </visual>
@@ -106,5 +98,5 @@
         <origin rpy="${M_PI/2.0} 0 ${-M_PI/2.0}" xyz="-0.021 -0.01 -0.029" />
         <geometry>
-          <mesh filename="package://sobit_mini_description/meshes/sobit_mini_wrist.dae" />
+          <mesh filename="package://sobit_mini_description/meshes/arm2_right.dae" />
         </geometry>
       </visual>

Commit message: モーター修正終了

File: sobit_mini_description/robots/sobit_mini.urdf.xacro (robot description, xacro)
@@ -22,6 +22,6 @@
   <xacro:left_arm prefix="left" parent="body_lift_link"/>
   <xacro:right_arm prefix="right" parent="body_lift_link"/>
-  <xacro:left_hand prefix="left_hand" parent="left_wrist_flex_link"/>
-  <xacro:right_hand prefix="right_hand" parent="right_wrist_flex_link"/>
+  <xacro:left_hand prefix="left_hand" parent="left_elbow_roll_link"/>
+  <xacro:right_hand prefix="right_hand" parent="right_elbow_roll_link"/>
   <xacro:head prefix="head" parent="body_lift_link"/>
   <xacro:sensor_asus_xtion_pro parent="head_tilt_link"/>

File: sobit_mini_description/urdf/left_arm/left_arm.urdf.xacro (robot description, xacro)
@@ -75,12 +75,12 @@
       </inertial>
     </link>
-    <joint name="${prefix}_wrist_flex_joint" type="revolute">
+    <joint name="${prefix}_elbow_roll_joint" type="revolute">
       <parent link="${prefix}_shoulder_flex_link" />
-      <child link="${prefix}_wrist_flex_link" />
+      <child link="${prefix}_elbow_roll_link" />
       <origin rpy="0 0 0" xyz="-0.0005 0.1105 0" />
-      <axis xyz="0 0 1" />
+      <axis xyz="0 0 -1" />
       <limit effort="30" lower="${-M_PI/2.0}" upper="${M_PI/2.0}" velocity="${M_PI/2.0}" />
     </joint>
-    <link name="${prefix}_wrist_flex_link">
+    <link name="${prefix}_elbow_roll_link">
       <collision>
         <origin rpy="0 0 0" xyz="0.0 0 -0.035" />

File: sobit_mini_description/urdf/right_arm/right_arm.urdf.xacro (robot description, xacro)
@@ -81,12 +81,12 @@
       </inertial>
     </link>
-    <joint name="${prefix}_wrist_flex_joint" type="revolute">
+    <joint name="${prefix}_elbow_roll_joint" type="revolute">
       <parent link="${prefix}_shoulder_flex_link" />
-      <child link="${prefix}_wrist_flex_link" />
+      <child link="${prefix}_elbow_roll_link" />
       <origin rpy="0 0 0" xyz="-0.0005 -0.1105 0" />
       <axis xyz="0 0 1" />
       <limit effort="30" lower="${-M_PI/2.0}" upper="${M_PI/2.0}" velocity="${M_PI/2.0}" />
     </joint>
-    <link name="${prefix}_wrist_flex_link">
+    <link name="${prefix}_elbow_roll_link">
       <collision>
         <origin rpy="0 0 0" xyz="0.0 0 -0.035" />

Commit message: fix xacro for noetic

File: sobit_mini_description/robots/sobit_mini.urdf.xacro (robot description, xacro)
@@ -1,4 +1,4 @@
 <?xml version="1.0" ?>
-<robot name="sobit_mini" xmlns:controller="http://playerstage.sourceforge.net/gazebo/xmlschema/#controller" xmlns:interface="http://playerstage.sourceforge.net/gazebo/xmlschema/#interface" xmlns:sensor="http://playerstage.sourceforge.net/gazebo/xmlschema/#sensor" xmlns:xacro="http://www.ros.org/wiki.xacro">
+<robot name="sobit_mini" xmlns:controller="http://playerstage.sourceforge.net/gazebo/xmlschema/#controller" xmlns:interface="http://playerstage.sourceforge.net/gazebo/xmlschema/#interface" xmlns:sensor="http://playerstage.sourceforge.net/gazebo/xmlschema/#sensor" xmlns:xacro="http://www.ros.org/wiki/xacro">
   <!-- common xacro -->
   <xacro:include filename="$(find sobit_mini_description)/urdf/common.xacro" />
@@ -18,5 +18,5 @@
   <xacro:include filename="$(find sobit_education_description)/urdf/urg_sup/urg_sup.urdf.xacro" />
   <xacro:base/>
-  <stack_hexagons parent="base_link" />
+  <xacro:stack_hexagons parent="base_link" />
   <xacro:urg_sup parent="plate_bottom_link"/>
   <xacro:urg parent="base_urg_sup_link"/>

File: sobit_mini_description/urdf/body/body.urdf.xacro (robot description, xacro)
@@ -1,5 +1,4 @@
 <?xml version="1.0" encoding="UTF-8" ?>
-<robot name="body"
-  xmlns:xacro="http://ros.org/wiki/xacro">
+<robot name="body" xmlns:xacro="http://ros.org/wiki/xacro">
   <xacro:include filename="$(find sobit_mini_description)/urdf/body/body.transmission.xacro" />
   <xacro:macro name="body" params="prefix parent">

File: sobit_mini_description/urdf/common.xacro (robot description, xacro)
@@ -1,6 +1,6 @@
 <?xml version="1.0" ?>
-<robot xmlns:xacro="http://www.ros.org/wiki.xacro">
+<robot xmlns:xacro="http://www.ros.org/wiki/xacro">
   <xacro:property name="M_PI" value="3.14159265359" />
-  <macro name="position_joint_transmission" params="joint reduction">
+  <xacro:macro name="position_joint_transmission" params="joint reduction">
     <transmission name="${joint}_transmission">
       <type>transmission_interface/SimpleTransmission</type>
@@ -13,4 +13,4 @@
       </actuator>
     </transmission>
-  </macro>
+  </xacro:macro>
 </robot>

File: sobit_mini_description/urdf/sensor/urg.urdf.xacro (robot description, xacro)
@@ -12,5 +12,5 @@
           <mesh filename="package://sobit_mini_description/meshes/UST-20LX.dae" />
         </geometry>
-        <material name="Black" />
+        <material name="black" />
       </visual>
       <inertial>

File: sobit_mini_description/urdf/urg_sup/urg_sup.urdf.xacro (robot description, xacro)
@@ -1,5 +1,4 @@
 <?xml version="1.0" encoding="UTF-8" ?>
-<robot name="urg_sup"
-  xmlns:xacro="http://ros.org/wiki/xacro">
+<robot name="urg_sup" xmlns:xacro="http://ros.org/wiki/xacro">
   <xacro:macro name="urg_sup" params="parent">
     <joint name="base_urg_sup_joint" type="fixed">
