Commit message: first commit for ROS2 (humble devel)

File: sobit_mini_description/robots/sobit_mini.urdf.xacro (robot description, xacro)
@@ -1,9 +1,11 @@
-<?xml version="1.0" ?>
-<robot name="sobit_mini" xmlns:controller="http://playerstage.sourceforge.net/gazebo/xmlschema/#controller" xmlns:interface="http://playerstage.sourceforge.net/gazebo/xmlschema/#interface" xmlns:sensor="http://playerstage.sourceforge.net/gazebo/xmlschema/#sensor" xmlns:xacro="http://www.ros.org/wiki/xacro">
-  <xacro:arg name="visualize" default="false" />
-  <!-- common xacro -->
+<?xml version="1.0" encoding="UTF-8" ?>
+<!-- <robot name="sobit_mini" xmlns:controller="http://playerstage.sourceforge.net/gazebo/xmlschema/#controller" xmlns:interface="http://playerstage.sourceforge.net/gazebo/xmlschema/#interface" xmlns:sensor="http://playerstage.sourceforge.net/gazebo/xmlschema/#sensor" xmlns:xacro="http://www.ros.org/wiki/xacro"> -->
+<robot name="sobit_mini" xmlns:xacro="http://www.ros.org/wiki/xacro">
+  <!-- Add Common Xacro: transmissions, colors -->
   <xacro:include filename="$(find sobit_mini_description)/urdf/common.xacro" />
   <xacro:include filename="$(find sobit_mini_description)/urdf/materials.urdf.xacro" />
-  <!-- links and joints -->
+  <xacro:include filename="$(find sobit_mini_description)/urdf/transmission.urdf.xacro" />
+  <xacro:include filename="$(find sobit_mini_description)/urdf/controllers.urdf.xacro" />
+  <!-- Add URDF: links, joints -->
   <xacro:include filename="$(find sobit_mini_description)/urdf/base/base.urdf.xacro" />
   <xacro:include filename="$(find sobit_mini_description)/urdf/body/body.urdf.xacro" />
@@ -20,7 +22,15 @@
   <xacro:include filename="$(find urg_node)/urdf/hokuyo_ust.urdf.xacro" />
   <xacro:include filename="$(find realsense2_description)/urdf/_d435.urdf.xacro" />
+  <!-- Add URDF: gazebo -->
+  <xacro:include filename="$(find sobit_mini_description)/urdf/gazebo.urdf.xacro" />
+  <!-- Add variables -->
+  <xacro:arg name="enable_gz"                 default="False" />
+  <xacro:arg name="enable_gz_lidar"           default="True" />
+  <xacro:arg name="robot_name"                default="sobit_mini" />
+  <xacro:controllers name="joints_control" enable_gz="$(arg enable_gz)" robot_name="$(arg robot_name)" />
+  <!-- Connect the previous Links and Joints -->
   <xacro:base/>
   <xacro:stack_hexagons parent="base_link" />
-  <xacro:lidar prefix="lidar" parent="plate_bottom_link" visualize="$(arg visualize)" />
+  <xacro:lidar prefix="lidar" parent="plate_bottom_link" />
   <xacro:body prefix="body" parent="plate_middle_link"/>
   <xacro:left_arm prefix="l_arm" parent="body_front_pole_link"/>
@@ -28,12 +38,13 @@
   <xacro:left_hand prefix="l_hand" parent="l_arm_wrist_tilt_link"/>
   <xacro:right_hand prefix="r_hand" parent="r_arm_wrist_tilt_link"/>
-  <xacro:head prefix="head" parent="body_front_pole_link"/>
-  <xacro:realsense_d435 prefix="head_camera" parent="head_tilt_link" />
-  <xacro:mic prefix="mic" parent="head_tilt_link"/>
-  <gazebo>
-    <plugin name="gazebo_ros_control" filename="libgazebo_ros_control.so">
-      <robotSimType>gazebo_ros_control/DefaultRobotHWSim</robotSimType>
-      <legacyModeNS>true</legacyModeNS>
-    </plugin>
-  </gazebo>
+  <xacro:head prefix="head_camera" parent="body_front_pole_link"/>
+  <xacro:realsense_d435 prefix="head_camera" parent="head_camera_tilt_link" />
+  <xacro:mic prefix="mic" parent="head_camera_tilt_link"/>
+  <!-- Add Gazebo: plugins -->
+  <xacro:if value="${$(arg enable_gz)}">
+    <xacro:gazebo_sensors robot_name="$(arg robot_name)"
+      enable_gz_lidar="$(arg enable_gz_lidar)"
+      enable_gz_imu="$(arg enable_gz_imu)"
+    />
+  </xacro:if>
 </robot>

File: sobit_mini_description/urdf/base/base.urdf.xacro (robot description, xacro)
@@ -8,5 +8,5 @@
 <robot name="base" xmlns:xacro="http://ros.org/wiki/xacro">
   <xacro:include filename="$(find kobuki_description)/urdf/common_properties.urdf.xacro" />
-  <xacro:include filename="$(find kobuki_description)/urdf/kobuki_gazebo.urdf.xacro" />
+  <!-- <xacro:include filename="$(find kobuki_description)/urdf/kobuki_gazebo.urdf.xacro" /> -->
   <!-- Kobuki -->
   <xacro:macro name="base">

File: sobit_mini_description/urdf/body/body.transmission.xacro (robot description, xacro)
@@ -2,5 +2,5 @@
 <robot xmlns:xacro="http://ros.org/wiki/xacro">
   <xacro:macro name="body_transmission" params="prefix">
-    <position_joint_transmission joint="${prefix}_roll_joint" reduction="1" />
+    <xacro:position_joint_transmission joint="${prefix}_roll_joint" reduction="1" />
     <!--add transmission-->
     <transmission name="${prefix}_roll_trans">

File: sobit_mini_description/urdf/body/body.urdf.xacro (robot description, xacro)
@@ -1,5 +1,5 @@
 <?xml version="1.0" encoding="UTF-8" ?>
 <robot name="body" xmlns:xacro="http://ros.org/wiki/xacro">
-  <xacro:include filename="$(find sobit_mini_description)/urdf/body/body.transmission.xacro" />
+  <xacro:include filename="$(find sobit_mini_description)/urdf/body/body.transmission.xacro" />  <!-- XXXXXXXXXX -->
   <xacro:macro name="body" params="prefix parent">
     <joint name="${prefix}_small_gear_base_joint" type="fixed">
@@ -13,5 +13,5 @@
         <origin xyz="0.0 0.0 0.034" rpy="0.0 0.0 ${M_PI/2.0}" />
         <geometry>
-          <mesh filename="package://sobit_mini_description/meshes/body/sobit_mini_small_gear_motor.stl" />
+          <mesh filename="file://$(sobit_mini_description)/meshes/body/sobit_mini_small_gear_motor.stl" />
         </geometry>
         <material name="black" />
@@ -42,5 +42,5 @@
         <origin xyz="0.0 0.0 0.0" rpy="${M_PI/2.0} 0.0 ${M_PI/2.0}" />
         <geometry>
-          <mesh filename="package://sobit_mini_description/meshes/body/sobit_mini_small_gear.stl" />
+          <mesh filename="file://$(sobit_mini_description)/meshes/body/sobit_mini_small_gear.stl" />
         </geometry>
         <material name="black" />
@@ -70,5 +70,5 @@
         <origin xyz="0.0 0.0 0.0" rpy="0.0 0.0 0.0" />
         <geometry>
-          <mesh filename="package://sobit_mini_description/meshes/body/big_gear_base.stl" />
+          <mesh filename="file://$(sobit_mini_description)/meshes/body/big_gear_base.stl" />
         </geometry>
         <material name="silver" />
@@ -100,5 +100,5 @@
         <origin xyz="0.0 0.0 0.0" rpy="0.0 0.0 0.0" />
         <geometry>
-          <mesh filename="package://sobit_mini_description/meshes/body/sobit_mini_big_gear.stl" />
+          <mesh filename="file://$(sobit_mini_description)/meshes/body/sobit_mini_big_gear.stl" />
         </geometry>
         <material name="black" />
@@ -135,5 +135,5 @@
         <origin xyz="0.0 0.0 0.0" rpy="0 0 ${M_PI/2.0}" />
         <geometry>
-          <mesh filename="package://sobit_mini_description/meshes/body/sobit_mini_center_back.stl" />
+          <mesh filename="file://$(sobit_mini_description)/meshes/body/sobit_mini_center_back.stl" />
         </geometry>
         <material name="black" />
@@ -163,5 +163,5 @@
         <origin xyz="0.0 0.0 0.0" rpy="0.0 0.0 ${M_PI/2.0}" />
         <geometry>
-          <mesh filename="package://sobit_mini_description/meshes/body/spine.stl" />
+          <mesh filename="file://$(sobit_mini_description)/meshes/body/spine.stl" />
         </geometry>
         <material name="black" />
@@ -191,5 +191,5 @@
         <origin xyz="0.0 0.0 0.459" rpy="0.0 0.0 ${M_PI/2.0}" />
         <geometry>
-          <mesh filename="package://sobit_mini_description/meshes/body/sobit_mini_body_cover.dae" />
+          <mesh filename="file://$(sobit_mini_description)/meshes/body/sobit_mini_body_cover.dae" />
         </geometry>
       </visual>
@@ -204,5 +204,5 @@
     <!--plug-in to distribute joint condition data-->
     <gazebo>
-      <plugin name="joint_state_publisher" filename="libgazebo_ros_joint_state_publisher.so">
+      <plugin name="joint_state_publisher" filename="libgazebo_ros_joint_state_publisher.so">  <!-- XXXXXXXXXX -->
         <jointName>${prefix}_roll_joint</jointName>
       </plugin>
@@ -211,5 +211,5 @@
     <xacro:macro name="mimic_joint_plugin" params="name_prefix parent_joint mimic_joint has_pid:=false multiplier:=1.0 offset:=0 sensitiveness:=0.0 max_effort:=1.0 robot_namespace:=''">
       <gazebo>
-        <plugin name="${name_prefix}mimic_joint_plugin" filename="libroboticsgroup_upatras_gazebo_mimic_joint_plugin.so">
+        <plugin name="${name_prefix}mimic_joint_plugin" filename="libroboticsgroup_upatras_gazebo_mimic_joint_plugin.so">  <!-- XXXXXXXXXX -->
           <joint>${parent_joint}</joint>
           <mimicJoint>${mimic_joint}</mimicJoint>

File: sobit_mini_description/urdf/common.xacro (robot description, xacro)
@@ -6,11 +6,23 @@
       <type>transmission_interface/SimpleTransmission</type>
       <joint name="${joint}">
-        <hardwareInterface>PositionJointInterface</hardwareInterface>
+        <hardwareInterface>hardware_interface/PositionJointInterface</hardwareInterface>
       </joint>
       <actuator name="${joint}_actuator">
-        <hardwareInterface>PositionJointInterface</hardwareInterface>
+        <hardwareInterface>hardware_interface/PositionJointInterface</hardwareInterface>
         <mechanicalReduction>${reduction}</mechanicalReduction>
       </actuator>
     </transmission>
   </xacro:macro>
+  <xacro:macro name="effort_joint_transmission" params="joint reduction">
+    <transmission name="${joint}_transmission">
+      <type>transmission_interface/SimpleTransmission</type>
+      <joint name="${joint}">
+        <hardwareInterface>hardware_interface/EffortJointInterface</hardwareInterface>
+      </joint>
+      <actuator name="${joint}_actuator">
+        <hardwareInterface>hardware_interface/EffortJointInterface</hardwareInterface>
+        <mechanicalReduction>1</mechanicalReduction>
+      </actuator>
+    </transmission>
+  </xacro:macro>
 </robot>

File: sobit_mini_description/urdf/head/head.transmission.xacro (robot description, xacro)
@@ -2,34 +2,30 @@
 <robot xmlns:xacro="http://ros.org/wiki/xacro">
   <xacro:macro name="head_transmission" params="prefix">
-    <position_joint_transmission joint="${prefix}_pan_joint" reduction="1" />
-    <position_joint_transmission joint="${prefix}_tilt_joint" reduction="1" />
-    <!--add transmission-->
-    <transmission name="${prefix}_pan_trans">
+    <xacro:position_joint_transmission joint="${prefix}_camera_pan_joint" reduction="1" />
+    <xacro:position_joint_transmission joint="${prefix}_camera_tilt_joint" reduction="1" />
+    <!--add transmission--> <!-- XXXXXXXXXX -->
+    <!-- <transmission name="${prefix}_camera_pan_trans">
       <provideFeedback>true</provideFeedback>
       <implicitSpringDamper>0</implicitSpringDamper>
       <type>transmission_interface/SimpleTransmission</type>
-      <!--joint designation-->
-      <joint name="${prefix}_pan_joint">
+      <joint name="${prefix}_camera_pan_joint">
         <hardwareInterface>hardware_interface/PositionJointInterface</hardwareInterface>
       </joint>
-      <!--actuator definition-->
-      <actuator name="${prefix}_pan_motor">
+      <actuator name="${prefix}_camera_pan_motor">
         <hardwareInterface>hardware_interface/PositionJointInterface</hardwareInterface>
         <mechanicalReduction>1</mechanicalReduction>
       </actuator>
     </transmission>
-    <transmission name="${prefix}_tilt_trans">
+    <transmission name="${prefix}_camera_tilt_trans">
       <provideFeedback>true</provideFeedback>
       <implicitSpringDamper>0</implicitSpringDamper>
       <type>transmission_interface/SimpleTransmission</type>
-      <!--joint designation-->
-      <joint name="${prefix}_tilt_joint">
+      <joint name="${prefix}_camera_tilt_joint">
         <hardwareInterface>hardware_interface/PositionJointInterface</hardwareInterface>
       </joint>
-      <!--actuator definition-->
-      <actuator name="${prefix}_tilt_motor">
+      <actuator name="${prefix}_camera_tilt_motor">
         <hardwareInterface>hardware_interface/PositionJointInterface</hardwareInterface>
       </actuator>
-    </transmission>
+    </transmission> -->
   </xacro:macro>
 </robot>

File: sobit_mini_description/urdf/head/head.urdf.xacro (robot description, xacro)
@@ -2,4 +2,5 @@
 <robot name="head" xmlns:xacro="http://ros.org/wiki/xacro">
   <xacro:include filename="$(find sobit_mini_description)/urdf/head/head.transmission.xacro" />
+  <!-- <xacro:include filename="$(find sobit_mini_description)/urdf/head/head.gazebo.xacro" /> -->
   <xacro:macro name="head" params="prefix parent">
     <joint name="${prefix}_pan_joint" type="revolute">
@@ -14,5 +15,5 @@
         <origin xyz="0.0 0.0 0.0" rpy="0.0 0.0 ${M_PI/2.0}" />
         <geometry>
-          <mesh filename="package://sobit_mini_description/meshes/head/HEAD_PAN_JOINT.stl" />
+          <mesh filename="file://$(find sobit_mini_description)/meshes/head/head_camera_pan_joint.stl" />
         </geometry>
         <material name="black" />
@@ -37,5 +38,5 @@
         <origin xyz="0.0 0.0 0.0" rpy="0.0 0.0 ${M_PI/2.0}" />
         <geometry>
-          <mesh filename="package://sobit_mini_description/meshes/head/HEAD_TILT_JOINT.dae" />
+          <mesh filename="file://$(find sobit_mini_description)/meshes/head/head_camera_tilt_joint.dae" />
         </geometry>
       </visual>
@@ -55,5 +56,5 @@
     </link>
     <!--plug-in to distribute joint condition data-->
-    <gazebo>
+    <!-- <gazebo>
       <plugin name="joint_state_publisher" filename="libgazebo_ros_joint_state_publisher.so">
         <jointName>${prefix}_pan_joint, ${prefix}_tilt_joint</jointName>
@@ -63,5 +64,5 @@
       <material>Gazebo/Black</material>
     </gazebo>
-    <xacro:head_transmission prefix="${prefix}"/>
+    <xacro:head_transmission prefix="${prefix}"/> -->
   </xacro:macro>
 </robot>

File: sobit_mini_description/urdf/left_arm/left_arm.transmission.xacro (robot description, xacro)
@@ -6,14 +6,12 @@
     <position_joint_transmission joint="${prefix}_elbow_tilt_joint" reduction="1" />
     <position_joint_transmission joint="${prefix}_wrist_tilt_joint" reduction="1" />
-    <!--add transmission-->
-    <transmission name="${prefix}_shoulder_roll_trans">
+    <!--add transmission-->   <!-- XXXXXXXXXX -->
+    <!-- <transmission name="${prefix}_shoulder_roll_trans">
       <provideFeedback>true</provideFeedback>
       <implicitSpringDamper>0</implicitSpringDamper>
       <type>transmission_interface/SimpleTransmission</type>
-      <!--joint designation-->
       <joint name="${prefix}_shoulder_roll_joint">
         <hardwareInterface>hardware_interface/PositionJointInterface</hardwareInterface>
       </joint>
-      <!--actuator definition-->
       <actuator name="${prefix}_shoulder_roll_motor">
         <hardwareInterface>hardware_interface/PositionJointInterface</hardwareInterface>
@@ -25,9 +23,7 @@
       <implicitSpringDamper>0</implicitSpringDamper>
       <type>transmission_interface/SimpleTransmission</type>
-      <!--joint designation-->
       <joint name="${prefix}_shoulder_pan_joint">
         <hardwareInterface>hardware_interface/PositionJointInterface</hardwareInterface>
       </joint>
-      <!--actuator definition-->
       <actuator name="${prefix}_shoulder_pan_motor">
         <hardwareInterface>hardware_interface/PositionJointInterface</hardwareInterface>
@@ -39,9 +35,7 @@
       <implicitSpringDamper>0</implicitSpringDamper>
       <type>transmission_interface/SimpleTransmission</type>
-      <!--joint designation-->
       <joint name="${prefix}_elbow_tilt_joint">
         <hardwareInterface>hardware_interface/PositionJointInterface</hardwareInterface>
       </joint>
-      <!--actuator definition-->
       <actuator name="${prefix}_elbow_tilt_motor">
         <hardwareInterface>hardware_interface/PositionJointInterface</hardwareInterface>
@@ -53,14 +47,12 @@
       <implicitSpringDamper>0</implicitSpringDamper>
       <type>transmission_interface/SimpleTransmission</type>
-      <!--joint designation-->
       <joint name="${prefix}_wrist_tilt_joint">
         <hardwareInterface>hardware_interface/PositionJointInterface</hardwareInterface>
       </joint>
-      <!--actuator definition-->
       <actuator name="${prefix}_wrist_tilt_motor">
         <hardwareInterface>hardware_interface/PositionJointInterface</hardwareInterface>
         <mechanicalReduction>1</mechanicalReduction>
       </actuator>
-    </transmission>
+    </transmission> -->
   </xacro:macro>
 </robot>

File: sobit_mini_description/urdf/left_arm/left_arm.urdf.xacro (robot description, xacro)
@@ -2,4 +2,5 @@
 <robot name="left_arm" xmlns:xacro="http://ros.org/wiki/xacro">
   <xacro:include filename="$(find sobit_mini_description)/urdf/left_arm/left_arm.transmission.xacro" />
+  <!-- <xacro:include filename="$(find sobit_mini_description)/urdf/left_arm/left_arm.gazebo.xacro" /> -->
   <xacro:macro name="left_arm" params="prefix parent">
     <joint name="${prefix}_shoulder_fixed_joint" type="fixed">
@@ -14,5 +15,5 @@
         <origin xyz="0.0 0.0 0.0" rpy="0.0 0.0 ${M_PI/2.0}" />
         <geometry>
-          <mesh filename="package://sobit_mini_description/meshes/L_arm/L_ARM_SHOULDER_ROLL_JOINT.stl" />
+          <mesh filename="file://$(find sobit_mini_description)/meshes/l_arm/l_arm_shoulder_roll_joint.stl" />
         </geometry>
         <material name="black" />
@@ -43,5 +44,5 @@
         <origin xyz="0.0 0.0 0.0" rpy="0.0 0.0 ${M_PI/2.0}" />
         <geometry>
-          <mesh filename="package://sobit_mini_description/meshes/L_arm/L_ARM_SHOULDER_FLEX_JOINT.stl" />
+          <mesh filename="file://$(find sobit_mini_description)/meshes/l_arm/l_arm_shoulder_flex_joint.stl" />
         </geometry>
         <material name="black" />
@@ -72,5 +73,5 @@
         <origin xyz="0.0 0.0 0.0" rpy="0.0 0.0 ${M_PI/2.0}" />
         <geometry>
-          <mesh filename="package://sobit_mini_description/meshes/L_arm/L_ARM_ELBOW_TILT_JOINT.stl" />
+          <mesh filename="file://$(find sobit_mini_description)/meshes/l_arm/l_arm_elbow_tilt_joint.stl" />
         </geometry>
         <material name="black" />
@@ -101,5 +102,5 @@
         <origin xyz="0.0 0.0 0.0" rpy="0.0 0.0 ${M_PI/2.0}" />
         <geometry>
-          <mesh filename="package://sobit_mini_description/meshes/L_arm/L_ARM_WRIST_TILT_JOINT.stl" />
+          <mesh filename="file://$(find sobit_mini_description)/meshes/l_arm/l_arm_wrist_tilt_joint.stl" />
         </geometry>
         <material name="black" />
@@ -130,5 +131,5 @@
         <origin xyz="0.0 0.0 0.0" rpy="0.0 ${-M_PI/2.0} ${M_PI}" />
         <geometry>
-          <mesh filename="package://sobit_mini_description/meshes/L_hand/L_hand_JOINT.stl"/>
+          <mesh filename="file://$(find sobit_mini_description)/meshes/l_hand/l_hand_joint.stl"/>
         </geometry>
         <material name="black" />
@@ -148,26 +149,4 @@
       </inertial>
     </link>
-    <!--plug-in to distribute joint condition data-->
-    <gazebo>
-      <plugin name="joint_state_publisher" filename="libgazebo_ros_joint_state_publisher.so">
-        <jointName>${prefix}_shoulder_roll_joint, ${prefix}_shoulder_pan_joint, ${prefix}_elbow_tilt_joint, ${prefix}_wrist_tilt_joint</jointName>
-      </plugin>
-    </gazebo>
-    <gazebo reference="${prefix}_shoulder_fixed_link">
-      <material>Gazebo/Black</material>
-    </gazebo>
-    <gazebo reference="${prefix}_shoulder_roll_link">
-      <material>Gazebo/Black</material>
-    </gazebo>
-    <gazebo reference="${prefix}_shoulder_pan_link">
-      <material>Gazebo/Black</material>
-    </gazebo>
-    <gazebo reference="${prefix}_elbow_tilt_link">
-      <material>Gazebo/Black</material>
-    </gazebo>
-    <gazebo reference="${prefix}_wrist_tilt_link">
-      <material>Gazebo/Black</material>
-    </gazebo>
-    <xacro:left_arm_transmission prefix="${prefix}"/>
   </xacro:macro>
 </robot>

File: sobit_mini_description/urdf/left_hand/left_hand.transmission.xacro (robot description, xacro)
@@ -2,20 +2,18 @@
 <robot xmlns:xacro="http://ros.org/wiki/xacro">
   <xacro:macro name="l_hand_transmission" params="prefix">
-    <position_joint_transmission joint="${prefix}_motor_joint" reduction="1" />
+    <position_joint_transmission joint="${prefix}_joint" reduction="1" />
     <!--add transmission-->
-    <transmission name="${prefix}_joint_trans">
+    <!-- <transmission name="${prefix}_joint_trans">
       <provideFeedback>true</provideFeedback>
       <implicitSpringDamper>0</implicitSpringDamper>
       <type>transmission_interface/SimpleTransmission</type>
-      <!--joint designation-->
       <joint name="${prefix}_joint">
         <hardwareInterface>hardware_interface/PositionJointInterface</hardwareInterface>
       </joint>
-      <!--actuator definition-->
       <actuator name="${prefix}_joint_motor">
         <hardwareInterface>hardware_interface/PositionJointInterface</hardwareInterface>
         <mechanicalReduction>1</mechanicalReduction>
       </actuator>
-    </transmission>
+    </transmission> -->
   </xacro:macro>
 </robot>

File: sobit_mini_description/urdf/left_hand/left_hand.urdf.xacro (robot description, xacro)
@@ -2,4 +2,5 @@
 <robot name="left_hand" xmlns:xacro="http://ros.org/wiki/xacro">
   <xacro:include filename="$(find sobit_mini_description)/urdf/left_hand/left_hand.transmission.xacro" />
+  <!-- <xacro:include filename="$(find sobit_mini_description)/urdf/left_hand/left_hand.gazebo.xacro" /> -->  <!-- XXXXXXXXX -->
   <xacro:macro name="left_hand" params="prefix parent">
     <joint name="${prefix}_joint" type="revolute">
@@ -14,5 +15,5 @@
         <origin xyz="0.0 0.0 0.0" rpy="${M_PI/2.0} 0.0 0.0" />
         <geometry>
-          <mesh filename="package://sobit_mini_description/meshes/L_hand/L_hand_finger_r_joint.stl" />
+          <mesh filename="file://$(find sobit_mini_description)/meshes/l_hand/l_hand_finger_r_joint.stl" />
         </geometry>
         <material name="black" />
@@ -44,5 +45,5 @@
         <origin xyz="0.0 0.0 0.0" rpy="${M_PI/2.0} 0.0 0.0" />
         <geometry>
-          <mesh filename="package://sobit_mini_description/meshes/L_hand/L_hand_finger_l_joint.stl" />
+          <mesh filename="file://$(find sobit_mini_description)/meshes/l_hand/Ll_hand_finger_l_joint.stl" />
         </geometry>
         <material name="black" />

File: sobit_mini_description/urdf/materials.urdf.xacro (robot description, xacro)
@@ -6,10 +6,4 @@
   <material name="black">
     <color rgba="0.1 0.1 0.1 1.0" />
-  </material>
-  <material name="white">
-    <color rgba="1.0 1.0 1.0 1.0" />
-  </material>
-  <material name="silver">
-    <color rgba="0.741 0.752 0.760 1.0" />
   </material>
   <material name="red">
@@ -22,9 +16,13 @@
     <color rgba="0.0 0.0 1.0 1.0" />
   </material>
-    <material name="dark_grey">
+  <material name="white">
+    <color rgba="1.0 1.0 1.0 1.0" />
+  </material>
+  <material name="grey">
+    <color rgba="0.3 0.3 0.3 1.0" />
+  </material>
+  <material name="dark_grey">
     <color rgba="0.175 0.175 0.175 1.0" />
   </material>
-    <material name="grey">
-    <color rgba="0.3 0.3 0.3 1.0" />
-  </material>
 </robot>
+<!-- XXXXXXXXXXx -->
