Commit message: first commit for ROS2 (humble devel)

File: sobit_mini_description/urdf/right_arm/right_arm.transmission.xacro (robot description, xacro)
@@ -7,13 +7,11 @@
     <position_joint_transmission joint="${prefix}_wrist_tilt_joint" reduction="1" />
     <!--add transmission-->
-    <transmission name="${prefix}_shoulder_roll_trans">
+    <!-- <transmission name="${prefix}_shoulder_roll_trans">
       <provideFeedback>true</provideFeedback>
       <implicitSpringDamper>0</implicitSpringDamper>
       <type>transmission_interface/SimpleTransmission</type>
-      <!--joint designation-->
       <joint name="${prefix}_shoulder_roll_joint">
         <hardwareInterface>hardware_interface/PositionJointInterface</hardwareInterface>
       </joint>
-      <!--actuator definition-->
       <actuator name="${prefix}_shoulder_roll_motor">
         <hardwareInterface>hardware_interface/PositionJointInterface</hardwareInterface>
@@ -25,9 +23,7 @@
       <implicitSpringDamper>0</implicitSpringDamper>
       <type>transmission_interface/SimpleTransmission</type>
-      <!--joint designation-->
       <joint name="${prefix}_shoulder_pan_joint">
         <hardwareInterface>hardware_interface/PositionJointInterface</hardwareInterface>
       </joint>
-      <!--actuator definition-->
       <actuator name="${prefix}_shoulder_pan_motor">
         <hardwareInterface>hardware_interface/PositionJointInterface</hardwareInterface>
@@ -39,9 +35,7 @@
       <implicitSpringDamper>0</implicitSpringDamper>
       <type>transmission_interface/SimpleTransmission</type>
-      <!--joint designation-->
       <joint name="${prefix}_elbow_tilt_joint">
         <hardwareInterface>hardware_interface/PositionJointInterface</hardwareInterface>
       </joint>
-      <!--actuator definition-->
       <actuator name="${prefix}_elbow_tilt_motor">
         <hardwareInterface>hardware_interface/PositionJointInterface</hardwareInterface>
@@ -53,14 +47,12 @@
       <implicitSpringDamper>0</implicitSpringDamper>
       <type>transmission_interface/SimpleTransmission</type>
-      <!--joint designation-->
       <joint name="${prefix}_wrist_tilt_joint">
         <hardwareInterface>hardware_interface/PositionJointInterface</hardwareInterface>
       </joint>
-      <!--actuator definition-->
       <actuator name="${prefix}_wrist_tilt_motor">
         <hardwareInterface>hardware_interface/PositionJointInterface</hardwareInterface>
         <mechanicalReduction>1</mechanicalReduction>
       </actuator>
-    </transmission>
+    </transmission> -->
   </xacro:macro>
 </robot>

File: sobit_mini_description/urdf/right_arm/right_arm.urdf.xacro (robot description, xacro)
@@ -14,5 +14,5 @@
         <origin xyz="0.0 0.0 0.0" rpy="0.0 0.0 ${M_PI/2.0}" />
         <geometry>
-          <mesh filename="package://sobit_mini_description/meshes/R_arm/R_ARM_SHOULDER_ROLL_JOINT.stl" />
+          <mesh filename="file://$(find sobit_mini_description)/meshes/r_arm/r_arm_shoulder_roll_joint.stl" />
         </geometry>
         <material name="black"/>
@@ -43,5 +43,5 @@
         <origin xyz="0.0 0.0 0.0" rpy="0.0 0.0 ${M_PI/2.0}" />
         <geometry>
-          <mesh filename="package://sobit_mini_description/meshes/R_arm/R_ARM_SHOULDER_FLEX_JOINT.stl" />
+          <mesh filename="file://$(find sobit_mini_description)/meshes/r_arm/r_arm_shoulder_flex_joint.stl" />
         </geometry>
         <material name="black"/>
@@ -72,5 +72,5 @@
         <origin xyz="0.0 0.0 0.0" rpy="${M_PI/2.0} 0.0 ${M_PI/2.0}" />
         <geometry>
-          <mesh filename="package://sobit_mini_description/meshes/R_arm/R_ARM_ELBOW_TILT_JOINT.stl" />
+          <mesh filename="file://$(find sobit_mini_description)/meshes/r_arm/r_arm_elbow_tilt_joint.stl" />
         </geometry>
         <material name="black"/>
@@ -101,5 +101,5 @@
         <origin xyz="0.0 0.0 0.0" rpy="0.0 0.0 ${M_PI/2.0}" />
         <geometry>
-          <mesh filename="package://sobit_mini_description/meshes/R_arm/R_ARM_WRIST_TILT_JOINT.stl" />
+          <mesh filename="file://$(find sobit_mini_description)/meshes/r_arm/r_arm_wrist_tilt_joint.stl" />
         </geometry>
       <material name="black"/>
@@ -130,5 +130,5 @@
         <origin xyz="0.0 0.0 0.0" rpy="0.0 ${M_PI/2.0} 0.0" />
         <geometry>
-          <mesh filename="package://sobit_mini_description/meshes/R_hand/R_hand_JOINT.stl"/>
+          <mesh filename="file://$(find sobit_mini_description)/meshes/r_hand/r_hand_joint.stl"/>
         </geometry>
         <material name="black" />
@@ -148,26 +148,4 @@
       </inertial>
     </link>
-    <!--plug-in to distribute joint condition data-->
-    <gazebo>
-      <plugin name="joint_state_publisher" filename="libgazebo_ros_joint_state_publisher.so">
-        <jointName>${prefix}_shoulder_roll_joint, ${prefix}_shoulder_pan_joint, ${prefix}_elbow_tilt_joint, ${prefix}_wrist_tilt_joint</jointName>
-      </plugin>
-    </gazebo>
-    <gazebo reference="${prefix}_shoulder_fixed_link">
-      <material>Gazebo/Black</material>
-    </gazebo>
-    <gazebo reference="${prefix}_shoulder_roll_link">
-      <material>Gazebo/Black</material>
-    </gazebo>
-    <gazebo reference="${prefix}_shoulder_pan_link">
-      <material>Gazebo/Black</material>
-    </gazebo>
-    <gazebo reference="${prefix}_elbow_tilt_link">
-      <material>Gazebo/Black</material>
-    </gazebo>
-    <gazebo reference="${prefix}_wrist_tilt_link">
-      <material>Gazebo/Black</material>
-    </gazebo>
-    <xacro:right_arm_transmission prefix="${prefix}"/>
   </xacro:macro>
 </robot>

File: sobit_mini_description/urdf/right_hand/right_hand.transmission.xacro (robot description, xacro)
@@ -2,20 +2,18 @@
 <robot xmlns:xacro="http://ros.org/wiki/xacro">
   <xacro:macro name="r_hand_transmission" params="prefix">
-    <position_joint_transmission joint="${prefix}_motor_joint" reduction="1" />
-    <transmission name="${prefix}_joint_trans">
+    <position_joint_transmission joint="${prefix}_joint" reduction="1" />
+    <!--add transmission-->
+    <!-- <transmission name="${prefix}_joint_trans">
       <provideFeedback>true</provideFeedback>
       <implicitSpringDamper>0</implicitSpringDamper>
       <type>transmission_interface/SimpleTransmission</type>
-      <!--joint designation-->
       <joint name="${prefix}_joint">
-        <!-- <hardwareInterface>PositionJointInterface</hardwareInterface> -->
         <hardwareInterface>hardware_interface/PositionJointInterface</hardwareInterface>
       </joint>
-      <!--actuator definition-->
       <actuator name="${prefix}_joint_motor">
         <hardwareInterface>hardware_interface/PositionJointInterface</hardwareInterface>
         <mechanicalReduction>1</mechanicalReduction>
       </actuator>
-    </transmission>
+    </transmission> -->
   </xacro:macro>
 </robot>

File: sobit_mini_description/urdf/right_hand/right_hand.urdf.xacro (robot description, xacro)
@@ -2,4 +2,5 @@
 <robot name="right_hand" xmlns:xacro="http://ros.org/wiki/xacro">
   <xacro:include filename="$(find sobit_mini_description)/urdf/right_hand/right_hand.transmission.xacro" />
+  <!-- <xacro:include filename="$(find sobit_mini_description)/urdf/right_hand/right_hand.gazebo.xacro" /> -->  <!-- XXXXXXXXX -->
   <xacro:macro name="right_hand" params="prefix parent">
     <joint name="${prefix}_joint" type="revolute">
@@ -14,5 +15,5 @@
         <origin xyz="0.0 0.0 0.0" rpy="${M_PI/2.0} 0.0 0.0" />
         <geometry>
-          <mesh filename="package://sobit_mini_description/meshes/R_hand/R_hand_finger_l_joint.stl" />
+          <mesh filename="file://$(find sobit_mini_description)/meshes/r_hand/r_hand_finger_l_joint.stl" />
         </geometry>
         <material name="black" />
@@ -44,5 +45,5 @@
         <origin xyz="0.0 0.0 0.0" rpy="${M_PI/2.0} 0.0 0.0" />
         <geometry>
-          <mesh filename="package://sobit_mini_description/meshes/R_hand/R_hand_finger_r_joint.stl" />
+          <mesh filename="file://$(find sobit_mini_description)/meshes/r_hand/r_hand_finger_r_joint.stl" />
         </geometry>
         <material name="black" />

File: sobit_mini_description/urdf/sensor/lidar.urdf.xacro (robot description, xacro)
@@ -1,7 +1,7 @@
 <?xml version="1.0" encoding="UTF-8" ?>
 <robot name="lidar" xmlns:xacro="http://ros.org/wiki/xacro">
-  <xacro:macro name="lidar" params="prefix parent visualize">
+  <xacro:macro name="lidar" params="prefix parent">
     <joint name="${prefix}_base_joint" type="fixed">
-      <origin xyz="0.194084 0.0 0.0085" rpy="0 0 0" />
+      <origin xyz="0.08525 0.0 0.008" rpy="0.0 0.0 0.0" />
       <parent link="${parent}" />
       <child link="${prefix}_base_link" />
@@ -9,27 +9,48 @@
     <link name="${prefix}_base_link">
       <visual>
-        <origin xyz="0.0 0.0 0.0" rpy="0.0 0.0 ${3.0*M_PI/2.0}"/>
+        <!-- <origin xyz="0.0 0.0 0.0" rpy="0.0 0.0 ${3.0*M_PI/2.0}"/> -->
+        <origin xyz="0.0 0.0 ${M_PI}" rpy="0.0 0.0 0.0"/>
         <geometry>
-          <mesh filename="package://sobit_mini_description/meshes/sobit_mini_urg_sup.dae"/>
+          <mesh filename="file://$(find sobit_mini_description)/meshes/sobit_mini_urg_sup.dae" scale="0.001 0.001 0.001" />
         </geometry>
       </visual>
       <collision>
-        <origin xyz="0.0 0.0 0.0" rpy="0.0 0.0 ${3.0*M_PI/2.0}" />
+        <!-- <origin xyz="0.0 0.0 0.0" rpy="0.0 0.0 ${3.0*M_PI/2.0}" /> -->
+        <origin xyz="0.0 0.0 ${M_PI}" rpy="0.0 0.0 0.0" />
         <geometry>
-          <mesh filename="package://sobit_mini_description/meshes/sobit_mini_urg_sup.dae"/>
+          <mesh filename="file://$(find sobit_mini_description)/meshes/sobit_mini_urg_sup.dae" scale="0.001 0.001 0.001" />
         </geometry>
       </collision>
       <inertial>
-        <origin xyz="0.0 0.0 0.0" rpy="0.0 0.0 ${3.0*M_PI/2.0}" />
-        <mass value="0.000001" />
-        <inertia ixx="0.0001" ixy="0.0" ixz="0.0" iyy="0.0001" iyz="0.0" izz="0.0001" />
+        <!-- <origin xyz="0.0 0.0 0.0" rpy="0.0 0.0 ${3.0*M_PI/2.0}" /> -->
+        <origin xyz="-0.05675 0.0 -0.0275" rpy="0.0 0.0 0.0" />
+        <mass value="0.35" />
+        <!-- <inertia ixx="0.0001" ixy="0.0" ixz="0.0" iyy="0.0001" iyz="0.0" izz="0.0001" /> -->
+        <inertia ixx="${1/12*0.87*(0.055**2+0.05**2)}"  ixy="0.0" ixz="0.0"
+                 iyy="${1/12*0.87*(0.1575**2+0.055**2)}"  iyz="0.0"
+                 izz="${1/12*0.87*(0.1575**2+0.05**2)}" />
       </inertial>
     </link>
-    <xacro:hokuyo_ust_mount prefix="${prefix}" parent="${prefix}_base_link" topic="scan" min_angle="-1.57" max_angle="1.57" visualize="${visualize}" >
+    <joint name="${prefix}_sim_joint" type="fixed">
+      <parent link="${prefix}_base_link" />
+      <child link="sim_laser_frame" />
+      <origin xyz="0.3 0 0.0" rpy="0 0 0" />
+    </joint>
+    <link name="sim_laser_frame">
+      <inertial>
+        <origin xyz="0.3 0 0" rpy="0 0 0" />
+        <mass value="0.2" />
+        <inertia ixx="0.001" ixy="0" ixz="0"
+                 iyy="0.001" iyz="0"
+                 izz="0.001" />
+      </inertial>
+    </link>
+    <!-- <xacro:hokuyo_ust_mount prefix="${prefix}" parent="${prefix}_base_link" topic="scan" min_angle="-1.57" max_angle="1.57" visualize="${visualize}" > -->
+    <xacro:hokuyo_ust_mount prefix="${prefix}" parent="${prefix}_base_link" topic="scan" >
       <origin xyz="0.0 0.0 0.0" rpy="0.0 0.0 0.0" />
     </xacro:hokuyo_ust_mount>
-    <gazebo reference="${prefix}_base_link">
+    <!-- <gazebo reference="${prefix}_base_link">
       <material>Gazebo/Black</material>
-    </gazebo>
+    </gazebo> -->
   </xacro:macro>
 </robot>

File: sobit_mini_description/urdf/sensor/mic.urdf.xacro (robot description, xacro)
@@ -11,5 +11,5 @@
         <origin xyz="0.0 0.0 0.0" rpy="0.0 0.0 ${M_PI/2.0}" />
         <geometry>
-          <mesh filename="package://sobit_mini_description/meshes/sensor/mic.stl"/>
+          <mesh filename="file://$(find sobit_mini_description)/meshes/sensor/mic.stl" scale="0.001 0.001 0.001" />
         </geometry>
         <material name="black" />
@@ -18,19 +18,24 @@
         <origin xyz="0.0 0.0 0.0" rpy="0.0 0.0 ${M_PI/2.0}" />
         <geometry>
-          <mesh filename="package://sobit_mini_description/meshes/sensor/mic.stl" />
+          <mesh filename="file://$(find sobit_mini_description)/meshes/sensor/mic.stl" scale="0.001 0.001 0.001" />
         </geometry>
         <material name="black" />
       </collision>
       <inertial>
-        <origin xyz="0.0 0.0 0.0" rpy="0.0 0.0 ${M_PI/2.0}" />
-        <mass value="0.09507172" />
-        <inertia ixx="${1/12*0.09507172*(0.078**2 + 0.157**2)}" ixy="0.0" ixz="0.0"
+        <!-- <origin xyz="0.0 0.0 0.0" rpy="0.0 0.0 ${M_PI/2.0}" /> -->
+        <origin xyz="0.0 0.02827923 -0.04872082" rpy="${M_PI} 0.0 ${M_PI/2}" />
+        <!-- <mass value="0.09507172" /> -->
+        <mass value="0.47" />
+        <!-- <inertia ixx="${1/12*0.09507172*(0.078**2 + 0.157**2)}" ixy="0.0" ixz="0.0"
                  iyy="${1/12*0.09507172*(0.026**2 + 0.078**2)}" iyz="0.0"
-                 izz="${1/12*0.09507172*(0.026**2 + 0.157**2)}" />
+                 izz="${1/12*0.09507172*(0.026**2 + 0.157**2)}" /> -->
+        <inertia ixx="${1/12*0.87*(0.09744164**2+0.18154208**2)}"  ixy="0.0" ixz="0.0"
+                 iyy="${1/12*0.87*(0.02999522**2+0.09744164**2)}"  iyz="0.0"
+                 izz="${1/12*0.87*(0.02999522**2+0.18154208**2)}" />
       </inertial>
     </link>
-    <gazebo reference="${prefix}_base_link">
+    <!-- <gazebo reference="${prefix}_base_link">
       <material>Gazebo/Black</material>
-    </gazebo>
+    </gazebo> -->
   </xacro:macro>
 </robot>

File: sobit_mini_description/urdf/stacks/stacks.urdf.xacro (robot description, xacro)
@@ -4,5 +4,5 @@
  -->
 <robot name="stack_hexagons" xmlns:xacro="http://ros.org/wiki/xacro">
-  <xacro:include filename="$(find turtlebot_description)/urdf/common_properties.urdf.xacro" />
+  <xacro:include filename="$(find turtlebot2_description)/urdf/common_properties.urdf.xacro" />
   <!-- Xacro properties -->
   <xacro:property name="M_SCALE" value="0.001" />
@@ -19,5 +19,5 @@
         <origin xyz="0 0 0" rpy="0 0 0" />
         <geometry>
-          <mesh filename="package://sobit_mini_description/meshes/body/pole_bottom_39mm.stl" scale="${M_SCALE} ${M_SCALE} ${M_SCALE}" />
+          <mesh filename="file://$(find sobit_mini_description)/meshes/body/pole_bottom_39mm.stl" scale="${M_SCALE} ${M_SCALE} ${M_SCALE}" />
         </geometry>
         <material name="grey" />
@@ -48,5 +48,5 @@
         <origin xyz="0 0 0" rpy="0 ${M_PI} 0" />
         <geometry>
-          <mesh filename="package://sobit_mini_description/meshes/body/pole_middle_134mm.stl" scale="${M_SCALE} ${M_SCALE} ${M_SCALE}" />
+          <mesh filename="file://$(find sobit_mini_description)/meshes/body/pole_middle_134mm.stl" scale="${M_SCALE} ${M_SCALE} ${M_SCALE}" />
         </geometry>
         <material name="grey" />
@@ -77,5 +77,5 @@
         <origin xyz=" 0 0 0" rpy="0 0 0" />
         <geometry>
-          <mesh filename="package://sobit_mini_description/meshes/body/pole_top_134mm.stl" scale="${M_SCALE} ${M_SCALE} ${M_SCALE}" />
+          <mesh filename="file://$(find sobit_mini_description)/meshes/body/pole_top_134mm.stl" scale="${M_SCALE} ${M_SCALE} ${M_SCALE}" />
         </geometry>
         <material name="grey" />
@@ -106,5 +106,5 @@
         <origin xyz="0 0 0.0" rpy="0 0 0" />
         <geometry>
-          <mesh filename="package://turtlebot_description/meshes/sensors/sensor_pole.dae" />
+          <mesh filename="package://turtlebot2_description/meshes/sensors/sensor_pole.dae" />
         </geometry>
       </visual>
@@ -145,5 +145,5 @@
         <origin xyz="0 0 0" rpy="0 0 0" />
         <geometry>
-          <mesh filename="package://turtlebot_description/meshes/stacks/hexagons/plate_bottom.dae" />
+          <mesh filename="package://turtlebot2_description/meshes/stacks/hexagons/plate_bottom.dae" />
         </geometry>
       </visual>
@@ -179,5 +179,5 @@
         <origin xyz="0 0.0 0" rpy="0 0 0" />
         <geometry>
-          <mesh filename="package://turtlebot_description/meshes/stacks/hexagons/plate_top.dae" />
+          <mesh filename="package://turtlebot2_description/meshes/stacks/hexagons/plate_top.dae" />
         </geometry>
       </visual>
