Commit message: [FIX]

File: sobit_mini_description/robots/sobit_mini.urdf.xacro (robot description, xacro)
@@ -1,11 +1,8 @@
 <?xml version="1.0" encoding="UTF-8" ?>
-<!-- <robot name="sobit_mini" xmlns:controller="http://playerstage.sourceforge.net/gazebo/xmlschema/#controller" xmlns:interface="http://playerstage.sourceforge.net/gazebo/xmlschema/#interface" xmlns:sensor="http://playerstage.sourceforge.net/gazebo/xmlschema/#sensor" xmlns:xacro="http://www.ros.org/wiki/xacro"> -->
 <robot name="sobit_mini" xmlns:xacro="http://www.ros.org/wiki/xacro">
-  <!-- Add Common Xacro: transmissions, colors -->
   <xacro:include filename="$(find sobit_mini_description)/urdf/common.xacro" />
   <xacro:include filename="$(find sobit_mini_description)/urdf/materials.urdf.xacro" />
   <xacro:include filename="$(find sobit_mini_description)/urdf/transmission.urdf.xacro" />
   <xacro:include filename="$(find sobit_mini_description)/urdf/controllers.urdf.xacro" />
-  <!-- Add URDF: links, joints -->
   <xacro:include filename="$(find sobit_mini_description)/urdf/base/base.urdf.xacro" />
   <xacro:include filename="$(find sobit_mini_description)/urdf/body/body.urdf.xacro" />
@@ -21,13 +18,11 @@
   <xacro:include filename="$(find sobit_mini_description)/urdf/sensor/realsense_d435.urdf.xacro" />
   <xacro:include filename="$(find urg_node)/urdf/hokuyo_ust.urdf.xacro" />
+  <xacro:include filename="$(find sobit_mini_description)/urdf/gazebo.urdf.xacro" />
   <xacro:include filename="$(find realsense2_description)/urdf/_d435.urdf.xacro" />
-  <!-- Add URDF: gazebo -->
-  <xacro:include filename="$(find sobit_mini_description)/urdf/gazebo.urdf.xacro" />
-  <!-- Add variables -->
-  <xacro:arg name="enable_gz"                 default="False" />
-  <xacro:arg name="enable_gz_lidar"           default="True" />
-  <xacro:arg name="robot_name"                default="sobit_mini" />
+  <xacro:arg name="enable_gz" default="False" />
+  <xacro:arg name="enable_gz_lidar" default="True" />
+  <xacro:arg name="enable_gz_imu" default="True" />
+  <xacro:arg name="robot_name" default="sobit_mini" />
   <xacro:controllers name="joints_control" enable_gz="$(arg enable_gz)" robot_name="$(arg robot_name)" />
-  <!-- Connect the previous Links and Joints -->
   <xacro:base/>
   <xacro:stack_hexagons parent="base_link" />
@@ -41,6 +36,5 @@
   <xacro:realsense_d435 prefix="head_camera" parent="head_camera_tilt_link" />
   <xacro:mic prefix="mic" parent="head_camera_tilt_link"/>
-  <!-- Add Gazebo: plugins -->
-  <xacro:if value="${$(arg enable_gz)}">
+  <xacro:if value="$(arg enable_gz)">
     <xacro:gazebo_sensors robot_name="$(arg robot_name)"
       enable_gz_lidar="$(arg enable_gz_lidar)"

File: sobit_mini_description/urdf/body/body.urdf.xacro (robot description, xacro)
@@ -1,5 +1,5 @@
 <?xml version="1.0" encoding="UTF-8" ?>
 <robot name="body" xmlns:xacro="http://ros.org/wiki/xacro">
-  <xacro:include filename="$(find sobit_mini_description)/urdf/body/body.transmission.xacro" />  <!-- XXXXXXXXXX -->
+  <xacro:include filename="$(find sobit_mini_description)/urdf/body/body.transmission.xacro" />
   <xacro:macro name="body" params="prefix parent">
     <joint name="${prefix}_small_gear_base_joint" type="fixed">
@@ -181,11 +181,11 @@
       </inertial>
     </link>
-    <joint name="${prefix}_sobit_mini_cover" type="fixed">
-      <parent link="${prefix}_roll_link" />
-      <child link="${prefix}_sobit_mini_cover" />
+    <joint name="${prefix}_cover_joint" type="fixed">
+      <parent link="${prefix}_roll_link" />
+      <child link="${prefix}_cover_link" />
       <origin xyz="0.0 0.0 0.0" rpy="0.0 0.0 0.0" />
       <axis xyz="0 0 1" />
     </joint>
-    <link name="${prefix}_sobit_mini_cover">
+    <link name="${prefix}_cover_link">
       <visual>
         <origin xyz="0.0 0.0 0.459" rpy="0.0 0.0 ${M_PI/2.0}" />
@@ -202,32 +202,4 @@
       </inertial>
     </link>
-    <!--plug-in to distribute joint condition data-->
-    <gazebo>
-      <plugin name="joint_state_publisher" filename="libgazebo_ros_joint_state_publisher.so">  <!-- XXXXXXXXXX -->
-        <jointName>${prefix}_roll_joint</jointName>
-      </plugin>
-    </gazebo>
-    <!-- the following is the template to mimic a joint -->
-    <xacro:macro name="mimic_joint_plugin" params="name_prefix parent_joint mimic_joint has_pid:=false multiplier:=1.0 offset:=0 sensitiveness:=0.0 max_effort:=1.0 robot_namespace:=''">
-      <gazebo>
-        <plugin name="${name_prefix}mimic_joint_plugin" filename="libroboticsgroup_upatras_gazebo_mimic_joint_plugin.so">  <!-- XXXXXXXXXX -->
-          <joint>${parent_joint}</joint>
-          <mimicJoint>${mimic_joint}</mimicJoint>
-          <xacro:if value="${has_pid}">                     <!-- if set to true, PID parameters from "/gazebo_ros_control/pid_gains/${mimic_joint}" are loaded -->
-            <hasPID />
-          </xacro:if>
-          <multiplier>${multiplier}</multiplier>
-          <offset>${offset}</offset>
-          <sensitiveness>${sensitiveness}</sensitiveness>   <!-- if absolute difference between setpoint and process value is below this threshold, do nothing; 0.0 = disable [rad] -->
-          <maxEffort>${max_effort}</maxEffort>              <!-- only taken into account if has_pid:=true [Nm] -->
-          <xacro:unless value="${robot_namespace == ''}">
-            <robotNamespace>${robot_namespace}</robotNamespace>
-          </xacro:unless>
-        </plugin>
-      </gazebo>
-    </xacro:macro>
-    <xacro:mimic_joint_plugin name_prefix="${prefix}_joint"
-    parent_joint="${prefix}_roll_joint" mimic_joint="${prefix}_big_gear_base_joint"
-    has_pid="false" multiplier="0.1896551724" max_effort="1.0" />
     <gazebo reference="${prefix}_small_gear_base_link">
       <material>Gazebo/Black</material>

File: sobit_mini_description/urdf/head/head.gazebo.xacro (robot description, xacro)
@@ -17,20 +17,4 @@
       <mu2>1.0</mu2>
     </gazebo>
-    <gazebo>
-    <plugin name="joint_state_publisher" filename="libgazebo_ros_joint_state_publisher.so">
-      <jointName>head_camera_pan_joint, head_camera_tilt_joint</jointName>
-      <updateRate>1000.0</updateRate>
-    </plugin>
-  </gazebo>
   </xacro:macro>
 </robot>
-    <!--plug-in to distribute joint condition data-->
-    <!-- <gazebo>
-      <plugin name="joint_state_publisher" filename="libgazebo_ros_joint_state_publisher.so">
-        <jointName>${prefix}_camera_pan_joint, ${prefix}_camera_tilt_joint</jointName>
-      </plugin>
-    </gazebo>
-    <gazebo reference="${prefix}_camera_pan_link">
-      <material>Gazebo/Black</material>
-    </gazebo>
-    <xacro:head_transmission prefix="${prefix}"/> -->

File: sobit_mini_description/urdf/left_arm/left_arm.gazebo.xacro (robot description, xacro)
@@ -18,9 +18,4 @@
       <material>Gazebo/Black</material>
     </gazebo>
-    <gazebo>
-      <plugin name="joint_state_publisher" filename="libgazebo_ros_joint_state_publisher.so">
-        <jointName>left_arm_shoulder_roll_joint, left_arm_shoulder_pan_joint, left_arm_elbow_tilt_joint, left_arm_wrist_tilt_joint</jointName>
-      </plugin>
-    </gazebo>
   </xacro:macro>
 </robot>

File: sobit_mini_description/urdf/left_hand/left_hand.gazebo.xacro (robot description, xacro)
@@ -7,49 +7,4 @@
       <mu2>1.0</mu2>
     </gazebo>
-    <gazebo>
-      <plugin name="joint_state_publisher" filename="libgazebo_ros_joint_state_publisher.so">
-        <jointName>left_hand_joint</jointName>
-        <updateRate>1000.0</updateRate>
-      </plugin>
-    </gazebo>
-  </xacro:macro>
-    <!-- the following is the template to mimic a joint -->
-    <xacro:macro name="mimic_joint" params="name_prefix parent_joint mimic_joint has_pid:=false multiplier:=1.0 offset:=0 sensitiveness:=0.0 max_effort:=1.0 robot_namespace:=''">
-      <gazebo>
-        <plugin name="${name_prefix}mimic_joint_plugin" filename="libroboticsgroup_upatras_gazebo_mimic_joint_plugin.so">
-          <joint>${parent_joint}</joint>
-          <mimicJoint>${mimic_joint}</mimicJoint>
-          <xacro:if value="${has_pid}">                     <!-- if set to true, PID parameters from "/gazebo_ros_control/pid_gains/${mimic_joint}" are loaded -->
-            <hasPID />
-          </xacro:if>
-          <multiplier>${multiplier}</multiplier>
-          <offset>${offset}</offset>
-          <sensitiveness>${sensitiveness}</sensitiveness>   <!-- if absolute difference between setpoint and process value is below this threshold, do nothing; 0.0 = disable [rad] -->
-          <maxEffort>${max_effort}</maxEffort>              <!-- only taken into account if has_pid:=true [Nm] -->
-          <xacro:unless value="${robot_namespace == ''}">
-            <robotNamespace>${robot_namespace}</robotNamespace>
-          </xacro:unless>
-        </plugin>
-      </gazebo>
-    </xacro:macro>
-  <xacro:macro name="gazebo">
-    <!-- Gazebo -->
-    <gazebo>
-      <plugin name="gazebo_ros_control" filename="libgazebo_ros_control.so">
-        <robotNamespace>/$(arg robot_namespace)</robotNamespace>
-        <robotSimType>gazebo_ros_control/DefaultRobotHWSim</robotSimType>
-        <legacyModeNS>true</legacyModeNS>
-      </plugin>
-    </gazebo>
-    <!-- <xacro:mimic_joint_plugin name_prefix="${prefix}_joint"
-    parent_joint="${prefix}_joint" mimic_joint="${prefix}_left_finger_joint"
-    has_pid="false" multiplier="1.0" max_effort="1.0" />
-    <gazebo reference="${prefix}_right_finger_link">
-      <material>Gazebo/Black</material>
-    </gazebo>
-    <gazebo reference="${prefix}_left_finger_link">
-      <material>Gazebo/Black</material>
-    </gazebo>
-    <xacro:l_hand_transmission prefix="${prefix}"/> -->
   </xacro:macro>
 </robot>

File: sobit_mini_description/urdf/left_hand/left_hand.urdf.xacro (robot description, xacro)
@@ -2,5 +2,4 @@
 <robot name="left_hand" xmlns:xacro="http://ros.org/wiki/xacro">
   <xacro:include filename="$(find sobit_mini_description)/urdf/left_hand/left_hand.transmission.xacro" />
-  <!-- <xacro:include filename="$(find sobit_mini_description)/urdf/left_hand/left_hand.gazebo.xacro" /> -->  <!-- XXXXXXXXX -->
   <xacro:macro name="left_hand" params="prefix parent">
     <joint name="${prefix}_joint" type="revolute">
@@ -63,33 +62,4 @@
       </inertial>
     </link>
-    <!--plug-in to distribute joint condition data-->
-    <gazebo>
-      <plugin name="joint_state_publisher" filename="libgazebo_ros_joint_state_publisher.so">
-        <robotNamespace>/</robotNamespace>
-        <jointName>${prefix}_joint</jointName>
-      </plugin>
-    </gazebo>
-    <!-- the following is the template to mimic a joint -->
-    <xacro:macro name="mimic_joint_plugin" params="name_prefix parent_joint mimic_joint has_pid:=false multiplier:=1.0 offset:=0 sensitiveness:=0.0 max_effort:=1.0 robot_namespace:=''">
-      <gazebo>
-        <plugin name="${name_prefix}mimic_joint_plugin" filename="libroboticsgroup_upatras_gazebo_mimic_joint_plugin.so">
-          <joint>${parent_joint}</joint>
-          <mimicJoint>${mimic_joint}</mimicJoint>
-          <xacro:if value="${has_pid}">                     <!-- if set to true, PID parameters from "/gazebo_ros_control/pid_gains/${mimic_joint}" are loaded -->
-            <hasPID />
-          </xacro:if>
-          <multiplier>${multiplier}</multiplier>
-          <offset>${offset}</offset>
-          <sensitiveness>${sensitiveness}</sensitiveness>   <!-- if absolute difference between setpoint and process value is below this threshold, do nothing; 0.0 = disable [rad] -->
-          <maxEffort>${max_effort}</maxEffort>              <!-- only taken into account if has_pid:=true [Nm] -->
-          <xacro:unless value="${robot_namespace == ''}">
-            <robotNamespace>${robot_namespace}</robotNamespace>
-          </xacro:unless>
-        </plugin>
-      </gazebo>
-    </xacro:macro>
-    <xacro:mimic_joint_plugin name_prefix="${prefix}_joint"
-    parent_joint="${prefix}_joint" mimic_joint="${prefix}_left_finger_joint"
-    has_pid="false" multiplier="1.0" max_effort="1.0" />
     <gazebo reference="${prefix}_right_finger_link">
       <material>Gazebo/Black</material>

File: sobit_mini_description/urdf/right_arm/right_arm.gazebo.xacro (robot description, xacro)
@@ -18,9 +18,4 @@
       <material>Gazebo/Black</material>
     </gazebo>
-    <gazebo>
-      <plugin name="joint_state_publisher" filename="libgazebo_ros_joint_state_publisher.so">
-        <jointName>right_arm_shoulder_roll_joint, right_arm_shoulder_pan_joint, right_arm_elbow_tilt_joint, right_arm_wrist_tilt_joint</jointName>
-      </plugin>
-    </gazebo>
   </xacro:macro>
 </robot>

File: sobit_mini_description/urdf/right_hand/right_hand.gazebo.xacro (robot description, xacro)
@@ -7,49 +7,4 @@
       <mu2>1.0</mu2>
     </gazebo>
-    <gazebo>
-      <plugin name="joint_state_publisher" filename="libgazebo_ros_joint_state_publisher.so">
-        <jointName>right_hand_joint</jointName>
-        <updateRate>1000.0</updateRate>
-      </plugin>
-    </gazebo>
-  </xacro:macro>
-    <!-- the following is the template to mimic a joint -->
-    <xacro:macro name="mimic_joint" params="name_prefix parent_joint mimic_joint has_pid:=false multiplier:=1.0 offset:=0 sensitiveness:=0.0 max_effort:=1.0 robot_namespace:=''">
-      <gazebo>
-        <plugin name="${name_prefix}mimic_joint_plugin" filename="libroboticsgroup_upatras_gazebo_mimic_joint_plugin.so">
-          <joint>${parent_joint}</joint>
-          <mimicJoint>${mimic_joint}</mimicJoint>
-          <xacro:if value="${has_pid}">                     <!-- if set to true, PID parameters from "/gazebo_ros_control/pid_gains/${mimic_joint}" are loaded -->
-            <hasPID />
-          </xacro:if>
-          <multiplier>${multiplier}</multiplier>
-          <offset>${offset}</offset>
-          <sensitiveness>${sensitiveness}</sensitiveness>   <!-- if absolute difference between setpoint and process value is below this threshold, do nothing; 0.0 = disable [rad] -->
-          <maxEffort>${max_effort}</maxEffort>              <!-- only taken into account if has_pid:=true [Nm] -->
-          <xacro:unless value="${robot_namespace == ''}">
-            <robotNamespace>${robot_namespace}</robotNamespace>
-          </xacro:unless>
-        </plugin>
-      </gazebo>
-    </xacro:macro>
-  <xacro:macro name="gazebo">
-    <!-- Gazebo -->
-    <gazebo>
-      <plugin name="gazebo_ros_control" filename="libgazebo_ros_control.so">
-        <robotNamespace>/$(arg robot_namespace)</robotNamespace>
-        <robotSimType>gazebo_ros_control/DefaultRobotHWSim</robotSimType>
-        <legacyModeNS>true</legacyModeNS>
-      </plugin>
-    </gazebo>
-    <!-- <xacro:mimic_joint_plugin name_prefix="${prefix}_joint"
-    parent_joint="${prefix}_joint" mimic_joint="${prefix}_left_finger_joint"
-    has_pid="false" multiplier="1.0" max_effort="1.0" />
-    <gazebo reference="${prefix}_right_finger_link">
-      <material>Gazebo/Black</material>
-    </gazebo>
-    <gazebo reference="${prefix}_left_finger_link">
-      <material>Gazebo/Black</material>
-    </gazebo>
-    <xacro:r_hand_transmission prefix="${prefix}"/> -->
   </xacro:macro>
 </robot>

File: sobit_mini_description/urdf/right_hand/right_hand.urdf.xacro (robot description, xacro)
@@ -2,5 +2,4 @@
 <robot name="right_hand" xmlns:xacro="http://ros.org/wiki/xacro">
   <xacro:include filename="$(find sobit_mini_description)/urdf/right_hand/right_hand.transmission.xacro" />
-  <!-- <xacro:include filename="$(find sobit_mini_description)/urdf/right_hand/right_hand.gazebo.xacro" /> -->  <!-- XXXXXXXXX -->
   <xacro:macro name="right_hand" params="prefix parent">
     <joint name="${prefix}_joint" type="revolute">
@@ -63,33 +62,4 @@
       </inertial>
     </link>
-    <!--plug-in to distribute joint condition data-->
-    <gazebo>
-      <plugin name="joint_state_publisher" filename="libgazebo_ros_joint_state_publisher.so">
-        <robotNamespace>/</robotNamespace>
-        <jointName>${prefix}_joint</jointName>
-      </plugin>
-    </gazebo>
-    <!-- the following is the template to mimic a joint -->
-    <xacro:macro name="mimic_joint_plugin" params="name_prefix parent_joint mimic_joint has_pid:=false multiplier:=1.0 offset:=0 sensitiveness:=0.0 max_effort:=1.0 robot_namespace:=''">
-      <gazebo>
-        <plugin name="${name_prefix}mimic_joint_plugin" filename="libroboticsgroup_upatras_gazebo_mimic_joint_plugin.so">
-          <joint>${parent_joint}</joint>
-          <mimicJoint>${mimic_joint}</mimicJoint>
-          <xacro:if value="${has_pid}">                     <!-- if set to true, PID parameters from "/gazebo_ros_control/pid_gains/${mimic_joint}" are loaded -->
-            <hasPID />
-          </xacro:if>
-          <multiplier>${multiplier}</multiplier>
-          <offset>${offset}</offset>
-          <sensitiveness>${sensitiveness}</sensitiveness>   <!-- if absolute difference between setpoint and process value is below this threshold, do nothing; 0.0 = disable [rad] -->
-          <maxEffort>${max_effort}</maxEffort>              <!-- only taken into account if has_pid:=true [Nm] -->
-          <xacro:unless value="${robot_namespace == ''}">
-            <robotNamespace>${robot_namespace}</robotNamespace>
-          </xacro:unless>
-        </plugin>
-      </gazebo>
-    </xacro:macro>
-    <xacro:mimic_joint_plugin name_prefix="${prefix}_joint"
-    parent_joint="${prefix}_joint" mimic_joint="${prefix}_right_finger_joint"
-    has_pid="false" multiplier="1.0" max_effort="1.0" />
     <gazebo reference="${prefix}_right_finger_link">
       <material>Gazebo/Black</material>
