Commit message: Fix gazebo mode of SOBIT MINI(URDF)

File: sobit_mini_description/robots/sobit_mini.urdf.xacro (robot description, xacro)
@@ -22,5 +22,4 @@
   <xacro:arg name="enable_gz" default="False" />
   <xacro:arg name="enable_gz_lidar" default="True" />
-  <xacro:arg name="enable_gz_imu" default="True" />
   <xacro:arg name="robot_name" default="sobit_mini" />
   <xacro:controllers name="joints_control" enable_gz="$(arg enable_gz)" robot_name="$(arg robot_name)" />
@@ -39,5 +38,4 @@
     <xacro:gazebo_sensors robot_name="$(arg robot_name)"
       enable_gz_lidar="$(arg enable_gz_lidar)"
-      enable_gz_imu="$(arg enable_gz_imu)"
     />
   </xacro:if>

File: sobit_mini_description/urdf/body/body.urdf.xacro (robot description, xacro)
@@ -115,5 +115,5 @@
         <inertia ixx="${1/12*0.37382712*(3*(0.118**2 + 0.104**2) + 0.033**2)}" ixy="0.0" ixz="0.0"
                  iyy="${1/12*0.37382712*(3*(0.118**2 + 0.104**2) + 0.033**2)}" iyz="0.0"
-                 izz="${1/2*(0.118**2 + 0.104**2)}" />
+                 izz="${1/2*0.37382712*(0.118**2 + 0.104**2)}" />
       </inertial>
     </link>
@@ -122,5 +122,5 @@
       <child link="${prefix}_big_gear_link" />
       <origin xyz="0.0 0.0 0.0" rpy="0.0 0.0 0.0" />
-      <axis xyz="0 0 1" />
+      <axis xyz="0 0 -1" />
     </joint>
     <link name="${prefix}_big_gear_link"/>

File: sobit_mini_description/urdf/controllers.urdf.xacro (robot description, xacro)
@@ -248,4 +248,15 @@
         <state_interface name="effort"/>
       </joint>
+      <xacro:if value="${$(arg enable_gz)}">
+        <joint name="body_big_gear_base_joint">
+          <param name="mimic">body_roll_joint</param>
+          <param name="multiplier">0.1896551724</param>
+          <state_interface name="position">
+            <param name="initial_value">0.0</param>
+          </state_interface>
+          <state_interface name="velocity"/>
+          <state_interface name="effort"/>
+        </joint>
+      </xacro:if>
     </ros2_control>
     <!-- Differential Drive -->

File: sobit_mini_description/urdf/gazebo.urdf.xacro (robot description, xacro)
@@ -2,13 +2,63 @@
 <!-- SOBIT MINI (Gazebo) -->
 <robot name="sobit_mini_gazebo" xmlns:xacro="http://ros.org/wiki/xacro">
-  <xacro:macro name="gazebo_sensors" params="robot_name enable_gz_front_cam_color:=True enable_gz_back_cam_color:=True enable_gz_head_cam_color:=True enable_gz_head_cam_depth:=True enable_gz_hand_cam_color:=True enable_gz_hand_cam_depth:=True enable_gz_lidar:=True enable_gz_imu:=True">
+  <xacro:macro name="gazebo_sensors" params="robot_name enable_gz_head_cam_color:=True enable_gz_head_cam_depth:=True enable_gz_lidar:=True">
+    <!-- Sensor - Head Camera (Color) -->
+    <xacro:if value="${enable_gz_head_cam_color}">
+      <gazebo reference="head_camera_link">
+        <sensor name="head_camera_color" type="camera">
+          <pose>0.05 0.0 0.0 0.0 0.0 0.0</pose>
+          <ignition_frame_id>${robot_name}/head_camera_link</ignition_frame_id>
+          <topic>${robot_name}/head_camera_base/color/image_raw</topic>
+          <always_on>1</always_on>
+          <visualize>true</visualize>
+          <update_rate>1</update_rate>
+          <camera name="head_camera_color">
+            <horizontal_fov>1.21126</horizontal_fov>
+            <image>
+              <width>640</width>
+              <height>480</height>
+              <format>RGB_INT8</format>
+            </image>
+            <clip>
+              <near>0.1</near>
+              <far>10</far>
+            </clip>
+          </camera>
+        </sensor>
+      </gazebo>
+    </xacro:if>
+    <!-- Sensor - Head Camera (Depth) -->
+    <xacro:if value="${enable_gz_head_cam_depth}">
+      <gazebo reference="head_camera_link">
+        <sensor name="head_camera_depth" type="depth">
+          <!-- <pose>0.0 0.0 ${0.0175/2} ${M_PI/2} -${M_PI/2} 0.0</pose> -->
+          <!-- <pose>0.0 0.0 -0.6 0.0 0.0 0.0</pose> -->
+          <pose>0.05 0.0 0.0 0.0 0.0 0.0</pose>
+          <ignition_frame_id>${robot_name}/head_camera_link</ignition_frame_id>
+          <topic>${robot_name}/head_camera_base/depth/image_raw</topic>
+          <always_on>1</always_on>
+          <visualize>true</visualize>
+          <update_rate>1</update_rate>
+          <camera name="head_camera_depth">
+            <horizontal_fov>1.48702</horizontal_fov>
+            <image>
+              <width>640</width>
+              <height>480</height>
+            </image>
+            <clip>
+              <near>0.1</near>
+              <far>10</far>
+            </clip>
+          </camera>
+        </sensor>
+      </gazebo>
+    </xacro:if>
     <!-- Sensor: LiDAR -->
     <xacro:if value="${enable_gz_lidar}">
-      <gazebo reference="sim_laser_frame">
+      <gazebo reference="lidar_laser">
         <sensor name="lidar" type="gpu_lidar">
           <pose>0 0 0 0 0 0</pose>
-          <ignition_frame_id>${robot_name}/sim_laser_frame</ignition_frame_id>
-          <!-- <gz_frame_id>${robot_name}/sim_laser_frame</gz_frame_id> -->
-          <topic>${robot_name}/lidar/scan</topic>
+          <ignition_frame_id>${robot_name}/lidar_laser</ignition_frame_id>
+          <topic>${robot_name}/scan</topic>
           <always_on>1</always_on>
           <visualize>true</visualize>
@@ -19,6 +69,6 @@
                 <samples>640</samples>
                 <resolution>1</resolution>
-                <min_angle>-2.4870942</min_angle>
-                <max_angle>2.4870942</max_angle>
+                <min_angle>-1.5708</min_angle>
+                <max_angle>1.5708</max_angle>
               </horizontal>
               <vertical>
@@ -38,19 +88,6 @@
       </gazebo>
     </xacro:if>
-    <!-- Publish Pose -->
-    <!-- <gazebo>
-      <plugin
-          filename="gz-sim-pose-publisher-system"
-          name="gz::sim::systems::PosePublisher">
-        <publish_link_pose>true</publish_link_pose>
-        <publish_collision_pose>false</publish_collision_pose>
-        <publish_visual_pose>false</publish_visual_pose>
-        <publish_sensor_pose>false</publish_sensor_pose>
-        <publish_nested_model_pose>true</publish_nested_model_pose>
-      </plugin>
-    </gazebo> -->
     <!-- Publish Joint States -->
     <gazebo>
-      <!-- <plugin filename="ignition-gazebo-joint-state-publisher-system" name="ignition::gazebo::systems::JointStatePublisher"> -->
       <plugin filename="gz-sim-joint-state-publisher-system" name="gz::sim::systems::JointStatePublisher">
         <topic>${robot_name}/joint_states</topic>

File: sobit_mini_description/urdf/sensor/lidar.urdf.xacro (robot description, xacro)
@@ -9,5 +9,4 @@
     <link name="${prefix}_base_link">
       <visual>
-        <!-- <origin xyz="0.0 0.0 0.0" rpy="0.0 0.0 ${3.0*M_PI/2.0}"/> -->
         <origin xyz="0.0 0.0 ${M_PI}" rpy="0.0 0.0 0.0"/>
         <geometry>
@@ -17,8 +16,7 @@
       </visual>
       <collision>
-        <!-- <origin xyz="0.0 0.0 0.0" rpy="0.0 0.0 ${3.0*M_PI/2.0}" /> -->
         <origin xyz="0.0 0.0 ${M_PI}" rpy="0.0 0.0 0.0" />
         <geometry>
-          <mesh filename="file://$(find sobit_mini_description)/meshes/sobit_mini_urg_sup.dae" scale="0.001 0.001 0.001" />
+          <box size="0.092 0.184 0.007"/>
         </geometry>
       </collision>
@@ -26,22 +24,7 @@
         <origin xyz="-0.05675 0.0 -0.0275" rpy="0.0 0.0 0.0" />
         <mass value="0.35" />
-        <!-- <inertia ixx="0.0001" ixy="0.0" ixz="0.0" iyy="0.0001" iyz="0.0" izz="0.0001" /> -->
         <inertia ixx="${1/12*0.87*(0.055**2+0.05**2)}"  ixy="0.0" ixz="0.0"
                  iyy="${1/12*0.87*(0.1575**2+0.055**2)}"  iyz="0.0"
                  izz="${1/12*0.87*(0.1575**2+0.05**2)}" />
-      </inertial>
-    </link>
-    <joint name="${prefix}_sim_joint" type="fixed">
-      <parent link="${prefix}_base_link" />
-      <child link="sim_laser_frame" />
-      <origin xyz="0.3 0 0.0" rpy="0 0 0" />
-    </joint>
-    <link name="sim_laser_frame">
-      <inertial>
-        <origin xyz="0.3 0 0" rpy="0 0 0" />
-        <mass value="0.2" />
-        <inertia ixx="0.001" ixy="0" ixz="0"
-                 iyy="0.001" iyz="0"
-                 izz="0.001" />
       </inertial>
     </link>

Commit message: Update jazzy version

File: sobit_mini_description/robots/sobit_mini.urdf.xacro (robot description, xacro)
@@ -24,4 +24,6 @@
   <xacro:arg name="enable_gz_head_cam_color" default="True" />
   <xacro:arg name="enable_gz_head_cam_depth" default="True" />
+  <!-- DXL Ports -->
+  <xacro:arg name="dxl_sm_port"  default="/dev/ttyUSB0" />
   <xacro:arg name="robot_name" default="sobit_mini" />
   <xacro:controllers name="joints_control" enable_gz="$(arg enable_gz)" robot_name="$(arg robot_name)" />

File: sobit_mini_description/urdf/controllers.urdf.xacro (robot description, xacro)
@@ -11,6 +11,7 @@
         </xacro:if>
         <xacro:unless value="${$(arg enable_gz)}">
+          <xacro:property name="dxl_sm_port" value="$(arg dxl_sm_port)"/>
           <plugin>dynamixel_hardware/DynamixelHardware</plugin>
-          <param name="port_name">/dev/ttyUSB0</param>
+          <param name="port_name">${dxl_sm_port}</param>
           <param name="baud_rate">1000000</param>
           <!-- <param name="use_dummy">true</param> -->
