Commit message: バグの修正

File: sobit_mini_description/urdf/sensor/xtion.urdf.xacro (robot description, xacro)
@@ -17,5 +17,5 @@
     <link name="camera_fixed_link" />
     <joint name="camera_rgb_joint" type="fixed">
-      <origin xyz="0.013 0.0220 0.022" rpy="0 -0.1221 0" />
+      <origin xyz="0.011 0.0220 0.022" rpy="0 -0.1221 0" />
       <parent link="camera_fixed_link" />
       <child link="rgb_link" />
