Commit message: update/urg_position

File: sobit_mini_description/urdf/sensor/urg.urdf.xacro (robot description, xacro)
@@ -3,5 +3,5 @@
   <xacro:macro name="urg" params="parent">
     <joint name="laser" type="fixed">
-      <origin xyz="0.205 0.0 0.01" rpy="0 0 0" />
+      <origin xyz="0.0 0.0 0.0" rpy="0 0 0" />
       <parent link="${parent}" />
       <child link="base_laser_link" />
