Commit message: urdf の修正

File: sobit_mini_description/urdf/stacks/stacks.urdf.xacro (robot description, xacro)
@@ -95,5 +95,5 @@
     <link name="pole_kinect_${number}_link">
       <visual>
-        <origin xyz="0 0 -0.01" rpy="0 0 0" />
+        <origin xyz="0 0 0.0025" rpy="0 0 0" />
         <geometry>
           <mesh filename="package://turtlebot_description/meshes/sensors/sensor_pole.dae" />
@@ -149,8 +149,8 @@
       </inertial>
     </link>
-    <stack_middle_pole parent="${parent}" number="0" x_loc="0.0381" y_loc="0.1505" z_loc="0.1735" />
-    <stack_middle_pole parent="${parent}" number="1" x_loc="0.0381" y_loc="-0.1505" z_loc="0.1735" />
-    <stack_middle_pole parent="${parent}" number="2" x_loc="-0.0381" y_loc="0.1505" z_loc="0.1735" />
-    <stack_middle_pole parent="${parent}" number="3" x_loc="-0.0381" y_loc="-0.1505" z_loc="0.1735" />
+    <stack_3d_sensor_pole parent="${parent}" number="0" x_loc="0.0381" y_loc="0.1505" z_loc="0.1735" />
+    <stack_3d_sensor_pole parent="${parent}" number="1" x_loc="0.0381" y_loc="-0.1505" z_loc="0.1735" />
+    <stack_3d_sensor_pole parent="${parent}" number="2" x_loc="-0.0381" y_loc="0.1505" z_loc="0.1735" />
+    <stack_3d_sensor_pole parent="${parent}" number="3" x_loc="-0.0381" y_loc="-0.1505" z_loc="0.1735" />
     <joint name="plate_middle_joint" type="fixed">
       <origin xyz="-0.01364 0.0 0.222" rpy="0 0 0" />
