Commit message: urdf完成

File: sobit_mini_description/urdf/left_arm/left_arm.urdf.xacro (robot description, xacro)
@@ -12,7 +12,7 @@
     <link name="${prefix}_shoulder_fixed_link">
       <visual>
-        <origin rpy="${M_PI/2.0} 0 ${M_PI}" xyz="0.0 0.081 0.007" />
+        <origin rpy="${M_PI/2.0} 0 ${M_PI}" xyz="0.0199 0.09019 -0.0089" />
         <geometry>
-          <mesh filename="package://sobit_mini_description/meshes/sobit_mini_shoulder1.dae" />
+          <mesh filename="package://sobit_mini_description/meshes/shoulder1.dae" />
         </geometry>
       </visual>
@@ -26,5 +26,5 @@
       <parent link="${prefix}_shoulder_fixed_link" />
       <child link="${prefix}_shoulder_roll_link" />
-      <origin rpy="0 0 0" xyz="0.0 0.11986 0.03941" />
+      <origin rpy="0 0 0" xyz="0.0 0.14146 0.03941" />
       <axis xyz="0 -1 0" />
       <limit effort="30" lower="${-M_PI/2.0}" upper="${M_PI/2.0}" velocity="${M_PI}" />
@@ -38,5 +38,5 @@
       </collision>
       <visual>
-        <origin rpy="0 ${M_PI/2.0} 0" xyz="0.0 0.0525 0.0" />
+        <origin rpy="0 ${M_PI/2.0} 0" xyz="0.0 0.0509 0.0" />
         <geometry>
           <mesh filename="package://sobit_mini_description/meshes/sobit_mini_shoulder2.dae" />
@@ -52,5 +52,5 @@
       <parent link="${prefix}_shoulder_roll_link" />
       <child link="${prefix}_shoulder_flex_link" />
-      <origin rpy="${M_PI/2.0} 0 0" xyz="0.0 0.0525 0.0" />
+      <origin rpy="0 0 0" xyz="0 0.0511 0.0" />
       <axis xyz="1 0 0" />
       <limit effort="30" lower="${-M_PI/2.0}" upper="${M_PI/2.0}" velocity="${M_PI/2.0}" />
@@ -64,7 +64,7 @@
       </collision>
       <visual>
-        <origin rpy="0 ${M_PI} ${M_PI/2.0}" xyz="0.018 0.017 -0.14803" />
+        <origin rpy="${-M_PI/2.0} ${-M_PI/2.0} 0" xyz="-0.0265 0.0702 -0.017" />
         <geometry>
-          <mesh filename="package://sobit_mini_description/meshes/sobit_mini_arm.dae" />
+          <mesh filename="package://sobit_mini_description/meshes/arm1_left.dae" />
         </geometry>
       </visual>
@@ -78,6 +78,6 @@
       <parent link="${prefix}_shoulder_flex_link" />
       <child link="${prefix}_wrist_flex_link" />
-      <origin rpy="0 0 0" xyz="0 0 -0.1892" />
-      <axis xyz="1 0 0" />
+      <origin rpy="0 0 0" xyz="-0.0005 0.1105 0" />
+      <axis xyz="0 0 1" />
       <limit effort="30" lower="${-M_PI/2.0}" upper="${M_PI/2.0}" velocity="${M_PI/2.0}" />
     </joint>
@@ -90,7 +90,7 @@
       </collision>
       <visual>
-        <origin rpy="${M_PI/2.0} 0 ${M_PI/2.0}" xyz="0.021 0.01 -0.029" />
+        <origin rpy="${-M_PI/2.0} ${-M_PI/2.0} 0" xyz="-0.0260  -0.0405 -0.0172" />
         <geometry>
-          <mesh filename="package://sobit_mini_description/meshes/sobit_mini_wrist.dae" />
+          <mesh filename="package://sobit_mini_description/meshes/arm2_left.dae" />
         </geometry>
       </visual>

File: sobit_mini_description/urdf/left_hand/left_hand.urdf.xacro (robot description, xacro)
@@ -3,7 +3,16 @@
   <xacro:include filename="$(find sobit_mini_description)/urdf/left_hand/left_hand.transmission.xacro" />
   <xacro:macro name="left_hand" params="prefix parent">
+    <joint name="${prefix}_motor_dummy_joint" type="fixed">
+      <parent link="${parent}" />
+      <child link="${prefix}_motor_dummy_link" />
+      <origin rpy="${M_PI/2.0} ${-M_PI/2.0} 0" xyz="0 0.15 0" />
+      <axis xyz="0 1 0" />
+      <limit lower="0.0" upper="${M_PI/2.0}" effort="1" velocity="1" />
+    </joint>
+    <link name="${prefix}_motor_dummy_link" />
     <joint name="${prefix}_motor_joint" type="revolute">
-      <parent link="${parent}" />
+      <parent link="${prefix}_motor_dummy_link" />
       <child link="${prefix}_motor_link" />
+      <origin rpy="0 0 0" xyz="0 0 0" />
       <axis xyz="0 1 0" />
       <limit lower="0.0" upper="${M_PI/2.0}" effort="1" velocity="1" />
@@ -11,7 +20,7 @@
     <link name="${prefix}_motor_link" />
     <joint name="${prefix}_left_finger_joint" type="revolute">
-      <parent link="${parent}" />
+      <parent link="${prefix}_motor_dummy_link" />
       <child link="${prefix}_left_finger_link" />
-      <origin rpy="0 0 0" xyz="-0.015855 0.0 -0.04202" />
+      <origin rpy="0 0 0" xyz="-0.015855 0.0 0.0" />
       <axis xyz="0 1 0" />
       <limit lower="-1.0" upper="0.0" effort="1" velocity="1" />
@@ -38,7 +47,7 @@
     </link>
     <joint name="${prefix}_right_finger_joint" type="revolute">
-      <parent link="${parent}" />
+      <parent link="${prefix}_motor_dummy_link" />
       <child link="${prefix}_right_finger_link" />
-      <origin rpy="0 0 0" xyz="0.015855 0.0 -0.04202" />
+      <origin rpy="0 0 0" xyz="0.015855 0.0 0.0" />
       <axis xyz="0 1 0" />
       <limit lower="0.0" upper="1.0" effort="1" velocity="1" />

File: sobit_mini_description/urdf/right_arm/right_arm.urdf.xacro (robot description, xacro)
@@ -32,5 +32,5 @@
       <parent link="${prefix}_shoulder_fixed_link" />
       <child link="${prefix}_shoulder_roll_link" />
-      <origin rpy="0 0 0" xyz="0.0 -0.13946 0.03941" />
+      <origin rpy="0 0 0" xyz="0.0 -0.14146 0.03941" />
       <axis xyz="0 -1 0" />
       <limit effort="30" lower="${-M_PI/2.0}" upper="${M_PI/2.0}" velocity="${M_PI/2.0}" />
@@ -44,5 +44,5 @@
       </collision>
       <visual>
-        <origin rpy="0 ${-M_PI/2.0} ${M_PI}" xyz="0.0 -0.0525 0.0" />
+        <origin rpy="0 ${-M_PI/2.0} ${M_PI}" xyz="0.0 -0.0509 0.0" />
         <geometry>
           <mesh filename="package://sobit_mini_description/meshes/sobit_mini_shoulder2.dae" />
@@ -58,5 +58,5 @@
       <parent link="${prefix}_shoulder_roll_link" />
       <child link="${prefix}_shoulder_flex_link" />
-      <origin rpy="${-M_PI/2.0} 0 0" xyz="0 -0.0525 0.0" />
+      <origin rpy="0 0 0" xyz="0 -0.0511 0.0" />
       <axis xyz="-1 0 0" />
       <limit effort="30" lower="${-M_PI/2.0}" upper="${M_PI/2.0}" velocity="${M_PI/2.0}" />
@@ -70,5 +70,5 @@
       </collision>
       <visual>
-        <origin rpy="0 ${M_PI} ${M_PI/2.0}" xyz="0.018 0.017 -0.14803" />
+        <origin rpy="${M_PI} ${M_PI/2.0} ${M_PI/2.0}" xyz="-0.0265 -0.0702 -0.06227" />
         <geometry>
           <mesh filename="package://sobit_mini_description/meshes/arm1_right.dae" />
@@ -84,6 +84,6 @@
       <parent link="${prefix}_shoulder_flex_link" />
       <child link="${prefix}_wrist_flex_link" />
-      <origin rpy="0 0 0" xyz="0 0 -0.1892" />
-      <axis xyz="-1 0 0" />
+      <origin rpy="0 0 0" xyz="-0.0005 -0.1105 0" />
+      <axis xyz="0 0 1" />
       <limit effort="30" lower="${-M_PI/2.0}" upper="${M_PI/2.0}" velocity="${M_PI/2.0}" />
     </joint>
@@ -96,5 +96,5 @@
       </collision>
       <visual>
-        <origin rpy="${M_PI/2.0} 0 ${-M_PI/2.0}" xyz="-0.021 -0.01 -0.029" />
+        <origin rpy="${M_PI/2.0} ${M_PI/2.0} 0" xyz="-0.0260 0.0405 -0.0624" />
         <geometry>
           <mesh filename="package://sobit_mini_description/meshes/arm2_right.dae" />

File: sobit_mini_description/urdf/right_hand/right_hand.urdf.xacro (robot description, xacro)
@@ -3,7 +3,16 @@
   <xacro:include filename="$(find sobit_mini_description)/urdf/right_hand/right_hand.transmission.xacro" />
   <xacro:macro name="right_hand" params="prefix parent">
+    <joint name="${prefix}_motor_dummy_joint" type="fixed">
+      <parent link="${parent}" />
+      <child link="${prefix}_motor_dummylink" />
+      <origin rpy="${-M_PI/2.0} ${M_PI/2.0} 0" xyz="0 -0.15 0" />
+      <axis xyz="0 1 0" />
+      <limit lower="0.0" upper="${M_PI/2.0}" effort="1" velocity="1" />
+    </joint>
+    <link name="${prefix}_motor_dummylink" />
     <joint name="${prefix}_motor_joint" type="revolute">
-      <parent link="${parent}" />
+      <parent link="${prefix}_motor_dummylink" />
       <child link="${prefix}_motor_link" />
+      <origin rpy="0 0 0" xyz="0 0 0" />
       <axis xyz="0 1 0" />
       <limit lower="0.0" upper="${M_PI/2.0}" effort="1" velocity="1" />
@@ -11,7 +20,7 @@
     <link name="${prefix}_motor_link" />
     <joint name="${prefix}_left_finger_joint" type="revolute">
-      <parent link="${parent}" />
+      <parent link="${prefix}_motor_dummylink" />
       <child link="${prefix}_left_finger_link" />
-      <origin rpy="0 0 0" xyz="0.015855 0.0 -0.04202" />
+      <origin rpy="0 0 0" xyz="0.015855 0.0 0" />
       <axis xyz="0 1 0" />
       <limit lower="-1" upper="0" effort="1" velocity="1" />
@@ -38,7 +47,7 @@
     </link>
     <joint name="${prefix}_right_finger_joint" type="revolute">
-      <parent link="${parent}" />
+      <parent link="${prefix}_motor_dummylink" />
       <child link="${prefix}_right_finger_link" />
-      <origin rpy="0 0 0" xyz="-0.015855 0.0 -0.04202" />
+      <origin rpy="0 0 0" xyz="-0.015855 0.0 0" />
       <axis xyz="0 1 0" />
       <limit lower="-1.0" upper="0.0" effort="1" velocity="1" />
