Commit message: add library and change PID of hand motor,URDF

File: sobit_mini_description/urdf/left_arm/left_arm.transmission.xacro (robot description, xacro)
@@ -2,7 +2,8 @@
 <robot xmlns:xacro="http://ros.org/wiki/xacro">
   <xacro:macro name="left_arm_transmission" params="prefix">
-    <position_joint_transmission joint="${prefix}_shoulder_flex_joint" reduction="1" />
     <position_joint_transmission joint="${prefix}_shoulder_roll_joint" reduction="1" />
-    <position_joint_transmission joint="${prefix}_wrist_flex_joint" reduction="1" />
+    <position_joint_transmission joint="${prefix}_shoulder_pan_joint" reduction="1" />
+    <position_joint_transmission joint="${prefix}_elbow_tilt_joint" reduction="1" />
+    <position_joint_transmission joint="${prefix}_wrist_tilt_joint" reduction="1" />
   </xacro:macro>
 </robot>

File: sobit_mini_description/urdf/left_arm/left_arm.urdf.xacro (robot description, xacro)
@@ -37,5 +37,5 @@
       <origin rpy="0 0 0" xyz="0.0 0.1415 0.015161" />
       <axis xyz="0 -1 0" />
-      <limit effort="30" lower="${-M_PI/2.0}" upper="${M_PI/2.0}" velocity="${M_PI}" />
+      <limit effort="30" lower="${-M_PI/2.0}" upper="${M_PI}" velocity="${M_PI}" />
     </joint>
     <link name="${prefix}_shoulder_roll_link">

File: sobit_mini_description/urdf/left_hand/left_hand.urdf.xacro (robot description, xacro)
@@ -3,14 +3,16 @@
   <xacro:include filename="$(find sobit_mini_description)/urdf/left_hand/left_hand.transmission.xacro" />
   <xacro:macro name="left_hand" params="prefix parent">
-    <joint name="${prefix}_motor_dummy_joint" type="fixed">
+    <joint name="${prefix}_base_joint" type="fixed">
       <parent link="${parent}" />
-      <child link="${prefix}_motor_dummy_link" />
-      <origin rpy="${M_PI/2.0} ${-M_PI/2.0} 0" xyz="0.0 0.04725 0.0" />
+      <child link="${prefix}_base_link" />
+      <!-- <origin rpy="${M_PI/2.0} ${-M_PI/2.0} 0" xyz="0.0 0.04725 0.0" /> -->
+      <origin rpy="${M_PI/2.0} ${-M_PI/2.0} 0" xyz="0.0 0.0 0.0" />
       <axis xyz="0 1 0" />
       <limit lower="0.0" upper="${M_PI/2.0}" effort="1" velocity="1" />
     </joint>
-    <link name="${prefix}_motor_dummy_link">
+    <link name="${prefix}_base_link">
       <visual>
-        <origin xyz="0.0 0.0 0.04725" rpy="${M_PI/2.0} 0.0 0.0" />
+        <!-- <origin xyz="0.0 0.0 0.04725" rpy="${M_PI/2.0} 0.0 0.0" /> -->
+        <origin xyz="0.0 0.0 0.0" rpy="${M_PI/2.0} 0.0 0.0" />
         <geometry>
           <mesh filename="package://sobit_mini_description/meshes/L_hand/L_hand_JOINT.stl"/>
@@ -19,5 +21,6 @@
       </visual>
       <collision>
-        <origin xyz="0.0 0.0 0.04725" rpy="${M_PI/2.0} 0.0 0.0" />
+        <!-- <origin xyz="0.0 0.0 0.04725" rpy="${M_PI/2.0} 0.0 0.0" /> -->
+        <origin xyz="0.0 0.0 0.0" rpy="${M_PI/2.0} 0.0 0.0" />
         <geometry>
           <mesh filename="package://sobit_mini_description/meshes/L_hand/L_hand_JOINT.stl"/>
@@ -33,7 +36,9 @@
     </link>
     <joint name="${prefix}_joint" type="revolute">
-      <parent link="${prefix}_motor_dummy_link" />
+      <parent link="${prefix}_base_link" />
+      <!-- <parent link="${parent}" /> -->
       <child link="${prefix}_motor_link" />
-      <origin rpy="0 0 0" xyz="0 0 0" />
+      <!-- <origin rpy="0 0 0" xyz="0 0 0" /> -->
+      <origin rpy="0 0 0" xyz="-0.015855 0.0 -0.04725" />
       <axis xyz="0 1 0" />
       <limit lower="0.0" upper="${M_PI/2.0}" effort="1" velocity="1" />
@@ -41,7 +46,10 @@
     <link name="${prefix}_motor_link" />
     <joint name="${prefix}_right_finger_joint" type="revolute">
-      <parent link="${prefix}_motor_dummy_link" />
+      <parent link="${prefix}_base_link" />
+      <!-- <parent link="${parent}" /> -->
       <child link="${prefix}_right_finger_link" />
-      <origin rpy="0 0 0" xyz="-0.015855 0.0 0.0" />
+      <!-- <origin rpy="0 0 0" xyz="-0.015855 0.0 0.0" /> -->
+      <!-- <origin rpy="${M_PI/2.0} ${-M_PI/2.0} 0" xyz="0.0 0.04725 -0.015855" /> -->
+      <origin rpy="0 0 0" xyz="-0.015855 0.0 -0.04725" />
       <axis xyz="0 -1 0" />
       <limit lower="-1.0" upper="0.0" effort="1" velocity="1" />
@@ -71,7 +79,10 @@
     </link>
     <joint name="${prefix}_left_finger_joint" type="revolute">
-      <parent link="${prefix}_motor_dummy_link" />
+      <parent link="${prefix}_base_link" />
+      <!-- <parent link="${parent}" /> -->
       <child link="${prefix}_left_finger_link" />
-      <origin rpy="0 0 0" xyz="0.015855 0.0 0.0" />
+      <!-- <origin rpy="0 0 0" xyz="0.015855 0.0 0.0" /> -->
+      <!-- <origin rpy="${M_PI/2.0} ${-M_PI/2.0} 0" xyz="0.0 0.04725 0.015855" /> -->
+      <origin rpy="0 0 0" xyz="0.015855 0.0 -0.04725" />
       <axis xyz="0 1 0" />
       <limit lower="0.0" upper="1.0" effort="1" velocity="1" />

File: sobit_mini_description/urdf/right_arm/right_arm.transmission.xacro (robot description, xacro)
@@ -2,7 +2,8 @@
 <robot xmlns:xacro="http://ros.org/wiki/xacro">
   <xacro:macro name="right_arm_transmission" params="prefix">
-    <position_joint_transmission joint="${prefix}_shoulder_flex_joint" reduction="1" />
     <position_joint_transmission joint="${prefix}_shoulder_roll_joint" reduction="1" />
-    <position_joint_transmission joint="${prefix}_wrist_flex_joint" reduction="1" />
+    <position_joint_transmission joint="${prefix}_shoulder_pan_joint" reduction="1" />
+    <position_joint_transmission joint="${prefix}_elbow_tilt_joint" reduction="1" />
+    <position_joint_transmission joint="${prefix}_wrist_tilt_joint" reduction="1" />
   </xacro:macro>
 </robot>

File: sobit_mini_description/urdf/right_arm/right_arm.urdf.xacro (robot description, xacro)
@@ -37,5 +37,5 @@
       <origin rpy="0 0 0" xyz="0.0 -0.1415 0.015161" />
       <axis xyz="0 -1 0" />
-      <limit effort="30" lower="${-M_PI/2.0}" upper="${M_PI/2.0}" velocity="${M_PI/2.0}" />
+      <limit effort="30" lower="${-M_PI/2.0}" upper="${M_PI}" velocity="${M_PI/2.0}" />
     </joint>
     <link name="${prefix}_shoulder_roll_link">

File: sobit_mini_description/urdf/right_hand/right_hand.urdf.xacro (robot description, xacro)
@@ -3,14 +3,16 @@
   <xacro:include filename="$(find sobit_mini_description)/urdf/right_hand/right_hand.transmission.xacro" />
   <xacro:macro name="right_hand" params="prefix parent">
-    <joint name="${prefix}_motor_dummy_joint" type="fixed">
+    <joint name="${prefix}_base_joint" type="fixed">
       <parent link="${parent}" />
-      <child link="${prefix}_motor_dummylink" />
-      <origin xyz="0.0 -0.04725 0.0" rpy="${-M_PI/2.0} ${M_PI/2.0} 0" />
+      <child link="${prefix}_base_link" />
+      <!-- <origin xyz="0.0 -0.04725 0.0" rpy="${-M_PI/2.0} ${M_PI/2.0} 0" /> -->
+      <origin  rpy="${-M_PI/2.0} ${M_PI/2.0} 0" xyz="0.0 0.0 0.0"/>
       <axis xyz="0 1 0" />
       <limit lower="0.0" upper="${M_PI/2.0}" effort="1" velocity="1" />
     </joint>
-    <link name="${prefix}_motor_dummylink">
+    <link name="${prefix}_base_link">
       <visual>
-        <origin xyz="0.0 0.0 0.04725" rpy="${M_PI/2.0} 0.0 0.0" />
+        <!-- <origin xyz="0.0 0.0 0.04725" rpy="${M_PI/2.0} 0.0 0.0" /> -->
+        <origin xyz="0.0 0.0 0.0" rpy="${M_PI/2.0} 0.0 0.0" />
         <geometry>
           <mesh filename="package://sobit_mini_description/meshes/R_hand/R_hand_JOINT.stl"/>
@@ -19,5 +21,6 @@
       </visual>
       <collision>
-        <origin xyz="0.0 0.0 0.04725" rpy="${M_PI/2.0} 0.0 0.0" />
+        <!-- <origin xyz="0.0 0.0 0.04725" rpy="${M_PI/2.0} 0.0 0.0" /> -->
+        <origin xyz="0.0 0.0 0.0" rpy="${M_PI/2.0} 0.0 0.0" />
         <geometry>
           <mesh filename="package://sobit_mini_description/meshes/R_hand/R_hand_JOINT.stl"/>
@@ -33,7 +36,8 @@
     </link>
     <joint name="${prefix}_joint" type="revolute">
-      <parent link="${prefix}_motor_dummylink" />
+      <parent link="${prefix}_base_link" />
       <child link="${prefix}_motor_link" />
-      <origin xyz="0.0 0.0 0.0" rpy="0.0 0.0 0.0" />
+      <!-- <origin xyz="0.0 0.0 0.0" rpy="0.0 0.0 0.0" /> -->
+      <origin rpy="0 0 0" xyz="0.015855 0.0 -0.04725" />
       <axis xyz="0 1 0" />
       <limit lower="0.0" upper="${M_PI/2.0}" effort="1" velocity="1" />
@@ -41,7 +45,8 @@
     <link name="${prefix}_motor_link" />
     <joint name="${prefix}_left_finger_joint" type="revolute">
-      <parent link="${prefix}_motor_dummylink" />
+      <parent link="${prefix}_base_link" />
       <child link="${prefix}_left_finger_link" />
-      <origin xyz="0.015855 0.0 0.0" rpy="0 0 0" />
+      <!-- <origin xyz="0.015855 0.0 0.0" rpy="0 0 0" /> -->
+      <origin rpy="0 0 0" xyz="0.015855 0.0 -0.04725" />
       <axis xyz="0 1 0" />
       <limit lower="-1" upper="0" effort="1" velocity="1" />
@@ -71,7 +76,8 @@
     </link>
     <joint name="${prefix}_right_finger_joint" type="revolute">
-      <parent link="${prefix}_motor_dummylink" />
+      <parent link="${prefix}_base_link" />
       <child link="${prefix}_right_finger_link" />
-      <origin xyz="-0.015855 0.0 0.0" rpy="0 0 0" />
+      <!-- <origin xyz="-0.015855 0.0 0.0" rpy="0 0 0" /> -->
+      <origin rpy="0 0 0" xyz="-0.015855 0.0 -0.04725" />
       <axis xyz="0 1 0" />
       <limit lower="-1.0" upper="0.0" effort="1" velocity="1" />
