Commit message: Rewrite setip.sh. Changing joint orientation of urdf model

File: sobit_mini_description/urdf/body/body.urdf.xacro (robot description, xacro)
@@ -62,16 +62,10 @@
       <parent link="${prefix}_big_gear_base_link" />
       <child link="${prefix}_roll_link" />
-      <origin xyz="0.0 0.0 0.0" rpy="0.0 0.0 0.0" />
-      <axis xyz="0 0 -1" />
+      <!-- <origin xyz="0.0 0.0 0.0" rpy="0.0 0.0 0.0" /> -->
+      <origin xyz="0.0 0.0 0.0325" rpy="0.0 0.0 0.0" />
+      <axis xyz="0 0 1" />
       <limit effort="30" lower="${-M_PI/2.0}" upper="${M_PI/2}" velocity="${M_PI/2.0}" />
     </joint>
-    <link name="${prefix}_roll_link"/>
-    <joint name="${prefix}_big_gear_joint" type="fixed">
-      <parent link="${prefix}_roll_link" />
-      <child link="${prefix}_big_gear_link" />
-      <origin xyz="0.0 0.0 0.0325" rpy="0.0 0.0 0.0" />
-      <axis xyz="0 0 1" />
-    </joint>
-    <link name="${prefix}_big_gear_link">
+    <link name="${prefix}_roll_link">
       <visual>
         <origin xyz="0.0 0.0 0.0" rpy="0.0 0.0 0.0" />
@@ -95,6 +89,14 @@
       </inertial>
     </link>
+    <joint name="${prefix}_big_gear_joint" type="fixed">
+      <parent link="${prefix}_roll_link" />
+      <child link="${prefix}_big_gear_link" />
+      <origin xyz="0.0 0.0 0.0" rpy="0.0 0.0 0.0" />
+      <axis xyz="0 0 1" />
+    </joint>
+    <link name="${prefix}_big_gear_link"/>
     <joint name="${prefix}_back_pole_joint" type="fixed">
-      <parent link="${prefix}_big_gear_link" />
+      <!-- <parent link="${prefix}_big_gear_link" /> -->
+      <parent link="${prefix}_roll_link" />
       <child link="${prefix}_back_pole_link" />
       <origin xyz="-0.01 0.0 0.058" rpy="0.0 0.0 0.0" />
@@ -124,5 +126,6 @@
     </link>
     <joint name="${prefix}_front_pole_joint" type="fixed">
-      <parent link="${prefix}_big_gear_link" />
+      <!-- <parent link="${prefix}_big_gear_link" /> -->
+      <parent link="${prefix}_roll_link" />
       <child link="${prefix}_front_pole_link" />
       <origin xyz="0.0 0.0 0.0005" rpy="0.0 0.0 0.0" />
@@ -152,5 +155,6 @@
     </link>
     <joint name="${prefix}_sobit_mini_cover" type="fixed">
-      <parent link="${prefix}_big_gear_link" />
+      <!-- <parent link="${prefix}_big_gear_link" /> -->
+      <parent link="${prefix}_roll_link" />
       <child link="${prefix}_sobit_mini_cover" />
       <origin xyz="0.0 0.0 0.0" rpy="0.0 0.0 0.0" />

File: sobit_mini_description/urdf/left_arm/left_arm.urdf.xacro (robot description, xacro)
@@ -36,6 +36,6 @@
       <child link="${prefix}_shoulder_roll_link" />
       <origin rpy="0 0 0" xyz="0.0 0.1415 0.015161" />
-      <axis xyz="0 -1 0" />
-      <limit effort="30" lower="${-M_PI/2.0}" upper="${M_PI}" velocity="${M_PI}" />
+      <axis xyz="0 1 0" />
+      <limit effort="30" lower="${-M_PI}" upper="${M_PI/2.0}" velocity="${M_PI}" />
     </joint>
     <link name="${prefix}_shoulder_roll_link">
@@ -95,5 +95,5 @@
       <origin rpy="0 0 0" xyz="0 0.11125 0" />
       <axis xyz="0 0 1" />
-      <limit effort="30" lower="${-M_PI/2.0}" upper="${M_PI/2.0}" velocity="${M_PI/2.0}" />
+      <limit effort="30" lower="${-M_PI/2.0}" upper="0.0" velocity="${M_PI/2.0}" />
     </joint>
     <link name="${prefix}_elbow_tilt_link">
@@ -126,5 +126,26 @@
       <limit effort="30" lower="${-M_PI/2.0}" upper="${M_PI/2.0}" velocity="${M_PI/2.0}" />
     </joint>
-    <link name="${prefix}_wrist_tilt_link"/>
+    <link name="${prefix}_wrist_tilt_link">
+      <visual>
+        <origin xyz="0.0 0.0 0.0" rpy="0.0 ${-M_PI/2.0} ${M_PI}" />
+        <geometry>
+          <mesh filename="package://sobit_mini_description/meshes/L_hand/L_hand_JOINT.stl"/>
+        </geometry>
+        <material name="black" />
+      </visual>
+      <collision>
+        <origin xyz="0.0 0.0 0.0" rpy="0.0 ${-M_PI/2.0} ${M_PI}" />
+        <geometry>
+          <mesh filename="package://sobit_mini_description/meshes/L_hand/L_hand_JOINT.stl"/>
+        </geometry>
+      </collision>
+      <inertial>
+        <origin xyz="0.0 0.0 0.0" rpy="0.0 0.0 0.0" />
+        <mass value="0.08" />
+        <inertia ixx="1.0" ixy="0.0" ixz="0.0"
+                 iyy="1.0" iyz="0.0"
+                 izz="1.0" />
+      </inertial>
+    </link>
     <xacro:left_arm_transmission prefix="${prefix}"/>
   </xacro:macro>

File: sobit_mini_description/urdf/left_hand/left_hand.urdf.xacro (robot description, xacro)
@@ -3,56 +3,14 @@
   <xacro:include filename="$(find sobit_mini_description)/urdf/left_hand/left_hand.transmission.xacro" />
   <xacro:macro name="left_hand" params="prefix parent">
-    <joint name="${prefix}_base_joint" type="fixed">
+    <!-- <joint name="${prefix}_right_finger_joint" type="revolute"> -->
+    <joint name="${prefix}_joint" type="revolute">
+      <!-- <parent link="${prefix}_base_link" /> -->
       <parent link="${parent}" />
-      <child link="${prefix}_base_link" />
-      <!-- <origin rpy="${M_PI/2.0} ${-M_PI/2.0} 0" xyz="0.0 0.04725 0.0" /> -->
-      <origin rpy="${M_PI/2.0} ${-M_PI/2.0} 0" xyz="0.0 0.0 0.0" />
-      <axis xyz="0 1 0" />
-      <limit lower="0.0" upper="${M_PI/2.0}" effort="1" velocity="1" />
-    </joint>
-    <link name="${prefix}_base_link">
-      <visual>
-        <!-- <origin xyz="0.0 0.0 0.04725" rpy="${M_PI/2.0} 0.0 0.0" /> -->
-        <origin xyz="0.0 0.0 0.0" rpy="${M_PI/2.0} 0.0 0.0" />
-        <geometry>
-          <mesh filename="package://sobit_mini_description/meshes/L_hand/L_hand_JOINT.stl"/>
-        </geometry>
-        <material name="black" />
-      </visual>
-      <collision>
-        <!-- <origin xyz="0.0 0.0 0.04725" rpy="${M_PI/2.0} 0.0 0.0" /> -->
-        <origin xyz="0.0 0.0 0.0" rpy="${M_PI/2.0} 0.0 0.0" />
-        <geometry>
-          <mesh filename="package://sobit_mini_description/meshes/L_hand/L_hand_JOINT.stl"/>
-        </geometry>
-      </collision>
-      <inertial>
-        <origin xyz="0.0 0.0 0.0" rpy="0.0 0.0 0.0" />
-        <mass value="0.08" />
-        <inertia ixx="1.0" ixy="0.0" ixz="0.0"
-                 iyy="1.0" iyz="0.0"
-                 izz="1.0" />
-      </inertial>
-    </link>
-    <joint name="${prefix}_joint" type="revolute">
-      <parent link="${prefix}_base_link" />
-      <!-- <parent link="${parent}" /> -->
-      <child link="${prefix}_motor_link" />
-      <!-- <origin rpy="0 0 0" xyz="0 0 0" /> -->
-      <origin rpy="0 0 0" xyz="-0.015855 0.0 -0.04725" />
-      <axis xyz="0 1 0" />
-      <limit lower="0.0" upper="${M_PI/2.0}" effort="1" velocity="1" />
-    </joint>
-    <link name="${prefix}_motor_link" />
-    <joint name="${prefix}_right_finger_joint" type="revolute">
-      <parent link="${prefix}_base_link" />
-      <!-- <parent link="${parent}" /> -->
       <child link="${prefix}_right_finger_link" />
-      <!-- <origin rpy="0 0 0" xyz="-0.015855 0.0 0.0" /> -->
-      <!-- <origin rpy="${M_PI/2.0} ${-M_PI/2.0} 0" xyz="0.0 0.04725 -0.015855" /> -->
-      <origin rpy="0 0 0" xyz="-0.015855 0.0 -0.04725" />
+      <!-- <origin rpy="0 0 0" xyz="-0.015855 0.0 -0.04725" /> -->
+      <origin rpy="${M_PI/2.0} ${-M_PI/2.0} 0" xyz="0.0 0.04725 -0.015855" />
+      <!-- <origin rpy="${M_PI/2.0} ${-M_PI/2.0} 0" xyz="-0.015855 0.0 -0.04725" /> -->
       <axis xyz="0 -1 0" />
-      <limit lower="-1.0" upper="0.0" effort="1" velocity="1" />
-      <mimic joint="${prefix}_joint" multiplier="1.0" />
+      <limit lower="-1.0" upper="0.0" effort="30" velocity="${M_PI/2.0}" />
     </joint>
     <link name="${prefix}_right_finger_link">
@@ -79,12 +37,12 @@
     </link>
     <joint name="${prefix}_left_finger_joint" type="revolute">
-      <parent link="${prefix}_base_link" />
-      <!-- <parent link="${parent}" /> -->
+      <!-- <parent link="${prefix}_base_link" /> -->
+      <parent link="${parent}" />
       <child link="${prefix}_left_finger_link" />
-      <!-- <origin rpy="0 0 0" xyz="0.015855 0.0 0.0" /> -->
-      <!-- <origin rpy="${M_PI/2.0} ${-M_PI/2.0} 0" xyz="0.0 0.04725 0.015855" /> -->
-      <origin rpy="0 0 0" xyz="0.015855 0.0 -0.04725" />
+      <!-- <origin rpy="0 0 0" xyz="0.015855 0.0 -0.04725" /> -->
+      <origin rpy="${M_PI/2.0} ${-M_PI/2.0} 0" xyz="0.0 0.04725 0.015855" />
       <axis xyz="0 1 0" />
-      <limit lower="0.0" upper="1.0" effort="1" velocity="1" />
+      <limit lower="0.0" upper="1.0" effort="30" velocity="${M_PI/2.0}" />
+      <!-- <mimic joint="${prefix}_right_finger_joint" multiplier="1.0" /> -->
       <mimic joint="${prefix}_joint" multiplier="1.0" />
     </joint>
@@ -109,5 +67,4 @@
       </inertial>
     </link>
-    <!-- <xacro:left_hand_transmission prefix="${prefix}"/> -->
     <xacro:l_hand_transmission prefix="${prefix}"/>
   </xacro:macro>

File: sobit_mini_description/urdf/right_arm/right_arm.urdf.xacro (robot description, xacro)
@@ -95,5 +95,5 @@
       <origin rpy="0 0 0" xyz="0 -0.11125 0" />
       <axis xyz="0 0 1" />
-      <limit effort="30" lower="${-M_PI/2.0}" upper="${M_PI/2.0}" velocity="${M_PI/2.0}" />
+      <limit effort="30" lower="0.0" upper="${M_PI/2.0}" velocity="${M_PI/2.0}" />
     </joint>
     <link name="${prefix}_elbow_tilt_link">
@@ -126,5 +126,26 @@
       <limit effort="30" lower="${-M_PI/2.0}" upper="${M_PI/2.0}" velocity="${M_PI/2.0}" />
     </joint>
-    <link name="${prefix}_wrist_tilt_link"/>
+    <link name="${prefix}_wrist_tilt_link">
+      <visual>
+        <origin xyz="0.0 0.0 0.0" rpy="0.0 ${M_PI/2.0} 0.0" />
+        <geometry>
+          <mesh filename="package://sobit_mini_description/meshes/R_hand/R_hand_JOINT.stl"/>
+        </geometry>
+        <material name="black" />
+      </visual>
+      <collision>
+        <origin xyz="0.0 0.0 0.0" rpy="0.0 ${M_PI/2.0} 0.0" />
+        <geometry>
+          <mesh filename="package://sobit_mini_description/meshes/R_hand/R_hand_JOINT.stl"/>
+        </geometry>
+      </collision>
+      <inertial>
+        <origin xyz="0.0 0.0 0.0" rpy="0.0 0.0 0.0" />
+        <mass value="0.08" />
+        <inertia ixx="1.0" ixy="0.0" ixz="0.0"
+                 iyy="1.0" iyz="0.0"
+                 izz="1.0" />
+      </inertial>
+    </link>
     <xacro:right_arm_transmission prefix="${prefix}"/>
   </xacro:macro>

File: sobit_mini_description/urdf/right_hand/right_hand.urdf.xacro (robot description, xacro)
@@ -3,53 +3,13 @@
   <xacro:include filename="$(find sobit_mini_description)/urdf/right_hand/right_hand.transmission.xacro" />
   <xacro:macro name="right_hand" params="prefix parent">
-    <joint name="${prefix}_base_joint" type="fixed">
+    <!-- <joint name="${prefix}_left_finger_joint" type="revolute"> -->
+    <joint name="${prefix}_joint" type="revolute">
+      <!-- <parent link="${prefix}_base_link" /> -->
       <parent link="${parent}" />
-      <child link="${prefix}_base_link" />
-      <!-- <origin xyz="0.0 -0.04725 0.0" rpy="${-M_PI/2.0} ${M_PI/2.0} 0" /> -->
-      <origin  rpy="${-M_PI/2.0} ${M_PI/2.0} 0" xyz="0.0 0.0 0.0"/>
-      <axis xyz="0 1 0" />
-      <limit lower="0.0" upper="${M_PI/2.0}" effort="1" velocity="1" />
-    </joint>
-    <link name="${prefix}_base_link">
-      <visual>
-        <!-- <origin xyz="0.0 0.0 0.04725" rpy="${M_PI/2.0} 0.0 0.0" /> -->
-        <origin xyz="0.0 0.0 0.0" rpy="${M_PI/2.0} 0.0 0.0" />
-        <geometry>
-          <mesh filename="package://sobit_mini_description/meshes/R_hand/R_hand_JOINT.stl"/>
-        </geometry>
-        <material name="black" />
-      </visual>
-      <collision>
-        <!-- <origin xyz="0.0 0.0 0.04725" rpy="${M_PI/2.0} 0.0 0.0" /> -->
-        <origin xyz="0.0 0.0 0.0" rpy="${M_PI/2.0} 0.0 0.0" />
-        <geometry>
-          <mesh filename="package://sobit_mini_description/meshes/R_hand/R_hand_JOINT.stl"/>
-        </geometry>
-      </collision>
-      <inertial>
-        <origin xyz="0.0 0.0 0.0" rpy="0.0 0.0 0.0" />
-        <mass value="0.08" />
-        <inertia ixx="1.0" ixy="0.0" ixz="0.0"
-                 iyy="1.0" iyz="0.0"
-                 izz="1.0" />
-      </inertial>
-    </link>
-    <joint name="${prefix}_joint" type="revolute">
-      <parent link="${prefix}_base_link" />
-      <child link="${prefix}_motor_link" />
-      <!-- <origin xyz="0.0 0.0 0.0" rpy="0.0 0.0 0.0" /> -->
-      <origin rpy="0 0 0" xyz="0.015855 0.0 -0.04725" />
-      <axis xyz="0 1 0" />
-      <limit lower="0.0" upper="${M_PI/2.0}" effort="1" velocity="1" />
-    </joint>
-    <link name="${prefix}_motor_link" />
-    <joint name="${prefix}_left_finger_joint" type="revolute">
-      <parent link="${prefix}_base_link" />
       <child link="${prefix}_left_finger_link" />
-      <!-- <origin xyz="0.015855 0.0 0.0" rpy="0 0 0" /> -->
-      <origin rpy="0 0 0" xyz="0.015855 0.0 -0.04725" />
-      <axis xyz="0 1 0" />
-      <limit lower="-1" upper="0" effort="1" velocity="1" />
-      <mimic joint="${prefix}_joint" multiplier="-1.0"/>
+      <!-- <origin rpy="0 0 0" xyz="0.015855 0.0 -0.04725" /> -->
+      <origin rpy="${-M_PI/2.0} ${M_PI/2.0} 0" xyz="0.0 -0.04725 -0.015855" />
+      <axis xyz="0 -1 0" />
+      <limit lower="0" upper="1" effort="30" velocity="${M_PI/2.0}" />
     </joint>
     <link name="${prefix}_left_finger_link">
@@ -76,10 +36,12 @@
     </link>
     <joint name="${prefix}_right_finger_joint" type="revolute">
-      <parent link="${prefix}_base_link" />
+      <!-- <parent link="${prefix}_base_link" /> -->
+      <parent link="${parent}" />
       <child link="${prefix}_right_finger_link" />
-      <!-- <origin xyz="-0.015855 0.0 0.0" rpy="0 0 0" /> -->
-      <origin rpy="0 0 0" xyz="-0.015855 0.0 -0.04725" />
+      <!-- <origin rpy="0 0 0" xyz="-0.015855 0.0 -0.04725" /> -->
+      <origin rpy="${-M_PI/2.0} ${M_PI/2.0} 0" xyz="0.0 -0.04725 0.015855" />
       <axis xyz="0 1 0" />
-      <limit lower="-1.0" upper="0.0" effort="1" velocity="1" />
+      <limit lower="-1.0" upper="0.0" effort="30" velocity="${M_PI/2.0}" />
+      <!-- <mimic joint="${prefix}_left_finger_joint" multiplier="1.0" /> -->
       <mimic joint="${prefix}_joint" multiplier="1.0" />
     </joint>
@@ -106,5 +68,4 @@
       </inertial>
     </link>
-    <!-- <xacro:right_hand_transmission prefix="${prefix}"/> -->
     <xacro:r_hand_transmission prefix="${prefix}"/>
   </xacro:macro>

Commit message: update joint_control and urdf

File: sobit_mini_description/urdf/body/body.urdf.xacro (robot description, xacro)
@@ -3,13 +3,46 @@
   <xacro:include filename="$(find sobit_mini_description)/urdf/body/body.transmission.xacro" />
   <xacro:macro name="body" params="prefix parent">
-    <joint name="${prefix}_small_gear_joint" type="fixed">
+    <joint name="${prefix}_small_gear_base_joint" type="fixed">
       <parent link="${parent}" />
+      <child link="${prefix}_small_gear_base_link" />
+      <origin xyz="0.0 -0.13925 0.0031" rpy="0 0 0" />
+      <axis xyz="0 0 1" />
+    </joint>
+    <link name="${prefix}_small_gear_base_link">
+      <visual>
+        <origin xyz="0.0 0.0 0.034" rpy="0.0 0.0 ${M_PI/2.0}" />
+        <!-- <origin xyz="0.0 0.0 0.0" rpy="0.0 0.0 0.0" /> -->
+        <geometry>
+          <mesh filename="package://sobit_mini_description/meshes/body/sobit_mini_small_gear_motor.stl" />
+        </geometry>
+        <material name="black" />
+      </visual>
+      <collision>
+        <origin xyz="0.0 0.0 0.034" rpy="0.0 0.0 ${M_PI/2.0}" />
+        <geometry>
+          <mesh filename="package://sobit_mini_description/meshes/body/sobit_mini_small_gear_motor.stl" />
+        </geometry>
+      </collision>
+      <inertial>
+        <origin xyz="0.0 0.0 0.0" rpy="0.0 0.0 0.0" />
+        <mass value="1" />
+        <inertia ixx="1.0" ixy="0.0" ixz="0.0"
+                 iyy="1.0" iyz="0.0"
+                 izz="1.0" />
+      </inertial>
+    </link>
+    <!-- <joint name="${prefix}_small_gear_joint" type="revolute"> -->
+    <joint name="${prefix}_roll_joint" type="revolute">
+      <parent link="${prefix}_small_gear_base_link" />
       <child link="${prefix}_small_gear_link" />
-      <origin xyz="0.0 -0.14 0.0" rpy="0 0 0" />
-      <axis xyz="0 0 1" />
+      <origin xyz="0.0 0.0 0.036" rpy="0 0 ${M_PI/2.0}" />
+      <axis xyz="0 0 1" />
+      <limit effort="30" lower="${-1.31825*M_PI}" upper="${1.31825*M_PI}" velocity="${M_PI/2.0}" />
+      <!-- <limit effort="30" lower="${-M_PI/4.0}" upper="${M_PI/4.0}" velocity="${M_PI/2.0}" /> -->
     </joint>
     <link name="${prefix}_small_gear_link">
       <visual>
-        <origin xyz="0.0 0.0 0.0" rpy="${M_PI} ${M_PI} ${M_PI/2.0}" />
+        <origin xyz="0.0 0.0 0.0" rpy="${M_PI/2.0} 0.0 0.0" />
+        <!-- <origin xyz="0.0 0.0 0.0" rpy="0.0 0.0 0.0" /> -->
         <geometry>
           <mesh filename="package://sobit_mini_description/meshes/body/sobit_mini_small_gear.stl" />
@@ -18,5 +51,5 @@
       </visual>
       <collision>
-        <origin xyz="0.0 0.0 0.0" rpy="${M_PI} ${M_PI} ${M_PI/2.0}" />
+        <origin xyz="0.0 0.0 0.0" rpy="${M_PI/2.0} 0.0 0.0" />
         <geometry>
           <mesh filename="package://sobit_mini_description/meshes/body/sobit_mini_small_gear.stl" />
@@ -48,16 +81,16 @@
         <origin xyz="0.0 0.0 0.0" rpy="0.0 0.0 0.0" />
         <geometry>
-          <mesh filename="package://sobit_mini_description/meshes/body/sobit_mini_small_gear.stl" />
-        </geometry>
-      </collision>
-      <inertial>
-        <origin xyz="0.0 0.0 0.0" rpy="0.0 0.0 0.0" />
-        <mass value="1" />
-        <inertia ixx="1.0" ixy="0.0" ixz="0.0"
-                 iyy="1.0" iyz="0.0"
-                 izz="1.0" />
-      </inertial>
-    </link>
-    <joint name="${prefix}_roll_joint" type="revolute">
+          <mesh filename="package://sobit_mini_description/meshes/body/big_gear_base.stl" />
+        </geometry>
+      </collision>
+      <inertial>
+        <origin xyz="0.0 0.0 0.0" rpy="0.0 0.0 0.0" />
+        <mass value="1" />
+        <inertia ixx="1.0" ixy="0.0" ixz="0.0"
+                 iyy="1.0" iyz="0.0"
+                 izz="1.0" />
+      </inertial>
+    </link>
+    <joint name="${prefix}_big_gear_base_joint" type="revolute">
       <parent link="${prefix}_big_gear_base_link" />
       <child link="${prefix}_roll_link" />
@@ -65,5 +98,6 @@
       <origin xyz="0.0 0.0 0.0325" rpy="0.0 0.0 0.0" />
       <axis xyz="0 0 1" />
-      <limit effort="30" lower="${-M_PI/2.0}" upper="${M_PI/2}" velocity="${M_PI/2.0}" />
+      <limit effort="30" lower="${M_PI/4.0}" upper="${-M_PI/4.0}" velocity="${M_PI/2.0}" />
+      <mimic joint="${prefix}_roll_joint" multiplier="-0.1896551724" offset="0.0"/>
     </joint>
     <link name="${prefix}_roll_link">
