Commit message: update library

File: sobit_mini_description/urdf/body/body.urdf.xacro (robot description, xacro)
@@ -12,5 +12,4 @@
       <visual>
         <origin xyz="0.0 0.0 0.034" rpy="0.0 0.0 ${M_PI/2.0}" />
-        <!-- <origin xyz="0.0 0.0 0.0" rpy="0.0 0.0 0.0" /> -->
         <geometry>
           <mesh filename="package://sobit_mini_description/meshes/body/sobit_mini_small_gear_motor.stl" />
@@ -32,5 +31,4 @@
       </inertial>
     </link>
-    <!-- <joint name="${prefix}_small_gear_joint" type="revolute"> -->
     <joint name="${prefix}_roll_joint" type="revolute">
       <parent link="${prefix}_small_gear_base_link" />
@@ -39,10 +37,8 @@
       <axis xyz="0 0 1" />
       <limit effort="30" lower="${-1.31825*M_PI}" upper="${1.31825*M_PI}" velocity="${M_PI/2.0}" />
-      <!-- <limit effort="30" lower="${-M_PI/4.0}" upper="${M_PI/4.0}" velocity="${M_PI/2.0}" /> -->
     </joint>
     <link name="${prefix}_small_gear_link">
       <visual>
         <origin xyz="0.0 0.0 0.0" rpy="${M_PI/2.0} 0.0 0.0" />
-        <!-- <origin xyz="0.0 0.0 0.0" rpy="0.0 0.0 0.0" /> -->
         <geometry>
           <mesh filename="package://sobit_mini_description/meshes/body/sobit_mini_small_gear.stl" />
@@ -95,5 +91,4 @@
       <parent link="${prefix}_big_gear_base_link" />
       <child link="${prefix}_roll_link" />
-      <!-- <origin xyz="0.0 0.0 0.0" rpy="0.0 0.0 0.0" /> -->
       <origin xyz="0.0 0.0 0.0325" rpy="0.0 0.0 0.0" />
       <axis xyz="0 0 1" />
@@ -131,5 +126,4 @@
     <link name="${prefix}_big_gear_link"/>
     <joint name="${prefix}_back_pole_joint" type="fixed">
-      <!-- <parent link="${prefix}_big_gear_link" /> -->
       <parent link="${prefix}_roll_link" />
       <child link="${prefix}_back_pole_link" />
@@ -160,5 +154,4 @@
     </link>
     <joint name="${prefix}_front_pole_joint" type="fixed">
-      <!-- <parent link="${prefix}_big_gear_link" /> -->
       <parent link="${prefix}_roll_link" />
       <child link="${prefix}_front_pole_link" />
@@ -189,5 +182,4 @@
     </link>
     <joint name="${prefix}_sobit_mini_cover" type="fixed">
-      <!-- <parent link="${prefix}_big_gear_link" /> -->
       <parent link="${prefix}_roll_link" />
       <child link="${prefix}_sobit_mini_cover" />

File: sobit_mini_description/urdf/head/head.urdf.xacro (robot description, xacro)
@@ -8,5 +8,5 @@
       <origin xyz="0.0 0.0 0.516" rpy="0.0 0.0 0.0" />
       <axis xyz="0 0 1" />
-      <limit effort="30" lower="-2.617" upper="2.617" velocity="${M_PI/2.0}" />
+      <limit effort="30" lower="-1.57" upper="1.57" velocity="${M_PI/2.0}" />
     </joint>
     <link name="${prefix}_pan_link">

File: sobit_mini_description/urdf/left_arm/left_arm.urdf.xacro (robot description, xacro)
@@ -66,5 +66,5 @@
       <origin rpy="0 0 0" xyz="0.0 0.05375 0.0" />
       <axis xyz="1 0 0" />
-      <limit effort="30" lower="${-M_PI/2.0}" upper="${M_PI/2.0}" velocity="${M_PI/2.0}" />
+      <limit effort="30" lower="${-M_PI/2.0}" upper="1.22173" velocity="${M_PI/2.0}" />
     </joint>
     <link name="${prefix}_shoulder_pan_link">

File: sobit_mini_description/urdf/left_hand/left_hand.urdf.xacro (robot description, xacro)
@@ -3,12 +3,8 @@
   <xacro:include filename="$(find sobit_mini_description)/urdf/left_hand/left_hand.transmission.xacro" />
   <xacro:macro name="left_hand" params="prefix parent">
-    <!-- <joint name="${prefix}_right_finger_joint" type="revolute"> -->
     <joint name="${prefix}_joint" type="revolute">
-      <!-- <parent link="${prefix}_base_link" /> -->
       <parent link="${parent}" />
       <child link="${prefix}_right_finger_link" />
-      <!-- <origin rpy="0 0 0" xyz="-0.015855 0.0 -0.04725" /> -->
       <origin rpy="${M_PI/2.0} ${-M_PI/2.0} 0" xyz="0.0 0.04725 -0.015855" />
-      <!-- <origin rpy="${M_PI/2.0} ${-M_PI/2.0} 0" xyz="-0.015855 0.0 -0.04725" /> -->
       <axis xyz="0 -1 0" />
       <limit lower="-1.0" upper="0.0" effort="30" velocity="${M_PI/2.0}" />
@@ -37,12 +33,9 @@
     </link>
     <joint name="${prefix}_left_finger_joint" type="revolute">
-      <!-- <parent link="${prefix}_base_link" /> -->
       <parent link="${parent}" />
       <child link="${prefix}_left_finger_link" />
-      <!-- <origin rpy="0 0 0" xyz="0.015855 0.0 -0.04725" /> -->
       <origin rpy="${M_PI/2.0} ${-M_PI/2.0} 0" xyz="0.0 0.04725 0.015855" />
       <axis xyz="0 1 0" />
       <limit lower="0.0" upper="1.0" effort="30" velocity="${M_PI/2.0}" />
-      <!-- <mimic joint="${prefix}_right_finger_joint" multiplier="1.0" /> -->
       <mimic joint="${prefix}_joint" multiplier="1.0" />
     </joint>

File: sobit_mini_description/urdf/right_arm/right_arm.urdf.xacro (robot description, xacro)
@@ -66,5 +66,5 @@
       <origin rpy="0 0 0" xyz="0.0 -0.05375 0.0" />
       <axis xyz="1 0 0" />
-      <limit effort="30" lower="${-M_PI/2.0}" upper="${M_PI/2.0}" velocity="${M_PI/2.0}" />
+      <limit effort="30" lower="-1.22173" upper="${M_PI/2.0}" velocity="${M_PI/2.0}" />
     </joint>
     <link name="${prefix}_shoulder_pan_link">

File: sobit_mini_description/urdf/right_hand/right_hand.urdf.xacro (robot description, xacro)
@@ -3,10 +3,7 @@
   <xacro:include filename="$(find sobit_mini_description)/urdf/right_hand/right_hand.transmission.xacro" />
   <xacro:macro name="right_hand" params="prefix parent">
-    <!-- <joint name="${prefix}_left_finger_joint" type="revolute"> -->
     <joint name="${prefix}_joint" type="revolute">
-      <!-- <parent link="${prefix}_base_link" /> -->
       <parent link="${parent}" />
       <child link="${prefix}_left_finger_link" />
-      <!-- <origin rpy="0 0 0" xyz="0.015855 0.0 -0.04725" /> -->
       <origin rpy="${-M_PI/2.0} ${M_PI/2.0} 0" xyz="0.0 -0.04725 -0.015855" />
       <axis xyz="0 -1 0" />
@@ -36,12 +33,9 @@
     </link>
     <joint name="${prefix}_right_finger_joint" type="revolute">
-      <!-- <parent link="${prefix}_base_link" /> -->
       <parent link="${parent}" />
       <child link="${prefix}_right_finger_link" />
-      <!-- <origin rpy="0 0 0" xyz="-0.015855 0.0 -0.04725" /> -->
       <origin rpy="${-M_PI/2.0} ${M_PI/2.0} 0" xyz="0.0 -0.04725 0.015855" />
       <axis xyz="0 1 0" />
       <limit lower="-1.0" upper="0.0" effort="30" velocity="${M_PI/2.0}" />
-      <!-- <mimic joint="${prefix}_left_finger_joint" multiplier="1.0" /> -->
       <mimic joint="${prefix}_joint" multiplier="1.0" />
     </joint>

File: sobit_mini_description/urdf/sensor/mic.urdf.xacro (robot description, xacro)
@@ -5,5 +5,4 @@
       <parent link="${parent}" />
       <child link="${prefix}_base_link" />
-      <!-- <origin xyz="0.190 0.0 0.610" rpy="0.0 0.0 0.0" /> -->
       <origin xyz="-0.039589 0.0 0.169655" rpy="0.0 0.0 0.0" />
     </joint>
@@ -31,33 +30,4 @@
       </inertial>
     </link>
-    <!-- <link name="${prefix}_base_link">
-      <visual>
-        <origin xyz="0.0 0.0 0.0" rpy="${M_PI/2} 0 ${M_PI/2}" />
-        <geometry>
-          <mesh filename="package://sobit_edu_description/meshes/sensor/mic_base.stl" scale="0.001 0.001 0.001" />
-        </geometry>
-        <material name="black" />
-      </visual>
-      <collision>
-        <origin xyz="0.0 0.0 0.0" rpy="${M_PI/2} 0 ${M_PI/2}" />
-        <geometry>
-          <mesh filename="package://sobit_edu_description/meshes/sensor/mic_base.stl" scale="0.001 0.001 0.001" />
-        </geometry>
-        <material name="black" />
-      </collision>
-      <inertial>
-        <origin xyz="0.0 0.0 0.0" rpy="0 0 0" />
-        <mass value="1" />
-        <inertia ixx="1.0" ixy="0.0" ixz="0.0"
-                 iyy="1.0" iyz="0.0"
-                 izz="1.0" />
-      </inertial>
-    </link> -->
-    <!-- <joint name="${prefix}_joint" type="fixed">
-      <parent link="${prefix}_base_link" />
-      <child link="${prefix}_link" />
-      <origin xyz="-0.017007 0.0 0.020" rpy="0.0 0.0 0.0" />
-    </joint> -->
-    <!-- <link name="${prefix}_link"> -->
   </xacro:macro>
 </robot>

File: sobit_mini_description/urdf/sensor/realsense_d435.urdf.xacro (robot description, xacro)
@@ -3,5 +3,4 @@
   <xacro:macro name="realsense_d435" params="prefix parent">
     <joint name="${prefix}_base_joint" type="fixed">
-      <!-- <origin xyz="0.0908687 0.0 -0.01539994" rpy="0.0 0.0 0.0" /> -->
       <origin xyz="0.0045 0.0 0.169655" rpy="0.0 0.0 0.0" />
       <parent link="${parent}" />

File: sobit_mini_description/urdf/stacks/stacks.urdf.xacro (robot description, xacro)
@@ -19,5 +19,4 @@
         <origin xyz="0 0 0" rpy="0 0 0" />
         <geometry>
-          <!-- <mesh filename="package://turtlebot_description/meshes/stacks/hexagons/pole_bottom.dae" /> -->
           <mesh filename="package://sobit_mini_description/meshes/body/pole_bottom_39mm.stl" scale="${M_SCALE} ${M_SCALE} ${M_SCALE}" />
         </geometry>
@@ -49,5 +48,4 @@
         <origin xyz="0 0 0" rpy="0 ${M_PI} 0" />
         <geometry>
-          <!-- <mesh filename="package://turtlebot_description/meshes/sensors/sensor_pole.dae" /> -->
           <mesh filename="package://sobit_mini_description/meshes/body/pole_middle_134mm.stl" scale="${M_SCALE} ${M_SCALE} ${M_SCALE}" />
         </geometry>
@@ -79,5 +77,4 @@
         <origin xyz=" 0 0 0" rpy="0 0 0" />
         <geometry>
-          <!-- <mesh filename="package://turtlebot_description/meshes/stacks/hexagons/pole_top.dae" /> -->
           <mesh filename="package://sobit_mini_description/meshes/body/pole_top_134mm.stl" scale="${M_SCALE} ${M_SCALE} ${M_SCALE}" />
         </geometry>
@@ -174,5 +171,4 @@
     <xacro:stack_middle_pole parent="${parent}" number="7" x_loc="-0.0381" y_loc="-0.1505" z_loc="0.13385" /> -->
     <joint name="plate_middle_joint" type="fixed">
-      <!-- <origin xyz="-0.01364 0.0 0.222" rpy="0 0 0" /> -->
       <origin xyz="-0.01364 0.0 0.2646" rpy="0 0 0" />
       <parent link="${parent}" />
