Commit message: Fix the axis of head URDF

File: sobit_mini_description/urdf/head/head.urdf.xacro (robot description, xacro)
@@ -31,6 +31,6 @@
       <child link="${prefix}_tilt_link" />
       <origin xyz="0.0 0.0 0.017" rpy="0.0 0.0 0.0" />
-      <!-- <axis xyz="0 -1 0" /> -->
-      <axis xyz="0 1 0" />
+      <axis xyz="0 -1 0" />
+      <!-- <axis xyz="0 1 0" /> -->
       <limit effort="30" lower="-1" upper="1" velocity="${M_PI/2.0}" />
     </joint>
