Commit message: Change package and Cmakelist

File: sobit_mini_description/urdf/base/base.urdf.xacro (robot description, xacro)
@@ -54,11 +54,11 @@
       </inertial>
     </link>
-    <joint name="wheel_left_joint" type="continuous">
+    <joint name="wheel_l_joint" type="continuous">
       <parent link="base_link" />
-      <child link="wheel_left_link" />
+      <child link="wheel_l_link" />
       <origin xyz="0.00 ${0.23/2} 0.0250" rpy="${-M_PI/2} 0 0" />
       <axis xyz="0 0 1" />
     </joint>
-    <link name="wheel_left_link">
+    <link name="wheel_l_link">
       <visual>
         <geometry>
@@ -79,11 +79,11 @@
       </inertial>
     </link>
-    <joint name="wheel_right_joint" type="continuous">
+    <joint name="wheel_r_joint" type="continuous">
       <parent link="base_link" />
-      <child link="wheel_right_link" />
+      <child link="wheel_r_link" />
       <origin xyz="0.00 -${0.23/2} 0.0250" rpy="${-M_PI/2} 0 0" />
       <axis xyz="0 0 1" />
     </joint>
-    <link name="wheel_right_link">
+    <link name="wheel_r_link">
       <visual>
         <geometry>

Commit message: Update ROS2 for urdf

File: sobit_mini_description/urdf/base/base.urdf.xacro (robot description, xacro)
@@ -30,5 +30,5 @@
         <geometry>
           <!-- new mesh -->
-          <mesh filename="package://kobuki_description/meshes/main_body.dae" />
+          <mesh filename="file://$(find kobuki_description)/meshes/main_body.dae" />
         </geometry>
         <origin xyz="0.001 0 0.05199" rpy="0 0 0" />
@@ -63,5 +63,5 @@
       <visual>
         <geometry>
-          <mesh filename="package://kobuki_description/meshes/wheel.dae" />
+          <mesh filename="file://$(find kobuki_description)/meshes/wheel.dae" />
         </geometry>
         <origin xyz="0 0 0" rpy="0 0 0" />
@@ -90,5 +90,5 @@
       <visual>
         <geometry>
-          <mesh filename="package://kobuki_description/meshes/wheel.dae" />
+          <mesh filename="file://$(find kobuki_description)/meshes/wheel.dae" />
         </geometry>
         <origin xyz="0 0 0" rpy="0 0 0" />

File: sobit_mini_description/urdf/body/body.urdf.xacro (robot description, xacro)
@@ -13,5 +13,5 @@
         <origin xyz="0.0 0.0 0.034" rpy="0.0 0.0 ${M_PI/2.0}" />
         <geometry>
-          <mesh filename="file://$(sobit_mini_description)/meshes/body/sobit_mini_small_gear_motor.stl" />
+          <mesh filename="file://$(find sobit_mini_description)/meshes/body/sobit_mini_small_gear_motor.stl" />
         </geometry>
         <material name="black" />
@@ -42,5 +42,5 @@
         <origin xyz="0.0 0.0 0.0" rpy="${M_PI/2.0} 0.0 ${M_PI/2.0}" />
         <geometry>
-          <mesh filename="file://$(sobit_mini_description)/meshes/body/sobit_mini_small_gear.stl" />
+          <mesh filename="file://$(find sobit_mini_description)/meshes/body/sobit_mini_small_gear.stl" />
         </geometry>
         <material name="black" />
@@ -70,7 +70,7 @@
         <origin xyz="0.0 0.0 0.0" rpy="0.0 0.0 0.0" />
         <geometry>
-          <mesh filename="file://$(sobit_mini_description)/meshes/body/big_gear_base.stl" />
-        </geometry>
-        <material name="silver" />
+          <mesh filename="file://$(find sobit_mini_description)/meshes/body/big_gear_base.stl" />
+        </geometry>
+        <material name="grey" />
       </visual>
       <collision>
@@ -100,5 +100,5 @@
         <origin xyz="0.0 0.0 0.0" rpy="0.0 0.0 0.0" />
         <geometry>
-          <mesh filename="file://$(sobit_mini_description)/meshes/body/sobit_mini_big_gear.stl" />
+          <mesh filename="file://$(find sobit_mini_description)/meshes/body/sobit_mini_big_gear.stl" />
         </geometry>
         <material name="black" />
@@ -135,5 +135,5 @@
         <origin xyz="0.0 0.0 0.0" rpy="0 0 ${M_PI/2.0}" />
         <geometry>
-          <mesh filename="file://$(sobit_mini_description)/meshes/body/sobit_mini_center_back.stl" />
+          <mesh filename="file://$(find sobit_mini_description)/meshes/body/sobit_mini_center_back.stl" />
         </geometry>
         <material name="black" />
@@ -163,5 +163,5 @@
         <origin xyz="0.0 0.0 0.0" rpy="0.0 0.0 ${M_PI/2.0}" />
         <geometry>
-          <mesh filename="file://$(sobit_mini_description)/meshes/body/spine.stl" />
+          <mesh filename="file://$(find sobit_mini_description)/meshes/body/spine.stl" />
         </geometry>
         <material name="black" />
@@ -191,5 +191,5 @@
         <origin xyz="0.0 0.0 0.459" rpy="0.0 0.0 ${M_PI/2.0}" />
         <geometry>
-          <mesh filename="file://$(sobit_mini_description)/meshes/body/sobit_mini_body_cover.dae" />
+          <mesh filename="file://$(find sobit_mini_description)/meshes/body/sobit_mini_body_cover.dae" />
         </geometry>
       </visual>

File: sobit_mini_description/urdf/head/head.urdf.xacro (robot description, xacro)
@@ -31,5 +31,6 @@
       <child link="${prefix}_tilt_link" />
       <origin xyz="0.0 0.0 0.017" rpy="0.0 0.0 0.0" />
-      <axis xyz="0 -1 0" />
+      <!-- <axis xyz="0 -1 0" /> -->
+      <axis xyz="0 1 0" />
       <limit effort="30" lower="-1" upper="1" velocity="${M_PI/2.0}" />
     </joint>
@@ -63,6 +64,6 @@
     <gazebo reference="${prefix}_pan_link">
       <material>Gazebo/Black</material>
-    </gazebo>
-    <xacro:head_transmission prefix="${prefix}"/> -->
+    </gazebo> -->
+    <xacro:head_transmission prefix="${prefix}"/>
   </xacro:macro>
 </robot>

File: sobit_mini_description/urdf/left_hand/left_hand.urdf.xacro (robot description, xacro)
@@ -45,5 +45,5 @@
         <origin xyz="0.0 0.0 0.0" rpy="${M_PI/2.0} 0.0 0.0" />
         <geometry>
-          <mesh filename="file://$(find sobit_mini_description)/meshes/l_hand/Ll_hand_finger_l_joint.stl" />
+          <mesh filename="file://$(find sobit_mini_description)/meshes/l_hand/l_hand_finger_l_joint.stl" />
         </geometry>
         <material name="black" />

File: sobit_mini_description/urdf/sensor/lidar.urdf.xacro (robot description, xacro)
@@ -14,4 +14,5 @@
           <mesh filename="file://$(find sobit_mini_description)/meshes/sobit_mini_urg_sup.dae" scale="0.001 0.001 0.001" />
         </geometry>
+        <material name="black" />
       </visual>
       <collision>
@@ -23,5 +24,4 @@
       </collision>
       <inertial>
-        <!-- <origin xyz="0.0 0.0 0.0" rpy="0.0 0.0 ${3.0*M_PI/2.0}" /> -->
         <origin xyz="-0.05675 0.0 -0.0275" rpy="0.0 0.0 0.0" />
         <mass value="0.35" />
@@ -46,11 +46,7 @@
       </inertial>
     </link>
-    <!-- <xacro:hokuyo_ust_mount prefix="${prefix}" parent="${prefix}_base_link" topic="scan" min_angle="-1.57" max_angle="1.57" visualize="${visualize}" > -->
     <xacro:hokuyo_ust_mount prefix="${prefix}" parent="${prefix}_base_link" topic="scan" >
-      <origin xyz="0.0 0.0 0.0" rpy="0.0 0.0 0.0" />
+      <origin xyz="0.1105 0.0 0.0" rpy="0.0 0.0 0.0" />
     </xacro:hokuyo_ust_mount>
-    <!-- <gazebo reference="${prefix}_base_link">
-      <material>Gazebo/Black</material>
-    </gazebo> -->
   </xacro:macro>
 </robot>

File: sobit_mini_description/urdf/sensor/realsense_d435.urdf.xacro (robot description, xacro)
@@ -8,5 +8,6 @@
     </joint>
     <link name="${prefix}_base_link" />
-    <xacro:sensor_d435 parent="${prefix}_base_link" name="${prefix}" topics_ns="head_camera" >
+    <!-- <xacro:sensor_d435 parent="${prefix}_base_link" name="${prefix}" topics_ns="head_camera" > -->
+    <xacro:sensor_d435 parent="${prefix}_base_link" name="${prefix}" >
       <origin xyz="0.0 0.0 0.0" rpy="0.0 0.0 0.0" />
     </xacro:sensor_d435>

File: sobit_mini_description/urdf/stacks/stacks.urdf.xacro (robot description, xacro)
@@ -46,5 +46,5 @@
     <link name="pole_middle_${number}_link">
       <visual>
-        <origin xyz="0 0 0" rpy="0 ${M_PI} 0" />
+        <origin xyz="0.0 0.0 0.0" rpy="${M_PI/2.0} 0.0 0.0" />
         <geometry>
           <mesh filename="file://$(find sobit_mini_description)/meshes/body/pole_middle_134mm.stl" scale="${M_SCALE} ${M_SCALE} ${M_SCALE}" />
@@ -53,5 +53,5 @@
       </visual>
       <collision>
-        <origin xyz="0 0 0" rpy="0 0 0" />
+        <origin xyz="0.0 0.0 0.0" rpy="0.0 0.0 0.0" />
         <geometry>
           <cylinder length="0.0608" radius="0.006" />
@@ -75,12 +75,12 @@
     <link name="pole_top_${number}_link">
       <visual>
-        <origin xyz=" 0 0 0" rpy="0 0 0" />
-        <geometry>
-          <mesh filename="file://$(find sobit_mini_description)/meshes/body/pole_top_134mm.stl" scale="${M_SCALE} ${M_SCALE} ${M_SCALE}" />
+        <origin xyz="0.0 0.0 0.0" rpy="${M_PI/2.0} 0.0 0.0" />
+        <geometry>
+          <mesh filename="file://$(find sobit_mini_description)/meshes/body/pole_middle_134mm.stl" scale="${M_SCALE} ${M_SCALE} ${M_SCALE}" />
         </geometry>
         <material name="grey" />
       </visual>
       <collision>
-        <origin xyz="0 0 0" rpy="0 0 0" />
+        <origin xyz="0.0 0.0 0.0" rpy="0.0 0.0 0.0" />
         <geometry>
           <cylinder length="0.2032" radius="0.006" />
@@ -89,5 +89,5 @@
       <inertial>
         <mass value="0.060" />
-        <origin xyz="0 0 0" />
+        <origin xyz="0.0 0.0 0.0" />
         <inertia ixx="0.000206991" ixy="0.0" ixz="0.0"
                  iyy="0.000206991" iyz="0.0"
@@ -104,7 +104,7 @@
     <link name="pole_kinect_${number}_link">
       <visual>
-        <origin xyz="0 0 0.0" rpy="0 0 0" />
-        <geometry>
-          <mesh filename="package://turtlebot2_description/meshes/sensors/sensor_pole.dae" />
+        <origin xyz="0.0 0.0 0.0" rpy="0.0 0.0 0.0" />
+        <geometry>
+          <mesh filename="file://$(find turtlebot2_description)/meshes/sensors/sensor_pole.dae" />
         </geometry>
       </visual>
@@ -117,5 +117,5 @@
       <inertial>
         <mass value="0.020" />
-        <origin xyz="0 0 0" />
+        <origin xyz="0.0 0.0 0.0" />
         <inertia ixx="0.000014782" ixy="0.0" ixz="0.0"
                  iyy="0.000014782" iyz="0.0"
@@ -137,5 +137,5 @@
     <stack_bottom_pole parent="${parent}" number="5" x_loc="-0.055" y_loc="-0.120" z_loc="0.1028" />
     <joint name="plate_bottom_joint" type="fixed">
-      <origin xyz="0.02364 0.0 0.1306" rpy="0 0 0" />
+      <origin xyz="0.02364 0.0 0.1306" rpy="0.0 0.0 0.0" />
       <parent link="${parent}" />
       <child link="plate_bottom_link" />
@@ -143,11 +143,11 @@
     <link name="plate_bottom_link">
       <visual>
-        <origin xyz="0 0 0" rpy="0 0 0" />
-        <geometry>
-          <mesh filename="package://turtlebot2_description/meshes/stacks/hexagons/plate_bottom.dae" />
-        </geometry>
-      </visual>
-      <collision>
-        <origin xyz="-0.02364 0 0" rpy="0 0 0" />
+        <origin xyz="0.0 0.0 0.0" rpy="0.0 0.0 0.0" />
+        <geometry>
+          <mesh filename="file://$(find turtlebot2_description)/meshes/stacks/hexagons/plate_bottom.dae" />
+        </geometry>
+      </visual>
+      <collision>
+        <origin xyz="-0.02364 0.0 0.0" rpy="0.0 0.0 0.0" />
         <geometry>
           <cylinder length="0.006" radius="0.170" />
@@ -156,5 +156,5 @@
       <inertial>
         <mass value="0.520" />
-        <origin xyz="0 0 0" />
+        <origin xyz="0.0 0.0 0.0" />
         <inertia ixx="0.003328" ixy="0.0" ixz="0.0"
                  iyy="0.003328" iyz="0.0"
@@ -162,14 +162,14 @@
       </inertial>
     </link>
-    <stack_3d_sensor_pole parent="${parent}" number="0" x_loc="0.0381" y_loc="0.1505" z_loc="0.1735" />
+    <!-- <stack_3d_sensor_pole parent="${parent}" number="0" x_loc="0.0381" y_loc="0.1505" z_loc="0.1735" />
     <stack_3d_sensor_pole parent="${parent}" number="1" x_loc="0.0381" y_loc="-0.1505" z_loc="0.1735" />
     <stack_3d_sensor_pole parent="${parent}" number="2" x_loc="-0.0381" y_loc="0.1505" z_loc="0.1735" />
-    <stack_3d_sensor_pole parent="${parent}" number="3" x_loc="-0.0381" y_loc="-0.1505" z_loc="0.1735" />
-    <!-- <xacro:stack_middle_pole parent="${parent}" number="4" x_loc="0.0381" y_loc="0.1505" z_loc="0.13385" />
-    <xacro:stack_middle_pole parent="${parent}" number="5" x_loc="0.0381" y_loc="-0.1505" z_loc="0.13385" />
-    <xacro:stack_middle_pole parent="${parent}" number="6" x_loc="-0.0381" y_loc="0.1505" z_loc="0.13385" />
-    <xacro:stack_middle_pole parent="${parent}" number="7" x_loc="-0.0381" y_loc="-0.1505" z_loc="0.13385" /> -->
+    <stack_3d_sensor_pole parent="${parent}" number="3" x_loc="-0.0381" y_loc="-0.1505" z_loc="0.1735" /> -->
+    <xacro:stack_middle_pole parent="${parent}" number="4" x_loc= "0.0381" y_loc= "0.1505" z_loc="0.13385" />
+    <xacro:stack_middle_pole parent="${parent}" number="5" x_loc= "0.0381" y_loc="-0.1505" z_loc="0.13385" />
+    <xacro:stack_middle_pole parent="${parent}" number="6" x_loc="-0.0381" y_loc= "0.1505" z_loc="0.13385" />
+    <xacro:stack_middle_pole parent="${parent}" number="7" x_loc="-0.0381" y_loc="-0.1505" z_loc="0.13385" />
     <joint name="plate_middle_joint" type="fixed">
-      <origin xyz="-0.01364 0.0 0.2646" rpy="0 0 0" />
+      <origin xyz="-0.01364 0.0 0.2646" rpy="0.0 0.0 0.0" />
       <parent link="${parent}" />
       <child link="plate_middle_link" />
@@ -177,7 +177,7 @@
     <link name="plate_middle_link">
       <visual>
-        <origin xyz="0 0.0 0" rpy="0 0 0" />
-        <geometry>
-          <mesh filename="package://turtlebot2_description/meshes/stacks/hexagons/plate_top.dae" />
+        <origin xyz="0.0 0.0 0.0" rpy="0.0 0.0 0.0" />
+        <geometry>
+          <mesh filename="file://$(find turtlebot2_description)/meshes/stacks/hexagons/plate_top.dae" />
         </geometry>
       </visual>
@@ -185,10 +185,11 @@
         <origin xyz="0.01364 0.0 0.0" rpy="0 0 0" />
         <geometry>
-          <cylinder length="0.006" radius="0.170" />
+          <!-- <cylinder length="0.006" radius="0.170" /> -->
+          <mesh filename="file://$(find turtlebot2_description)/meshes/stacks/hexagons/plate_middle.dae" />
         </geometry>
       </collision>
       <inertial>
         <mass value="0.520" />
-        <origin xyz="0 0 0" />
+        <origin xyz="0.0 0.0 0.0" />
         <inertia ixx="0.003328" ixy="0.0" ixz="0.0"
                  iyy="0.003328" iyz="0.0"
@@ -196,4 +197,8 @@
       </inertial>
     </link>
+    <xacro:stack_top_pole parent="${parent}" number="0" x_loc= "0.0381" y_loc= "0.1505" z_loc="0.23035" />
+    <xacro:stack_top_pole parent="${parent}" number="1" x_loc= "0.0381" y_loc="-0.1505" z_loc="0.23035" />
+    <xacro:stack_top_pole parent="${parent}" number="2" x_loc="-0.0381" y_loc= "0.1505" z_loc="0.23035" />
+    <xacro:stack_top_pole parent="${parent}" number="3" x_loc="-0.0381" y_loc="-0.1505" z_loc="0.23035" />
   </xacro:macro>
 </robot>

Commit message: fix bag of wheel

File: sobit_mini_description/urdf/base/base.urdf.xacro (robot description, xacro)
@@ -54,5 +54,5 @@
       </inertial>
     </link>
-    <joint name="wheel_l_joint" type="continuous">
+    <joint name="wheel_l_joint" type="fixed">
       <parent link="base_link" />
       <child link="wheel_l_link" />
@@ -81,5 +81,5 @@
       </inertial>
     </link>
-    <joint name="wheel_r_joint" type="continuous">
+    <joint name="wheel_r_joint" type="fixed">
       <parent link="base_link" />
       <child link="wheel_r_link" />
