Commit message: new versionof dynamixel hardware

File: sobit_mini_description/urdf/base/base.urdf.xacro (robot description, xacro)
@@ -54,5 +54,5 @@
       </inertial>
     </link>
-    <joint name="wheel_l_joint" type="fixed">
+    <joint name="wheel_l_joint" type="continuous">
       <parent link="base_link" />
       <child link="wheel_l_link" />
@@ -74,12 +74,12 @@
       </collision>
       <inertial>
-        <mass value="0.01" />
-        <origin xyz="0 0 0" />
-        <inertia ixx="0.001" ixy="0.0" ixz="0.0"
-                 iyy="0.001" iyz="0.0"
-                 izz="0.001" />
-      </inertial>
-    </link>
-    <joint name="wheel_r_joint" type="fixed">
+        <mass value="10" />
+        <origin xyz="0 0 0" />
+        <inertia ixx="0.001" ixy="0.0" ixz="0.0"
+                 iyy="0.001" iyz="0.0"
+                 izz="0.001" />
+      </inertial>
+    </link>
+    <joint name="wheel_r_joint" type="continuous">
       <parent link="base_link" />
       <child link="wheel_r_link" />
@@ -101,5 +101,5 @@
       </collision>
       <inertial>
-        <mass value="0.01" />
+        <mass value="10" />
         <origin xyz="0 0 0" />
         <inertia ixx="0.001" ixy="0.0" ixz="0.0"
@@ -198,49 +198,4 @@
       </inertial>
     </link>
-    <gazebo reference="base_link">
-	  <selfCollide>true</selfCollide>
-      <mu1>1.0</mu1>
-      <mu2>1.0</mu2>
-    </gazebo>
-    <gazebo reference="caster_front_link">
-	  <selfCollide>true</selfCollide>
-      <mu1>0.0</mu1>
-      <mu2>0.0</mu2>
-    </gazebo>
-    <gazebo reference="caster_back_link">
-	  <selfCollide>true</selfCollide>
-      <mu1>0.0</mu1>
-      <mu2>0.0</mu2>
-    </gazebo>
-    <gazebo reference="wheel_l_link">
-	  <selfCollide>true</selfCollide>
-      <mu1>1.0</mu1>
-      <mu2>1.0</mu2>
-    </gazebo>
-    <gazebo reference="wheel_r_link">
-	  <selfCollide>true</selfCollide>
-      <mu1>1.0</mu1>
-      <mu2>1.0</mu2>
-    </gazebo>
-    <gazebo>
-      <plugin name="differential_drive_controller" filename="libgazebo_ros_diff_drive.so">
-        <leftJoint>wheel_l_joint</leftJoint>
-        <rightJoint>wheel_r_joint</rightJoint>
-        <wheelSeparation>0.23</wheelSeparation>
-        <wheelDiameter>0.070</wheelDiameter>
-        <wheelAcceleration>1.0</wheelAcceleration>
-        <wheelTorque>20</wheelTorque>
-        <commandTopic>/mobile_base/commands/velocity</commandTopic>
-        <odometryTopic>odom</odometryTopic>
-        <odometryFrame>odom</odometryFrame>
-        <robotBaseFrame>base_footprint</robotBaseFrame>
-        <odometrySource>1</odometrySource>
-        <publishWheelTF>true</publishWheelTF>
-        <publishOdom>true</publishOdom>
-        <publishWheelJointState>true</publishWheelJointState>
-        <legacyMode>false</legacyMode>
-        <updateRate>50.0</updateRate>
-      </plugin>
-    </gazebo>
   </xacro:macro>
 </robot>

File: sobit_mini_description/urdf/controllers.urdf.xacro (robot description, xacro)
@@ -12,5 +12,5 @@
         <xacro:unless value="${$(arg enable_gz)}">
           <plugin>dynamixel_hardware/DynamixelHardware</plugin>
-          <param name="usb_port">/dev/ttyUSB0</param>
+          <param name="port_name">/dev/ttyUSB0</param>
           <param name="baud_rate">1000000</param>
           <!-- <param name="use_dummy">true</param> -->
@@ -19,10 +19,14 @@
       <!-- Position Drive: Arm -->
       <joint name="r_arm_shoulder_roll_joint">
-        <param name="id">21</param>
+        <xacro:unless value="${$(arg enable_gz)}">
+          <param name="id">21</param>
+          <param name="control_mode">0</param>
+          <param name="interface">rs</param>
+        </xacro:unless>
         <command_interface name="position">
           <param name="min">-1.57</param>
           <param name="max">3.14</param>  <!-- 1.57 -->
         </command_interface>
-        <command_interface name="velocity"/>
+        <!-- <command_interface name="velocity"/> -->
         <state_interface name="position">
           <param name="initial_value">0.0</param>
@@ -32,10 +36,14 @@
       </joint>
       <joint name="r_arm_shoulder_pan_joint">
-        <param name="id">22</param>
+        <xacro:unless value="${$(arg enable_gz)}">
+          <param name="id">22</param>
+          <param name="control_mode">0</param>
+          <param name="interface">rs</param>
+        </xacro:unless>
         <command_interface name="position">
           <param name="min">-1.22</param>
           <param name="max">1.57</param>
         </command_interface>
-        <command_interface name="velocity"/>
+        <!-- <command_interface name="velocity"/> -->
         <state_interface name="position">
           <param name="initial_value">1.25</param>
@@ -45,10 +53,14 @@
       </joint>
       <joint name="r_arm_elbow_tilt_joint">
-        <param name="id">23</param>
+        <xacro:unless value="${$(arg enable_gz)}">
+          <param name="id">23</param>
+          <param name="control_mode">0</param>
+          <param name="interface">rs</param>
+        </xacro:unless>
         <command_interface name="position">
           <param name="min">0.0</param>
           <param name="max">1.57</param>
         </command_interface>
-        <command_interface name="velocity"/>
+        <!-- <command_interface name="velocity"/> -->
         <state_interface name="position">
           <param name="initial_value">0.0</param>
@@ -58,10 +70,14 @@
       </joint>
       <joint name="r_arm_wrist_tilt_joint">
-        <param name="id">24</param>
-        <command_interface name="position">
-          <param name="min">-1.57</param>
-          <param name="max">1.57</param>
-        </command_interface>
-        <command_interface name="velocity"/>
+        <xacro:unless value="${$(arg enable_gz)}">
+          <param name="id">24</param>
+          <param name="control_mode">0</param>
+          <param name="interface">rs</param>
+        </xacro:unless>
+        <command_interface name="position">
+          <param name="min">-1.57</param>
+          <param name="max">1.57</param>
+        </command_interface>
+        <!-- <command_interface name="velocity"/> -->
         <state_interface name="position">
           <param name="initial_value">0.0</param>
@@ -71,10 +87,14 @@
       </joint>
       <joint name="l_arm_shoulder_roll_joint">
-        <param name="id">11</param>
+        <xacro:unless value="${$(arg enable_gz)}">
+          <param name="id">11</param>
+          <param name="control_mode">0</param>
+          <param name="interface">rs</param>
+        </xacro:unless>
         <command_interface name="position">
           <param name="min">-3.14</param>
           <param name="max">1.57</param>
         </command_interface>
-        <command_interface name="velocity"/>
+        <!-- <command_interface name="velocity"/> -->
         <state_interface name="position">
           <param name="initial_value">0.0</param>
@@ -84,10 +104,14 @@
       </joint>
       <joint name="l_arm_shoulder_pan_joint">
-        <param name="id">12</param>
+        <xacro:unless value="${$(arg enable_gz)}">
+          <param name="id">12</param>
+          <param name="control_mode">0</param>
+          <param name="interface">rs</param>
+        </xacro:unless>
         <command_interface name="position">
           <param name="min">-1.57</param>
           <param name="max">1.22</param>
         </command_interface>
-        <command_interface name="velocity"/>
+        <!-- <command_interface name="velocity"/> -->
         <state_interface name="position">
           <param name="initial_value">-1.25</param>
@@ -97,10 +121,14 @@
       </joint>
       <joint name="l_arm_elbow_tilt_joint">
-        <param name="id">13</param>
+        <xacro:unless value="${$(arg enable_gz)}">
+          <param name="id">13</param>
+          <param name="control_mode">0</param>
+          <param name="interface">rs</param>
+        </xacro:unless>
         <command_interface name="position">
           <param name="min">-1.57</param>
           <param name="max">0.0</param>
         </command_interface>
-        <command_interface name="velocity"/>
+        <!-- <command_interface name="velocity"/> -->
         <state_interface name="position">
           <param name="initial_value">0.0</param>
@@ -110,10 +138,14 @@
       </joint>
       <joint name="l_arm_wrist_tilt_joint">
-        <param name="id">14</param>
-        <command_interface name="position">
-          <param name="min">-1.57</param>
-          <param name="max">1.57</param>
-        </command_interface>
-        <command_interface name="velocity"/>
+        <xacro:unless value="${$(arg enable_gz)}">
+          <param name="id">14</param>
+          <param name="control_mode">0</param>
+          <param name="interface">rs</param>
+        </xacro:unless>
+        <command_interface name="position">
+          <param name="min">-1.57</param>
+          <param name="max">1.57</param>
+        </command_interface>
+        <!-- <command_interface name="velocity"/> -->
         <state_interface name="position">
           <param name="initial_value">0.0</param>
@@ -124,10 +156,16 @@
       <!-- Position Drive: Hand -->
       <joint name="r_hand_joint">
-        <param name="id">25</param>
+        <xacro:unless value="${$(arg enable_gz)}">
+          <param name="id">25</param>
+          <param name="control_mode">6</param>
+          <param name="Goal_Current">50</param>
+          <param name="interface">rs</param>
+          <!-- <param name="gear_ratio">-59.504383354</param> -->
+        </xacro:unless>
         <command_interface name="position">
           <param name="min">0.0</param>
           <param name="max">1.57</param>
         </command_interface>
-        <command_interface name="velocity"/>
+        <!-- <command_interface name="velocity"/> -->
         <state_interface name="position">
           <param name="initial_value">0.0</param>
@@ -137,10 +175,16 @@
       </joint>
       <joint name="l_hand_joint">
-        <param name="id">15</param>
+        <xacro:unless value="${$(arg enable_gz)}">
+          <param name="id">15</param>
+          <param name="control_mode">6</param>
+          <param name="Goal_Current">50</param>
+          <param name="interface">rs</param>
+          <!-- <param name="gear_ratio">-59.504383354</param> -->
+        </xacro:unless>
         <command_interface name="position">
           <param name="min">-1.57</param>
           <param name="max">0.0</param>
         </command_interface>
-        <command_interface name="velocity"/>
+        <!-- <command_interface name="velocity"/> -->
         <state_interface name="position">
           <param name="initial_value">0.0</param>
@@ -151,10 +195,14 @@
       <!-- Position Drive: Head -->
       <joint name="head_camera_pan_joint">
-        <param name="id">3</param>
-        <command_interface name="position">
-          <param name="min">-1.57</param>
-          <param name="max">1.57</param>
-        </command_interface>
-        <command_interface name="velocity"/>
+        <xacro:unless value="${$(arg enable_gz)}">
+          <param name="id">3</param>
+          <param name="control_mode">0</param>
+          <param name="interface">rs</param>
+        </xacro:unless>
+        <command_interface name="position">
+          <param name="min">-1.57</param>
+          <param name="max">1.57</param>
+        </command_interface>
+        <!-- <command_interface name="velocity"/> -->
         <state_interface name="position">
           <param name="initial_value">0.0</param>
@@ -164,10 +212,14 @@
       </joint>
       <joint name="head_camera_tilt_joint">
-        <param name="id">4</param>
+        <xacro:unless value="${$(arg enable_gz)}">
+          <param name="id">4</param>
+          <param name="control_mode">0</param>
+          <param name="interface">rs</param>
+        </xacro:unless>
         <command_interface name="position">
           <param name="min">-0.45</param>
           <param name="max">0.45</param>
         </command_interface>
-        <command_interface name="velocity"/>
+        <!-- <command_interface name="velocity"/> -->
         <state_interface name="position">
           <param name="initial_value">0.0</param>
@@ -178,10 +230,14 @@
       <!-- Position Drive: Body -->
       <joint name="body_roll_joint">
-        <param name="id">2</param>
+        <xacro:unless value="${$(arg enable_gz)}">
+          <param name="id">2</param>
+          <param name="control_mode">0</param>
+          <param name="interface">rs</param>
+        </xacro:unless>
         <command_interface name="position">
           <param name="min">-4.14</param>
           <param name="max">4.14</param>
         </command_interface>
-        <command_interface name="velocity"/>
+        <!-- <command_interface name="velocity"/> -->
         <state_interface name="position">
           <param name="initial_value">0.0</param>

File: sobit_mini_description/urdf/head/head.transmission.xacro (robot description, xacro)
@@ -4,28 +4,4 @@
     <xacro:position_joint_transmission joint="${prefix}_camera_pan_joint" reduction="1" />
     <xacro:position_joint_transmission joint="${prefix}_camera_tilt_joint" reduction="1" />
-    <!--add transmission--> <!-- XXXXXXXXXX -->
-    <!-- <transmission name="${prefix}_camera_pan_trans">
-      <provideFeedback>true</provideFeedback>
-      <implicitSpringDamper>0</implicitSpringDamper>
-      <type>transmission_interface/SimpleTransmission</type>
-      <joint name="${prefix}_camera_pan_joint">
-        <hardwareInterface>hardware_interface/PositionJointInterface</hardwareInterface>
-      </joint>
-      <actuator name="${prefix}_camera_pan_motor">
-        <hardwareInterface>hardware_interface/PositionJointInterface</hardwareInterface>
-        <mechanicalReduction>1</mechanicalReduction>
-      </actuator>
-    </transmission>
-    <transmission name="${prefix}_camera_tilt_trans">
-      <provideFeedback>true</provideFeedback>
-      <implicitSpringDamper>0</implicitSpringDamper>
-      <type>transmission_interface/SimpleTransmission</type>
-      <joint name="${prefix}_camera_tilt_joint">
-        <hardwareInterface>hardware_interface/PositionJointInterface</hardwareInterface>
-      </joint>
-      <actuator name="${prefix}_camera_tilt_motor">
-        <hardwareInterface>hardware_interface/PositionJointInterface</hardwareInterface>
-      </actuator>
-    </transmission> -->
   </xacro:macro>
 </robot>

File: sobit_mini_description/urdf/head/head.urdf.xacro (robot description, xacro)
@@ -2,5 +2,4 @@
 <robot name="head" xmlns:xacro="http://ros.org/wiki/xacro">
   <xacro:include filename="$(find sobit_mini_description)/urdf/head/head.transmission.xacro" />
-  <!-- <xacro:include filename="$(find sobit_mini_description)/urdf/head/head.gazebo.xacro" /> -->
   <xacro:macro name="head" params="prefix parent">
     <joint name="${prefix}_pan_joint" type="revolute">
@@ -56,13 +55,4 @@
       </inertial>
     </link>
-    <!--plug-in to distribute joint condition data-->
-    <!-- <gazebo>
-      <plugin name="joint_state_publisher" filename="libgazebo_ros_joint_state_publisher.so">
-        <jointName>${prefix}_pan_joint, ${prefix}_tilt_joint</jointName>
-      </plugin>
-    </gazebo>
-    <gazebo reference="${prefix}_pan_link">
-      <material>Gazebo/Black</material>
-    </gazebo> -->
     <xacro:head_transmission prefix="${prefix}"/>
   </xacro:macro>
