Commit message: Update collistion sensor URDF

File: sobit_mini_description/urdf/gazebo.urdf.xacro (robot description, xacro)
@@ -34,5 +34,5 @@
           <pose>0.05 0.0 0.0 0.0 0.0 0.0</pose>
           <ignition_frame_id>${robot_name}/head_camera_optical_frame</ignition_frame_id>
-          <topic>${robot_name}/head_camera_base/depth/image_raw</topic>
+          <topic>${robot_name}/head_camera_base/depth/image_rect_raw</topic>
           <always_on>1</always_on>
           <visualize>true</visualize>

File: sobit_mini_description/urdf/sensor/lidar.urdf.xacro (robot description, xacro)
@@ -9,5 +9,5 @@
     <link name="${prefix}_base_link">
       <visual>
-        <origin xyz="0.0 0.0 ${M_PI}" rpy="0.0 0.0 0.0"/>
+        <origin xyz="0.0 0.0 0.0" rpy="0.0 0.0 ${M_PI}"/>
         <geometry>
           <mesh filename="file://$(find sobit_mini_description)/meshes/sobit_mini_urg_sup.dae" scale="0.001 0.001 0.001" />
@@ -16,5 +16,5 @@
       </visual>
       <collision>
-        <origin xyz="0.0 0.0 ${M_PI}" rpy="0.0 0.0 0.0" />
+        <origin xyz="0.0 0.0 0.0" rpy="0.0 0.0 ${M_PI}" />
         <geometry>
           <box size="0.092 0.184 0.007"/>
