Commit message: [FIX] Tilt gear ratio

File: sobit_mini_description/urdf/controllers.urdf.xacro (robot description, xacro)
@@ -213,9 +213,10 @@
         <state_interface name="effort"/>
       </joint>
-      <joint name="head_camera_tilt_joint">
+<joint name="head_camera_tilt_joint">
         <xacro:unless value="${$(arg enable_gz)}">
           <param name="id">4</param>
           <param name="control_mode">0</param>
           <param name="interface">rs</param>
+          <param name="gear_ratio">1.85</param>
         </xacro:unless>
         <command_interface name="position">
@@ -223,5 +224,4 @@
           <param name="max">0.45</param>
         </command_interface>
-        <!-- <command_interface name="velocity"/> -->
         <state_interface name="position">
           <param name="initial_value">0.0</param>

File: sobit_mini_description/urdf/head/head.urdf.xacro (robot description, xacro)
@@ -32,5 +32,5 @@
       <axis xyz="0 -1 0" />
       <!-- <axis xyz="0 1 0" /> -->
-      <limit effort="30" lower="-1" upper="1" velocity="${M_PI/2.0}" />
+      <limit effort="30" lower="-0.45" upper="0.45" velocity="${M_PI/2.0}" />
     </joint>
     <link name="${prefix}_tilt_link">

File: sobit_mini_description/urdf/sensor/realsense_d435.urdf.xacro (robot description, xacro)
@@ -3,5 +3,5 @@
   <xacro:macro name="realsense_d435" params="prefix parent">
     <joint name="${prefix}_base_joint" type="fixed">
-      <origin xyz="0.0045 0.0 0.169655" rpy="0.0 0.0 0.0" />
+      <origin xyz="0.0045 0.0 0.169655" rpy="0.0 0.075 0.0" />
       <parent link="${parent}" />
       <child link="${prefix}_base_link" />

Commit message: [FIX] ign to gz

File: sobit_mini_description/urdf/controllers.urdf.xacro (robot description, xacro)
@@ -7,6 +7,5 @@
       <hardware>
         <xacro:if value="${$(arg enable_gz)}">
-          <plugin>ign_ros2_control/IgnitionSystem</plugin>
-          <!-- <plugin>gazebo_ros2_control/GazeboHardware</plugin> -->
+          <plugin>gz_ros2_control/GazeboSimSystem</plugin>
         </xacro:if>
         <xacro:unless value="${$(arg enable_gz)}">
@@ -214,5 +213,5 @@
         <state_interface name="effort"/>
       </joint>
-<joint name="head_camera_tilt_joint">
+      <joint name="head_camera_tilt_joint">
         <xacro:unless value="${$(arg enable_gz)}">
           <param name="id">4</param>
@@ -265,6 +264,5 @@
       <ros2_control name="${name}_base" type="system">
         <hardware>
-          <plugin>ign_ros2_control/IgnitionSystem</plugin>
-          <!-- <plugin>gazebo_ros2_control/GazeboHardware</plugin> -->
+          <plugin>gz_ros2_control/GazeboSimSystem</plugin>
         </hardware>
         <joint name="wheel_l_joint">
@@ -290,9 +288,8 @@
       </gazebo>
     </xacro:if>
-    <!-- Ignition ROS2 Control -->
+    <!-- Gazebo Sim ROS2 Control -->
     <xacro:if value="${$(arg enable_gz)}">
       <gazebo>
-        <!-- <plugin filename="gz_ros2_control-system" name="gz_ros2_control::GazeboSimROS2ControlPlugin"> -->
-        <plugin filename="ign_ros2_control-system" name="ign_ros2_control::IgnitionROS2ControlPlugin">
+        <plugin filename="gz_ros2_control-system" name="gz_ros2_control::GazeboSimROS2ControlPlugin">
           <ros>
             <namespace>${robot_name}</namespace>

File: sobit_mini_description/urdf/gazebo.urdf.xacro (robot description, xacro)
@@ -8,6 +8,6 @@
         <sensor name="head_camera_color" type="camera">
           <pose>0.05 0.0 0.0 0.0 0.0 0.0</pose>
-          <ignition_frame_id>${robot_name}/head_camera_optical_frame</ignition_frame_id>
-          <topic>${robot_name}/head_camera_base/color/image_raw</topic>
+          <gz_frame_id>${robot_name}/head_camera_optical_frame</gz_frame_id>
+          <topic>${robot_name}/head_camera_base/color</topic>
           <always_on>1</always_on>
           <visualize>true</visualize>
@@ -33,6 +33,6 @@
         <sensor name="head_camera_depth" type="depth">
           <pose>0.05 0.0 0.0 0.0 0.0 0.0</pose>
-          <ignition_frame_id>${robot_name}/head_camera_optical_frame</ignition_frame_id>
-          <topic>${robot_name}/head_camera_base/depth/image_rect_raw</topic>
+          <gz_frame_id>${robot_name}/head_camera_optical_frame</gz_frame_id>
+          <topic>${robot_name}/head_camera_base/depth</topic>
           <always_on>1</always_on>
           <visualize>true</visualize>
@@ -57,5 +57,5 @@
         <sensor name="lidar" type="gpu_lidar">
           <pose>0 0 0 0 0 0</pose>
-          <ignition_frame_id>${robot_name}/lidar_laser</ignition_frame_id>
+          <gz_frame_id>${robot_name}/lidar_laser</gz_frame_id>
           <topic>${robot_name}/scan</topic>
           <always_on>1</always_on>

Commit message: [UPD] add parameter Return_Delay_Time.

File: sobit_mini_description/urdf/controllers.urdf.xacro (robot description, xacro)
@@ -17,5 +17,5 @@
         </xacro:unless>
       </hardware>
-      <!-- Position Drive: Arm -->
+      <!-- Position Drive: Right Arm -->
       <joint name="r_arm_shoulder_roll_joint">
         <xacro:unless value="${$(arg enable_gz)}">
@@ -23,4 +23,5 @@
           <param name="control_mode">0</param>
           <param name="interface">rs</param>
+          <param name="Return_Delay_Time">0</param>
         </xacro:unless>
         <command_interface name="position">
@@ -40,4 +41,5 @@
           <param name="control_mode">0</param>
           <param name="interface">rs</param>
+          <param name="Return_Delay_Time">0</param>
         </xacro:unless>
         <command_interface name="position">
@@ -57,4 +59,5 @@
           <param name="control_mode">0</param>
           <param name="interface">rs</param>
+          <param name="Return_Delay_Time">0</param>
         </xacro:unless>
         <command_interface name="position">
@@ -74,16 +77,18 @@
           <param name="control_mode">0</param>
           <param name="interface">rs</param>
-        </xacro:unless>
-        <command_interface name="position">
-          <param name="min">-1.57</param>
-          <param name="max">1.57</param>
-        </command_interface>
-        <!-- <command_interface name="velocity"/> -->
-        <state_interface name="position">
-          <param name="initial_value">0.0</param>
-        </state_interface>
-        <state_interface name="velocity"/>
-        <state_interface name="effort"/>
-      </joint>
+          <param name="Return_Delay_Time">0</param>
+        </xacro:unless>
+        <command_interface name="position">
+          <param name="min">-1.57</param>
+          <param name="max">1.57</param>
+        </command_interface>
+        <!-- <command_interface name="velocity"/> -->
+        <state_interface name="position">
+          <param name="initial_value">0.0</param>
+        </state_interface>
+        <state_interface name="velocity"/>
+        <state_interface name="effort"/>
+      </joint>
+      <!-- Position Drive: Left Arm -->
       <joint name="l_arm_shoulder_roll_joint">
         <xacro:unless value="${$(arg enable_gz)}">
@@ -91,4 +96,5 @@
           <param name="control_mode">0</param>
           <param name="interface">rs</param>
+          <param name="Return_Delay_Time">0</param>
         </xacro:unless>
         <command_interface name="position">
@@ -108,4 +114,5 @@
           <param name="control_mode">0</param>
           <param name="interface">rs</param>
+          <param name="Return_Delay_Time">0</param>
         </xacro:unless>
         <command_interface name="position">
@@ -125,4 +132,5 @@
           <param name="control_mode">0</param>
           <param name="interface">rs</param>
+          <param name="Return_Delay_Time">0</param>
         </xacro:unless>
         <command_interface name="position">
@@ -142,17 +150,18 @@
           <param name="control_mode">0</param>
           <param name="interface">rs</param>
-        </xacro:unless>
-        <command_interface name="position">
-          <param name="min">-1.57</param>
-          <param name="max">1.57</param>
-        </command_interface>
-        <!-- <command_interface name="velocity"/> -->
-        <state_interface name="position">
-          <param name="initial_value">0.0</param>
-        </state_interface>
-        <state_interface name="velocity"/>
-        <state_interface name="effort"/>
-      </joint>
-      <!-- Position Drive: Hand -->
+          <param name="Return_Delay_Time">0</param>
+        </xacro:unless>
+        <command_interface name="position">
+          <param name="min">-1.57</param>
+          <param name="max">1.57</param>
+        </command_interface>
+        <!-- <command_interface name="velocity"/> -->
+        <state_interface name="position">
+          <param name="initial_value">0.0</param>
+        </state_interface>
+        <state_interface name="velocity"/>
+        <state_interface name="effort"/>
+      </joint>
+      <!-- Position Drive:  Right Hand -->
       <joint name="r_hand_joint">
         <xacro:unless value="${$(arg enable_gz)}">
@@ -163,4 +172,5 @@
           <param name="interface">rs</param>
           <!-- <param name="gear_ratio">-59.504383354</param> -->
+          <param name="Return_Delay_Time">0</param>
         </xacro:unless>
         <command_interface name="position">
@@ -175,4 +185,5 @@
         <state_interface name="effort"/>
       </joint>
+      <!-- Position Drive:  Left Hand -->
       <joint name="l_hand_joint">
         <xacro:unless value="${$(arg enable_gz)}">
@@ -183,4 +194,5 @@
           <param name="interface">rs</param>
           <!-- <param name="gear_ratio">-59.504383354</param> -->
+          <param name="Return_Delay_Time">0</param>
         </xacro:unless>
         <command_interface name="position">
@@ -201,4 +213,5 @@
           <param name="control_mode">0</param>
           <param name="interface">rs</param>
+          <param name="Return_Delay_Time">0</param>
         </xacro:unless>
         <command_interface name="position">
@@ -218,4 +231,5 @@
           <param name="control_mode">0</param>
           <param name="interface">rs</param>
+          <param name="Return_Delay_Time">0</param>
           <param name="gear_ratio">1.85</param>
         </xacro:unless>
@@ -236,4 +250,5 @@
           <param name="control_mode">0</param>
           <param name="interface">rs</param>
+          <param name="Return_Delay_Time">0</param>
         </xacro:unless>
         <command_interface name="position">
